File: hardware/base-station/esp32_p3.kicad_sch (KiCad schematic)
At the start: 35 parts, among them U1 W25Q64JVXGIQ TR, U15 479480001, U3 ESP32-S3, Y1 ECS-.327-6-16R-TR, Y2 ECS-400-10-37B2-CKY-TR

Commit message: hardware: BOM-cost pass across all four boards
Component changes from a cross-board cost review. Per-board component cost
(USD @~100qty): rocket $86.21 -> $61.39, base station $35.91 -> $29.89, with
the LoRa daughterboard and GNSS SAM-M10Q board added to the shared BOM.

Memory architecture
  - Rocket: MR25H10 MRAM deleted; the log ring moves to in-package PSRAM.
    ESP32-S3 -> ESP32-S3RH2 (2 MB quad PSRAM, no in-package flash, same land
    pattern; SPICS1/GPIO26 was already unconnected on every board).
    Persistence across boots is knowingly given up.
  - Rocket NAND F35SQB004G-WWT -> GD5F2GQ5UEYIGR: pin- and footprint-identical
    (verified against the U11 land pattern), 4 Gbit -> 2 Gbit, $11.61 -> $3.50.
    Needs the 4096 -> 2048 B page migration in firmware.
  - Base station: dedicated log flash deleted entirely. It wrote one ~183 B CSV
    row per received packet at the 2 Hz downlink (~366 B/s, and only while a
    flight is active), so 256 MB was ~204 hours of headroom. The firmware
    already falls back to the existing SPIFFS partition, so this promotes a
    tested path rather than needing new code.
  - Boot flash W25Q64JVXGIQ -> W25Q128JVSIQ on all four positions: 16 MB for
    LESS money ($3.10 -> $2.21). SCHEMATIC ONLY - the boards still need
    "Update PCB from Schematic" plus re-placement, since SOIC-8 208mil is 2.2x
    the DFN's area. The DFN's 9th (exposed) pad was a redundant GND tie; pin 4
    is GND on all four, so nothing is lost.

Power
  - LoRa + GNSS keep TPS62913 (low-noise, RF rails). The rocket briefly moved
    to it and was REVERTED to TPS62152: the TPS62913 is forced-PWM with 5 mA
    quiescent, which would have raised the pad-idle floor ~6x against the
    light-sleep work.
  - Base load switch TPS22810 -> TPS22918 (identical footprint and pin order;
    pin 3 EN/UVLO -> ON is safe because it was driven as a plain enable).
    CT cap 10 nF -> 2.2 nF to match the rocket's ramp; R8 (QOD->VOUT) deleted.
  - LoRa gains a 7.5k S-CONF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
Parts:
- U1: value W25Q64JVXGIQ TR -> W25Q128JVSIQ; footprint Footprints:DFN_XGIQ TR_WIN -> Footprints:SOIC-8_W25Q128JVSIQ
- U3: value ESP32-S3 -> ESP32-S3RH2
Changed lines of the file:
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@@
 			)
 		)
-		(property "Value" "W25Q64JVXGIQ TR"
+		(property "Value" "W25Q128JVSIQ"
 			(at 65.405 106.045 0)
 			(show_name no)
@@
 			)
 		)
-		(property "Footprint" "Footprints:DFN_XGIQ TR_WIN"
+		(property "Footprint" "Footprints:SOIC-8_W25Q128JVSIQ"
 			(at 21.59 115.57 0)
 			(hide yes)
@@
 			)
 		)
-		(property "Value" "ESP32-S3"
+		(property "Value" "ESP32-S3RH2"
 			(at 146.05 31.75 0)
 			(show_name no)

Commit message: hardware: battery protection, boost swap, and a capacitor voltage audit
Base station power chain, all verified against exported netlists:

- Protection: MAX17303G+ gauge/protector and its NTMD6N02R2G FET pair
  replaced by DW01A + 2x FS8205A. The MAX17303 had no firmware driver and
  the board never had a working coulomb counter, so state of charge already
  came from the voltage curve in bs_battery_soc.h; it now reads a 1M/1M
  divider on GPIO1. The FETs move from the positive rail to the negative
  one because the DW01A has no charge pump, so board ground is now P-,
  separated from the cell's B- by the FET stack. Two FS8205A in parallel
  put the 150 mV overcurrent trip at ~4.8-6.0 A instead of ~2.4-3.0 A.
  TH1 moves onto the BQ21040's TS pin, replacing a fixed 10k that had been
  defeating thermal charge cutoff.

- V_LORA retargeted 7.49 V -> 4.95 V and LM5157QRTERQ1 -> TPS61023DRLR.
  Nothing needed 7.4 V (everything downstream is 3.3 V behind the
  TPS62913), while an RFD868x-class radio is 5 V nominal with a 6 V
  absolute maximum, so the old rail put it permanently out of reach. Being
  synchronous and internally compensated also dropped D2, C35-C38 and R10.
  Inductor stays the fleet 2.2 uH: inside TI's 0.37-2.9 uH range and the
  only value meeting their ripple-under-40%-of-average guidance at load.

- Keystone 1043P holder -> MYOUNG BH-18650-A5BJ001-2D. Terminal pitch
  72.30 vs 72.22 mm, so the battery nets did not move; BT2 is rotated 180
  degrees because this part's positive end is mirrored.

Across all four boards:

- Every crystal was mis-loaded. 32.768 kHz parts saw ~9 pF against a 6 pF
  spec and the 40 MHz saw 12.5 pF against 10 pF, both pulling slow. Moved
  to Seiko SC-32S (12.5 pF) with 22 pF load caps, and the 40 MHz caps to
  18 pF. The tolerance being paid for had been swamped several times over.

- Capacitor voltage audit, new Min V rating column in the BOM. Three parts
  were operating outside their rating on 8.4 V rails: 47 uF and 100 u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
Parts:
- added J6: Conn_01x04, Connector_JST:JST_SH_BM04B-SRSS-TB_1x04-1MP_P1.00mm_Vertical, symbol Connector_Generic:Conn_01x04
- C2, C4: value 15 pF -> 22 pF
- C3, C6: value 22 pF -> 18 pF
- U1: symbol Custom:W25Q64JVXGIQ_TR -> Custom:W25Q128JVSIQ
- Y1: value ECS-.327-6-16R-TR -> SC-32S-32.768kHz-12.5pF; footprint Footprints:XTAL_ECS-.327-6-16R-TR -> Footprints:XTAL_SC-32S_3215; symbol Custom:ECS-.327-6-16R-TR -> Custom:SC-32S-32.768kHz-12.5pF
Connections:
- net GND: now also J6.1 (Pin_1); no longer U1.9
- net LoRa_RX: now also J6.3 (Pin_3)
- net LoRa_TX: now also J6.4 (Pin_4)
- net SCL_SENS: no longer U3.39 (GPIO34)
- net SDA_SENS: no longer U3.38 (GPIO33)
- net Volt_Read: now reaches U3.6 (GPIO1)
- new net V_LORA: J6.2 (Pin_2)
Other:
- note added: "E220-900MM22S LoRa Module"

Commit message: hardware: place Q3 and bump C10 to 10 uF on the base-station
Places the third FS8205A whose schematic went in with the previous
commit, so the protection stack is now Q1/Q2/Q3 on the board as well as
on the sheet.

C10 goes 1 uF -> 10 uF. Changed in both esp32_p3.kicad_sch and the
layout, so schematic and board agree.

The battery sheet is rewired - +9 wires, +3 junctions, -5 labels - with
no change to its part set.

Layout otherwise: 38 parts repositioned, 24 track segments removed, 35
vias added, one zone removed.

Co-Authored-By: Claude Opus 5 <noreply@anthropic.com>
Parts:
- C10: value 1 uF -> 10 uF
Connections:
- net SCL_SENS: now also U3.39 (GPIO34)
- net SDA_SENS: now also U3.38 (GPIO33)
Changed lines of the file:
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@@
 		)
 	)
+	(global_label "SDA_SENS"
+		(shape input)
+		(at 171.45 107.315 0)
+		(fields_autoplaced yes)
+		(effects
+			(font
+				(size 1.27 1.27)
+			)
+			(justify left)
+		)
+		(property "Intersheetrefs" "${INTERSHEET_REFS}"
+			(at 183.8694 107.315 0)
+			(hide yes)
+			(show_name no)
+			(do_not_autoplace no)
+			(effects
+				(font
+					(size 1.27 1.27)
+				)
+				(justify left)
+			)
+		)
+	)
 	(global_label "VDD_SPI"
 		(shape input)
@@
 		)
 	)
+	(global_label "SCL_SENS"
+		(shape input)
+		(at 171.45 109.855 0)
+		(fields_autoplaced yes)
+		(effects
+			(font
+				(size 1.27 1.27)
+			)
+			(justify left)
+		)
+		(property "Intersheetrefs" "${INTERSHEET_REFS}"
+			(at 183.8089 109.855 0)
+			(hide yes)
+			(show_name no)
+			(do_not_autoplace no)
+			(effects
+				(font
+					(size 1.27 1.27)
+				)
+				(justify left)
+			)
+		)
+	)
 	(global_label "M_MOSI"
 		(shape input)
@@
 			)
 		)
-		(property "Value" "1 uF"
+		(property "Value" "10 uF"
 			(at 183.515 39.37 0)
 			(show_name no)

Commit message: hardware: CHIP_PU reset RC fix on the base-station and rocket-computer S3
Both boards had Espressif's 10 k / 1 uF reset network drawn with the
capacitor on the supply side of the pull-up, where it acts as rail
decoupling and produces no delay. The LoRa V3 review (#692, finding 1)
turned this up; the same construction was present on all three boards.

  base-station    C8  (1 uF) +3V3 -> Net-(U3-CHIP_PU),  R1  reversed
  rocket-computer C25 (1 uF) +3V3 -> Net-(U15-CHIP_PU), R36 reversed

With the cap on the supply side the only capacitance on the CHIP_PU node
is the pin's own (~5 pF), so tau ~= 50 ns and CHIP_PU tracks the rail.
On the pin, tau = 10 k x 1 uF = 10 ms, past Espressif's 50 us t_STBL
floor. Closes the rocket-computer pre-fab review's H8.

Verified by netlist export: Net-(U3-CHIP_PU) = {C8.1, R1.2, U3.4} and
Net-(U15-CHIP_PU) = {C25.1, R36.2, U15.4}; component counts unchanged on
both boards.

Co-Authored-By: Claude Opus 5 <noreply@anthropic.com>
Connections:
- net +3V3: now also R1.1; no longer C8.1, R1.2
- net at U3.4 (CHIP_PU): now also C8.1, R1.2; no longer R1.1
Other:
- moved on the sheet: C8, R1
Changed lines of the file:
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@@
 	)
 	(junction
-		(at 113.03 29.845)
+		(at 111.125 45.085)
 		(diameter 0)
 		(color 0 0 0 0)
@@
 	(wire
 		(pts
+			(xy 120.65 45.085) (xy 120.65 53.975)
+		)
+		(stroke
+			(width 0)
+			(type default)
+		)
+	)
+	(wire
+		(pts
 			(xy 103.505 63.5) (xy 104.775 63.5)
 		)
@@
 	(wire
 		(pts
+			(xy 111.125 42.545) (xy 111.125 45.085)
+		)
+		(stroke
+			(width 0)
+			(type default)
+		)
+	)
+	(wire
+		(pts
 			(xy 106.68 86.36) (xy 79.375 86.36)
 		)
@@
 	(wire
 		(pts
-			(xy 175.895 33.02) (xy 183.515 33.02)
+			(xy 111.125 45.085) (xy 120.65 45.085)
 		)
 		(stroke
@@
 	(wire
 		(pts
-			(xy 217.17 72.39) (xy 217.17 74.93)
+			(xy 175.895 33.02) (xy 183.515 33.02)
 		)
 		(stroke
@@
 	(wire
 		(pts
-			(xy 98.425 55.88) (xy 85.725 55.88)
+			(xy 217.17 72.39) (xy 217.17 74.93)
 		)
 		(stroke
@@
 	(wire
 		(pts
-			(xy 79.375 86.36) (xy 77.47 86.36)
+			(xy 98.425 55.88) (xy 85.725 55.88)
 		)
 		(stroke
@@
 	(wire
 		(pts
-			(xy 113.03 29.845) (xy 113.03 53.975)
+			(xy 79.375 86.36) (xy 77.47 86.36)
 		)
 		(stroke
@@
 	(wire
 		(pts
-			(xy 44.45 119.38) (xy 44.45 121.92)
+			(xy 111.125 32.385) (xy 111.125 34.925)
 		)
 		(stroke
@@
 	(wire
 		(pts
-			(xy 91.44 36.195) (xy 94.615 36.195)
+			(xy 44.45 119.38) (xy 44.45 121.92)
 		)
 		(stroke
@@
 	(wire
 		(pts
-			(xy 113.03 29.845) (xy 118.11 29.845)
+			(xy 91.44 36.195) (xy 94.615 36.195)
 		)
 		(stroke
@@
 	(wire
 		(pts
-			(xy 113.03 28.575) (xy 113.03 29.845)
-		)
-		(stroke
-			(width 0)
-			(type default)
-		)
-	)
-	(wire
-		(pts
 			(xy 107.95 59.055) (xy 107.95 36.195)
 		)
@@
 	(symbol
 		(lib_id "power:GND")
-		(at 118.11 37.465 0)
+		(at 111.125 52.705 0)
 		(unit 1)
 		(body_style 1)
@@
 		(dnp no)
 		(property "Reference" "#PWR011"
-			(at 118.11 43.815 0)
+			(at 111.125 59.055 0)
 			(hide yes)
 			(show_name no)
@@
 		)
 		(property "Value" "GND"
-			(at 120.015 41.275 0)
+			(at 113.03 56.515 0)
 			(show_name no)
 			(do_not_autoplace no)
@@
 		)
 		(property "Footprint" ""
-			(at 118.11 37.465 0)
+			(at 111.125 52.705 0)
 			(hide yes)
 			(show_name no)
@@
 		)
 		(property "Datasheet" ""
-			(at 118.11 37.465 0)
+			(at 111.125 52.705 0)
 			(hide yes)
 			(show_name no)
@@
 		)
 		(property "Description" ""
-			(at 118.11 37.465 0)
+			(at 111.125 52.705 0)
 			(hide yes)
 			(show_name no)
@@
 	(symbol
 		(lib_id "power:+3V3")
-		(at 113.03 28.575 0)
+		(at 111.125 32.385 0)
 		(unit 1)
 		(body_style 1)
@@
 		(fields_autoplaced yes)
 		(property "Reference" "#PWR010"
-			(at 113.03 32.385 0)
+			(at 111.125 36.195 0)
 			(hide yes)
 			(show_name no)
@@
 		)
 		(property "Value" "+3V3"
-			(at 113.03 24.13 0)
+			(at 111.125 27.94 0)
 			(show_name no)
 			(do_not_autoplace no)
@@
 		)
 		(property "Footprint" ""
-			(at 113.03 28.575 0)
+			(at 111.125 32.385 0)
 			(hide yes)
 			(show_name no)
@@
 		)
 		(property "Datasheet" ""
-			(at 113.03 28.575 0)
+			(at 111.125 32.385 0)
 			(hide yes)
 			(show_name no)
@@
 		)
 		(property "Description" ""
-			(at 113.03 28.575 0)
+			(at 111.125 32.385 0)
 			(hide yes)
 			(show_name no)
@@
 	(symbol
 		(lib_id "Device:C")
-		(at 118.11 33.655 0)
+		(at 111.125 48.895 0)
 		(unit 1)
 		(body_style 1)
@@
 		(dnp no)
 		(property "Reference" "C8"
-			(at 118.11 31.115 0)
+			(at 111.125 46.355 0)
 			(show_name no)
 			(do_not_autoplace no)
@@
 		)
 		(property "Value" "1 uF"
-			(at 118.11 36.195 0)
+			(at 111.125 51.435 0)
 			(show_name no)
 			(do_not_autoplace no)
@@
 		)
 		(property "Footprint" "Capacitor_SMD:C_0402_1005Metric"
-			(at 119.0752 37.465 0)
+			(at 112.0902 52.705 0)
 			(hide yes)
 			(show_name no)
@@
 		)
 		(property "Datasheet" ""
-			(at 118.11 33.655 0)
+			(at 111.125 48.895 0)
 			(hide yes)
 			(show_name no)
@@
 		)
 		(property "Description" ""
-			(at 118.11 33.655 0)
+			(at 111.125 48.895 0)
 			(hide yes)
 			(show_name no)
@@
 	(symbol
 		(lib_id "Device:R_US")
-		(at 116.84 53.975 270)
+		(at 111.125 38.735 0)
 		(unit 1)
 		(body_style 1)
@@
 		(fields_autoplaced yes)
 		(property "Reference" "R1"
-			(at 116.84 47.625 90)
+			(at 113.665 37.4649 0)
 			(show_name no)
 			(do_not_autoplace no)
@@
 					(size 1.27 1.27)
 				)
+				(justify left)
 			)
 		)
 		(property "Value" "10 k"
-			(at 116.84 50.165 90)
+			(at 113.665 40.0049 0)
 			(show_name no)
 			(do_not_autoplace no)
@@
 					(size 1.27 1.27)
 				)
+				(justify left)
 			)
 		)
 		(property "Footprint" "Resistor_SMD:R_0402_1005Metric"
-			(at 116.586 54.991 90)
+			(at 112.141 38.989 90)
 			(hide yes)
 			(show_name no)
@@
 		)
 		(property "Datasheet" ""
-			(at 116.84 53.975 0)
+			(at 111.125 38.735 0)
 			(hide yes)
 			(show_name no)
@@
 		)
 		(property "Description" ""
-			(at 116.84 53.975 0)
+			(at 111.125 38.735 0)
 			(hide yes)
 			(show_name no)

Commit message: hardware: 40 MHz crystal load caps 18 pF -> 12 pF on all four networks
All four ECS-400-10-37B2-CKY-TR networks run 18 pF per leg against a
CL = 10 pF part. Measured per-leg stray (trace at ~0.09 pF/mm over a plane
0.1 mm away, plus pads, plus the S3's 2 pF CIN from datasheet Table 5-4)
puts the actual load near 12.5 pF -- about -33 ppm, outside the crystal's
own +/-10 ppm and outside Espressif's "tune to within +/-10 ppm".

12 pF lands the load near nominal and, more importantly, more than doubles
oscillator startup margin: |Rneg| goes as 1/(C1*C2), so 18 -> 12 pF is a
2.25x improvement against a 40 ohm ESR crystal.

  lora-daughterboard  C90 C92   Y6 -> U28 (S3)   +9 ppm   no RF
  rocket-computer     C20 C22   Y2 -> U15 (S3)   +9 ppm   BLE
  rocket-computer     C48 C49   Y4 -> U17 (P4)   +9 ppm   no radio on P4
  base-station        C3  C6    Y2 -> U3  (S3)  +17 ppm   BLE  -- see #704

The base station is the exception. Its crystal legs are 3.7 and 7.2 mm
against 11-12 mm on the others, so ~0.5 pF less stray per leg, and 12 pF
leaves it at +17 ppm. It is still an improvement on the -28 ppm it has
today, and both the base station and the rocket-computer S3 run BLE, where
the +/-10 ppm is a live radio spec rather than cosmetic. Issue #704 tracks
lengthening the base-station clock traces to match, which brings it to
+9 ppm and lets one cap value serve every board.

Two caveats recorded rather than hidden: the P4's XTAL pin capacitance is
not published, so its 2 pF is assumed from the S3 (costs nothing there --
no radio); and +9 ppm on the rocket-computer S3 has no margin against the
~1 pF uncertainty in the stray estimate. Measure and trim on the first
article, as Espressif's checklist instructs.

New BOM line: CL05C120JB5NNNC (12 pF 0402 C0G), 8 pieces. Only the LoRa
pair carries MPN fields today; those were kept in step.

Verified with kicad-cli on all three projects: zero connectivity changes,
no components added or removed, ERC violation counts identical before a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
Parts:
- C3, C6: value 18 pF -> 12 pF
Changed lines of the file:
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@@
 			)
 		)
-		(property "Value" "18 pF"
+		(property "Value" "12 pF"
 			(at 74.295 56.515 0)
 			(show_name no)
@@
 			)
 		)
-		(property "Value" "18 pF"
+		(property "Value" "12 pF"
 			(at 85.725 73.025 0)
 			(show_name no)

Commit message: hardware: MPN + Mfr on every purchased part of the three ESP32 boards
Closes the LoRa pre-fab review's finding 3, extended to the sibling boards.
Every non-DNP symbol now names the exact part the cross-board BOM prices, so
the schematic can no longer imply a part that was never quoted.

401 of 401 purchasable parts carry an MPN. The only exemptions are the three
DNP v3.x provisions on the rocket-computer (R74/R75 499 k, R76 0 R): not
fitted, so never purchased, so correctly absent from the BOM.

Values normalised so each part resolves to one BOM line:

  LoRa R74  "10 K" -> "10 k"   capital K split one part across two lines
  LoRa D6   "LED"  -> "Green"  no colour recorded, so no MPN could attach
  Y1/Y3/Y5  "SC-32S-32.768kHz-12.5pF" -> "ABS07-32.768KHZ-T"

Two stale legacy MP fields disagreed with both the Value and the BOM and were
corrected -- a symbol carrying two part numbers is the wrong-part-order hazard
this pass exists to remove:

  rocket U19  TPS259824LNRGER -> ...RGET.  Same die and RGE-24 package; the
              suffix is reel quantity, and power-eco.md documents RGET.
  base   U9   TPS63021DSJR -> TPS63020DSJR.  These are NOT interchangeable:
              63021 is fixed 3.3 V, 63020 is adjustable. U9 pin 3 (FB) drives
              a real divider (R13 1 M / R16 180 k -> 0.5 x (1 + 1M/180k) =
              3.28 V), which only the adjustable part uses. BOM was right.

The ABS07 keeps the existing XTAL_SC-32S_3215 footprint: both parts are
2-pad 3.2 x 1.5 mm tuning forks, so the land is correct and only the
footprint's name now reads for the superseded vendor.

ERC clean on all three boards after the pass.

Co-Authored-By: Claude Opus 5 <noreply@anthropic.com>
Parts:
- C1, C12, C14, C16, C17, C9: MPN (none) -> CL05B104KO5NNNC; Mfr (none) -> Samsung
- C10, C15, C19: MPN (none) -> CL05A106MQ5NUNC; Mfr (none) -> Samsung
- C11: MPN (none) -> CL05B103KB5NNNC; Mfr (none) -> Samsung
- C13, C18, C8: MPN (none) -> CL05A105KO5NNNC; Mfr (none) -> Samsung
- C2, C4: MPN (none) -> CL05C220JB5NNNC; Mfr (none) -> Samsung
- C25, C26: MPN (none) -> CC0402CRNPO9BN1R5; Mfr (none) -> Yageo
- C3, C6: MPN (none) -> CL05C120JB5NNNC; Mfr (none) -> Samsung
- J6: MPN (none) -> BM04B-SRSS-TB; Mfr (none) -> JST
- L2: MPN (none) -> LQW15AN24NH00D; Mfr (none) -> Murata
- L3: MPN (none) -> LQG15HS2N0S02D; Mfr (none) -> Murata
- L4: MPN (none) -> LQW15AN4N3C00D; Mfr (none) -> Murata
- L7: MPN (none) -> LQW15AN2N7C00D; Mfr (none) -> Murata
- R1, R2: MPN (none) -> RC0402FR-0710KL; Mfr (none) -> Yageo
- R3, R4: MPN (none) -> RC0402FR-0722RL; Mfr (none) -> Yageo
- R5, R6: MPN (none) -> RC0402FR-075K11L; Mfr (none) -> Yageo
- S3: MPN (none) -> KMR221GLFS; Mfr (none) -> C&K
- U1: MPN (none) -> W25Q128JVSIQ; Mfr (none) -> Winbond
- U15: MPN (none) -> 479480001; Mfr (none) -> Molex
- U3: MPN (none) -> ESP32-S3RH2; Mfr (none) -> Espressif
- Y1: value SC-32S-32.768kHz-12.5pF -> ABS07-32.768KHZ-T; MPN (none) -> ABS07-32.768KHZ-T; Mfr (none) -> Abracon
- Y2: MPN (none) -> ECS-400-10-37B2-CKY-TR; Mfr (none) -> ECS
