File: hardware/base-station/external_charger.kicad_sch (KiCad schematic)
At the start: 25 parts, among them J4 S3B-XH-A, U12 MP2672AGD-0000-Z

Commit message: hardware: BOM-cost pass across all four boards
Component changes from a cross-board cost review. Per-board component cost
(USD @~100qty): rocket $86.21 -> $61.39, base station $35.91 -> $29.89, with
the LoRa daughterboard and GNSS SAM-M10Q board added to the shared BOM.

Memory architecture
  - Rocket: MR25H10 MRAM deleted; the log ring moves to in-package PSRAM.
    ESP32-S3 -> ESP32-S3RH2 (2 MB quad PSRAM, no in-package flash, same land
    pattern; SPICS1/GPIO26 was already unconnected on every board).
    Persistence across boots is knowingly given up.
  - Rocket NAND F35SQB004G-WWT -> GD5F2GQ5UEYIGR: pin- and footprint-identical
    (verified against the U11 land pattern), 4 Gbit -> 2 Gbit, $11.61 -> $3.50.
    Needs the 4096 -> 2048 B page migration in firmware.
  - Base station: dedicated log flash deleted entirely. It wrote one ~183 B CSV
    row per received packet at the 2 Hz downlink (~366 B/s, and only while a
    flight is active), so 256 MB was ~204 hours of headroom. The firmware
    already falls back to the existing SPIFFS partition, so this promotes a
    tested path rather than needing new code.
  - Boot flash W25Q64JVXGIQ -> W25Q128JVSIQ on all four positions: 16 MB for
    LESS money ($3.10 -> $2.21). SCHEMATIC ONLY - the boards still need
    "Update PCB from Schematic" plus re-placement, since SOIC-8 208mil is 2.2x
    the DFN's area. The DFN's 9th (exposed) pad was a redundant GND tie; pin 4
    is GND on all four, so nothing is lost.

Power
  - LoRa + GNSS keep TPS62913 (low-noise, RF rails). The rocket briefly moved
    to it and was REVERTED to TPS62152: the TPS62913 is forced-PWM with 5 mA
    quiescent, which would have raised the pad-idle floor ~6x against the
    light-sleep work.
  - Base load switch TPS22810 -> TPS22918 (identical footprint and pin order;
    pin 3 EN/UVLO -> ON is safe because it was driven as a plain enable).
    CT cap 10 nF -> 2.2 nF to match the rocket's ramp; R8 (QOD->VOUT) deleted.
  - LoRa gains a 7.5k S-CONF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
Parts:
- C48: value 10 uF -> 22 uF
Changed lines of the file:
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@@
 			)
 		)
-		(property "Value" "10 uF"
+		(property "Value" "22 uF"
 			(at 94.615 72.39 0)
 			(show_name no)

Commit message: hardware: battery protection, boost swap, and a capacitor voltage audit
Base station power chain, all verified against exported netlists:

- Protection: MAX17303G+ gauge/protector and its NTMD6N02R2G FET pair
  replaced by DW01A + 2x FS8205A. The MAX17303 had no firmware driver and
  the board never had a working coulomb counter, so state of charge already
  came from the voltage curve in bs_battery_soc.h; it now reads a 1M/1M
  divider on GPIO1. The FETs move from the positive rail to the negative
  one because the DW01A has no charge pump, so board ground is now P-,
  separated from the cell's B- by the FET stack. Two FS8205A in parallel
  put the 150 mV overcurrent trip at ~4.8-6.0 A instead of ~2.4-3.0 A.
  TH1 moves onto the BQ21040's TS pin, replacing a fixed 10k that had been
  defeating thermal charge cutoff.

- V_LORA retargeted 7.49 V -> 4.95 V and LM5157QRTERQ1 -> TPS61023DRLR.
  Nothing needed 7.4 V (everything downstream is 3.3 V behind the
  TPS62913), while an RFD868x-class radio is 5 V nominal with a 6 V
  absolute maximum, so the old rail put it permanently out of reach. Being
  synchronous and internally compensated also dropped D2, C35-C38 and R10.
  Inductor stays the fleet 2.2 uH: inside TI's 0.37-2.9 uH range and the
  only value meeting their ripple-under-40%-of-average guidance at load.

- Keystone 1043P holder -> MYOUNG BH-18650-A5BJ001-2D. Terminal pitch
  72.30 vs 72.22 mm, so the battery nets did not move; BT2 is rotated 180
  degrees because this part's positive end is mirrored.

Across all four boards:

- Every crystal was mis-loaded. 32.768 kHz parts saw ~9 pF against a 6 pF
  spec and the 40 MHz saw 12.5 pF against 10 pF, both pulling slow. Moved
  to Seiko SC-32S (12.5 pF) with 22 pF load caps, and the 40 MHz caps to
  18 pF. The tolerance being paid for had been swamped several times over.

- Capacitor voltage audit, new Min V rating column in the BOM. Three parts
  were operating outside their rating on 8.4 V rails: 47 uF and 100 u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
Connections:
- net Vcc renamed CHG_VCC
Changed lines of the file:
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@@
 		)
 	)
-	(global_label "Vcc"
+	(global_label "CHG_VCC"
 		(shape input)
 		(at 100.965 83.82 90)
@@
 		)
 	)
-	(global_label "Vcc"
+	(global_label "CHG_VCC"
 		(shape input)
 		(at 212.725 97.155 90)
@@
 		)
 	)
-	(global_label "Vcc"
+	(global_label "CHG_VCC"
 		(shape input)
 		(at 98.425 105.41 90)
@@
 		)
 	)
-	(global_label "Vcc"
+	(global_label "CHG_VCC"
 		(shape input)
 		(at 125.73 114.3 90)

Commit message: hardware: MPN + Mfr on every purchased part of the three ESP32 boards
Closes the LoRa pre-fab review's finding 3, extended to the sibling boards.
Every non-DNP symbol now names the exact part the cross-board BOM prices, so
the schematic can no longer imply a part that was never quoted.

401 of 401 purchasable parts carry an MPN. The only exemptions are the three
DNP v3.x provisions on the rocket-computer (R74/R75 499 k, R76 0 R): not
fitted, so never purchased, so correctly absent from the BOM.

Values normalised so each part resolves to one BOM line:

  LoRa R74  "10 K" -> "10 k"   capital K split one part across two lines
  LoRa D6   "LED"  -> "Green"  no colour recorded, so no MPN could attach
  Y1/Y3/Y5  "SC-32S-32.768kHz-12.5pF" -> "ABS07-32.768KHZ-T"

Two stale legacy MP fields disagreed with both the Value and the BOM and were
corrected -- a symbol carrying two part numbers is the wrong-part-order hazard
this pass exists to remove:

  rocket U19  TPS259824LNRGER -> ...RGET.  Same die and RGE-24 package; the
              suffix is reel quantity, and power-eco.md documents RGET.
  base   U9   TPS63021DSJR -> TPS63020DSJR.  These are NOT interchangeable:
              63021 is fixed 3.3 V, 63020 is adjustable. U9 pin 3 (FB) drives
              a real divider (R13 1 M / R16 180 k -> 0.5 x (1 + 1M/180k) =
              3.28 V), which only the adjustable part uses. BOM was right.

The ABS07 keeps the existing XTAL_SC-32S_3215 footprint: both parts are
2-pad 3.2 x 1.5 mm tuning forks, so the land is correct and only the
footprint's name now reads for the superseded vendor.

ERC clean on all three boards after the pass.

Co-Authored-By: Claude Opus 5 <noreply@anthropic.com>
Parts:
- C48, C53, C54: MPN (none) -> CL21A226MOQNNNE; Mfr (none) -> Samsung
- C51: MPN (none) -> CL05A105KO5NNNC; Mfr (none) -> Samsung
- C52, C55, C56: MPN (none) -> CL05B104KO5NNNC; Mfr (none) -> Samsung
- D7: MPN (none) -> WP710A10YD; Mfr (none) -> Kingbright
- D8: MPN (none) -> APHHS1005QBC/D; Mfr (none) -> Kingbright
- J4: MPN (none) -> S3B-XH-A; Mfr (none) -> JST
- L6: MPN (none) -> SRP4020TA-1R5M; Mfr (none) -> Bourns
- R36: MPN (none) -> RC0402FR-075K49L; Mfr (none) -> Yageo
- R37: MPN (none) -> RC0402FR-072KL; Mfr (none) -> Yageo
- R38: MPN (none) -> RC0402FR-07150RL; Mfr (none) -> Yageo
- R39: MPN (none) -> RC0402FR-071KL; Mfr (none) -> Yageo
- R40: MPN (none) -> RC0402FR-07300KL; Mfr (none) -> Yageo
- R42, R48, R49, R50, R51: MPN (none) -> RC0402FR-07100KL; Mfr (none) -> Yageo
- R43: MPN (none) -> RC0402FR-076K04L; Mfr (none) -> Yageo
- R45, R47: MPN (none) -> RC0805FR-0760R4L; Mfr (none) -> Yageo
- U12: MPN (none) -> MP2672AGD-0000-Z; Mfr (none) -> MPS
