File: hardware/base-station/power.kicad_sch (KiCad schematic)
At the start: 25 parts, among them U2 TPS61023DRLR, U22 TPS22918DBVR, U9 TPS63020DSJR

Commit message: hardware: MPN + Mfr on every purchased part of the three ESP32 boards
Closes the LoRa pre-fab review's finding 3, extended to the sibling boards.
Every non-DNP symbol now names the exact part the cross-board BOM prices, so
the schematic can no longer imply a part that was never quoted.

401 of 401 purchasable parts carry an MPN. The only exemptions are the three
DNP v3.x provisions on the rocket-computer (R74/R75 499 k, R76 0 R): not
fitted, so never purchased, so correctly absent from the BOM.

Values normalised so each part resolves to one BOM line:

  LoRa R74  "10 K" -> "10 k"   capital K split one part across two lines
  LoRa D6   "LED"  -> "Green"  no colour recorded, so no MPN could attach
  Y1/Y3/Y5  "SC-32S-32.768kHz-12.5pF" -> "ABS07-32.768KHZ-T"

Two stale legacy MP fields disagreed with both the Value and the BOM and were
corrected -- a symbol carrying two part numbers is the wrong-part-order hazard
this pass exists to remove:

  rocket U19  TPS259824LNRGER -> ...RGET.  Same die and RGE-24 package; the
              suffix is reel quantity, and power-eco.md documents RGET.
  base   U9   TPS63021DSJR -> TPS63020DSJR.  These are NOT interchangeable:
              63021 is fixed 3.3 V, 63020 is adjustable. U9 pin 3 (FB) drives
              a real divider (R13 1 M / R16 180 k -> 0.5 x (1 + 1M/180k) =
              3.28 V), which only the adjustable part uses. BOM was right.

The ABS07 keeps the existing XTAL_SC-32S_3215 footprint: both parts are
2-pad 3.2 x 1.5 mm tuning forks, so the land is correct and only the
footprint's name now reads for the superseded vendor.

ERC clean on all three boards after the pass.

Co-Authored-By: Claude Opus 5 <noreply@anthropic.com>
Parts:
- C21: MPN (none) -> CL05B103KB5NNNC; Mfr (none) -> Samsung
- C23, C29: MPN (none) -> CL05B104KO5NNNC; Mfr (none) -> Samsung
- C34, C40, C58, C59, C60, C61, C62: MPN (none) -> CL21A226MOQNNNE; Mfr (none) -> Samsung
- C42: MPN (none) -> CL05A105KO5NNNC; Mfr (none) -> Samsung
- C88: MPN (none) -> CC0402KRX7R9BB222; Mfr (none) -> Yageo
- D6: MPN (none) -> WP710A10GD; Mfr (none) -> Kingbright
- L8, L9: MPN (none) -> VLS3012CX-2R2M-1; Mfr (none) -> TDK
- R11: MPN (none) -> RC0402FR-07732KL; Mfr (none) -> Yageo
- R12, R7: MPN (none) -> RC0402FR-07100KL; Mfr (none) -> Yageo
- R13: MPN (none) -> RC0402FR-071ML; Mfr (none) -> Yageo
- R16: MPN (none) -> RC0402FR-07180KL; Mfr (none) -> Yageo
- R54: MPN (none) -> RC0402FR-07150RL; Mfr (none) -> Yageo
- S1: MPN (none) -> PB400EEQR1BLK; Mfr (none) -> E-Switch
- U2: MPN (none) -> TPS61023DRLR; Mfr (none) -> Texas Instruments
- U22: MPN (none) -> TPS22918DBVR; Mfr (none) -> TI
- U9: MP TPS63021DSJR -> TPS63020DSJR; MPN (none) -> TPS63020DSJR; Mfr (none) -> TI

Commit message: hardware(base-station): power-switch review fixes -- MID balance resistors to 1206
Schematic-side only; the PCB has not caught up. Do not fabricate from this
revision.

Review of the base-station power switching (schematic only, this session).
The V5 defect is fixed in this revision: the V_LORA boost is now behind the
TPS22918 load switch, so S1 kills the LoRa daughterboard along with everything
else. Standby with S1 open measures out at ~6 uA typical (DW01A + the 1M/1M
sense divider + leakages), and both chargers stay upstream and fully
functional.

R45/R47 (MP2672A MID cell-balance) 0805 -> 1206, 0.75 W:
  RC0805FR-0760R4L (Yageo, 0.125 W) -> CRCW120660R4FKEAHP (Vishay, 0.75 W)

The pair is 2x 60.4 R in parallel = 30.2 R in the MID balance path. With
R_ON_BHS = 2.1 R (datasheet p9) and the high cell at 4.2 V, balance current is
4.2/32.3 = 130 mA, so each resistor carries 65 mA and burns 65mA^2 * 60.4 =
0.255 W. Balancing runs 249.8 ms of every 250 ms cycle (Figure 13, p24) -- so
that is continuous, not a pulse. The 0805 parts were at 204% of rating; even a
standard 0.25 W 1206 sits at 102%. The Vishay HP part is 0.75 W, i.e. 34%
loaded. Balance current is deliberately unchanged -- this is a power-rating
fix, not a re-tune. Value stays 60.4 R and MPS characterizes the part at
~17 R (p19), so 30.2 R is already the conservative side.

Metadata lockstep on three parts whose values moved but whose MPN fields did
not follow (all caught by the exact MPN-keyed BOM audit):
  R43 10 k    -> RC0402FR-0710KL   (was still the 6.04 k P/N)
  C42 10 uF   -> CL05A106MQ5NUNC   (was still the 1 uF P/N)
  R53 210 k   -> RC0402FR-07210KL  (copy-pasted from R52, kept its 675 R P/N)

R53 is the BQ21040 TS fail-safe: a floating TS does not suspend charging, it
enters TTDM (datasheet 8.4.6), which charges the cell with NTC monitoring,
termination and the 10-hour safety timer all disabled. 210 k holds TS in the
cold-fault window instead. Picked over the datasheet's 237 k because 237 k x
6.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
Parts:
- C42: value 1 uF -> 10 uF; MPN CL05A105KO5NNNC -> CL05A106MQ5NUNC
Connections:
- net V_SWITCH: now also C29.1, U9.1 (VINA), U9.12 (EN)
Changed lines of the file:
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@@
 	)
 	(junction
+		(at 142.875 43.18)
+		(diameter 0)
+		(color 0 0 0 0)
+	)
+	(junction
 		(at 209.55 44.45)
 		(diameter 0)
@@
 	)
 	(junction
+		(at 142.875 50.8)
+		(diameter 0)
+		(color 0 0 0 0)
+	)
+	(junction
 		(at 233.68 44.45)
 		(diameter 0)
@@
 	(wire
 		(pts
-			(xy 135.89 43.18) (xy 154.305 43.18)
+			(xy 135.89 43.18) (xy 142.875 43.18)
 		)
 		(stroke
@@
 	(wire
 		(pts
+			(xy 142.875 43.18) (xy 154.305 43.18)
+		)
+		(stroke
+			(width 0)
+			(type default)
+		)
+	)
+	(wire
+		(pts
 			(xy 196.85 78.105) (xy 200.025 78.105)
 		)
@@
 	(wire
 		(pts
+			(xy 142.875 43.18) (xy 142.875 50.8)
+		)
+		(stroke
+			(width 0)
+			(type default)
+		)
+	)
+	(wire
+		(pts
 			(xy 25.4 82.55) (xy 27.94 82.55)
 		)
@@
 			)
 		)
-		(property "Value" "1 uF"
+		(property "Value" "10 uF"
 			(at 48.26 48.26 0)
 			(show_name no)
@@
 			)
 		)
-		(property "MPN" "CL05A105KO5NNNC"
+		(property "MPN" "CL05A106MQ5NUNC"
 			(at 48.26 45.72 0)
 			(hide yes)

Commit message: hardware(base-station): pre-fab fixes -- JLC stackup, RF feed, R17/R18, EN margin
The board changes the 2026-08-02 pre-manufacturing review called for. Board is
DRC-clean: 0 errors, 0 unconnected items, 0 schematic-parity issues.

Electrical:
- R17 10 k -> 18.7 k and R18 1 k, both with MPNs that match their values. Both
  previously carried RC0402FR-075K11L (5.11 k). Built to that MPN the TPS61023
  EN pin would sit at 1.65 V driven low, above the 1.2 V V_EN_H ceiling, and the
  LoRa power-cycle recovery would never work with no symptom. 18.7 k/1 k gives
  0.174 V against the 0.35 V guaranteed-low floor, and is already a fleet MPN so
  it adds no BOM line.
- Antenna matching reduced to Molex section 6.0: L4 4.3 nH shunt alone, with
  C2 = 0 ohm realised as a direct trace. C25/C26/L7 removed. The previous
  four-element network put 4.3 nH in parallel with 1.5 pF, which is -j127.8 ohm
  at 2.44 GHz where the Molex reference is +j65.9 ohm -- a sign inversion, not a
  value shift. Accepted trade: this build has no tuning provision, so it must be
  characterised with the cell installed and the result carried into the next
  revision.
- U15 fixing pads 1-3 left individually unconnected. AS-479480001 calls them
  fixing pads and never specifies their net; grounding them is an unforced risk
  on an LDS part whose plating wraps the body.

Stackup and rules, now JLCPCB standard 4-layer:
- JLC04161H-7628: 0.2104 mm 7628 prepreg (Er 4.4), 0.5 oz inner copper, 1.065 mm
  core, ENIG, 1.5862 mm. The previous 0.1 mm prepreg and 1 oz inner layers were
  not a stackup any standard 4-layer order builds.
- RF feed re-solved for the new dielectric: 0.20 -> 0.36 mm, giving 49.7 ohm as
  CPWG at the 0.15 mm pour gap. At 0.20 mm on the new stackup it would have been
  ~68 ohm. New RF netclass carries the width and clearance.
- min_clearance 0.09 -> 0.10 (0.09 falls in the JLC 3.0-3.5 mil upcharge band),
  min_via_diameter 0.40 -> 0.45, annular 0.05 -> 0.075, drill 0.1 -> 0.3, silk
  text 0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
Parts:
- added C41: 22 uF, Capacitor_SMD:C_0805_2012Metric, symbol Device:C
- added R17: 18.7 k, Resistor_SMD:R_0402_1005Metric, symbol Device:R_US
- added R18: 1 k, Resistor_SMD:R_0402_1005Metric, symbol Device:R_US
- C42: value 10 uF -> 22 uF; footprint Capacitor_SMD:C_0402_1005Metric -> Capacitor_SMD:C_0805_2012Metric; MPN CL05A106MQ5NUNC -> CL21A226MOQNNNE
Connections:
- net +3V3: now also R17.2
- net GND: now also C41.2
- net V_LORA: now also C41.1
- net V_SWITCH: no longer U2.2 (EN)
- new net: R17.1, R18.1, U2.2 (EN)
- new net LoRa_EN: R18.2
Other:
- moved on the sheet: C34

Commit message: hardware: consolidate five resistor lines onto fleet values (rocket, base-station)
Cross-board BOM line reduction; netlist-verified functions, no ratio-
critical or safety-analyzed parts touched:

- rocket R3 10R -> 22R: FSUSB63 VCC supply filter, uA load; 22R is a
  three-board fleet line, retires the 10R line
- rocket R85 2.2k -> 2k: TPS22811 CAM_IMON gain load; joins the base's
  2k line, retires 2.2k. FIRMWARE: IMON scale changes by x0.909
- base R17 18.7k -> 100k: TPS61023 EN pull-up, value non-critical;
  retires the fleet's last 18.7k line
- base R40/R42 300k/100k -> 1M/180k: battery ADC divider re-ratioed
  onto fleet values (8.4V -> 1.281V at GPIO8, was 2.1V; source
  impedance 152k against the 100nF reservoir C55, pack drain drops
  21uA -> 7uA). FIRMWARE: scale constant 4.000 -> 6.5556; retires 300k
- PCB field sync included (R85's board-side MPN still carried the
  pre-fix 3.3k code; now consistent both sides)

Deliberately NOT consolidated after review: U9 stays CSD16323Q3 (pyro
arm FET -- WORKLIST H-2 glitch-margin analysis is against this part's
threshold; H-9 fire-return layout built into its drain pad); base L6
stays SRP4020TA-1R5M (it is the MP2672 switching inductor, not a
filter -- a VLS3012 would saturate).

ERC profiles unchanged both boards; DRC error-severity: base clean,
rocket = the three accepted courtyard overlaps. bom.csv regenerated.

Co-Authored-By: Claude Fable 5 <noreply@anthropic.com>
Parts:
- R17: value 18.7 k -> 100 k; MPN RC0402FR-0718K7L -> RC0402FR-07100KL
Changed lines of the file:
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@@
 			)
 		)
-		(property "Value" "18.7 k"
+		(property "Value" "100 k"
 			(at 69.215 130.81 90)
 			(show_name no)
@@
 			)
 		)
-		(property "MPN" "RC0402FR-0718K7L"
+		(property "MPN" "RC0402FR-07100KL"
 			(at 71.755 130.81 0)
 			(hide yes)

Commit message: hardware: base-station to fixed-output TPS63021, rev V6
U9 was three parts at once: a TPS63021 symbol and footprint, TPS63020 in its
Value/MPN/MP fields, and the adjustable part's feedback divider in the wiring.
The BOM generates from Value, so the board ordered a 63020 while the schematic
said 63021.

Settled on the fixed-output 63021: R13 (1M), R16 (180k), the divider's GND
symbol and its stub wire are gone, and FB now ties directly to the +3V3 rail as
the fixed part requires. That divider is correct for a 63020 and destructive on
a 63021 -- feeding FB 0.152x VOUT drives the loop toward ~21 V until OVP.

Copper changed, so major per docs/board-versioning.md: title block V5 -> V6.
Tag base-station-v6.0.0 at fab release, not here -- the release procedure tags
after DRC clears and gerbers plot.

bom.csv regenerated: R13 out of the 1M group (4->3), R16 out of the 180k group
(2->1), U9 now TPS63021DSJR. References kept expanded; kicad-cli 10.0.3 collapses
them to ranges, which is not this repo's committed style.

Verified: +3V3 and GND remain separate nets with no overlapping nodes. Deleting
a symbol leaves its wires behind, so that was the check that mattered.

THE PCB IS NOT YET SYNCED. Five schematic-parity items are outstanding -- U9's
value and MP field, pad 3's net, and the R13/R16 footprints -- all resolved by
one Update PCB from Schematic plus a short FB trace. 0 unconnected, 36 DRC, all
silkscreen.

Also annotates the 2026-08-02 review header. It states the stackup as found at
the start of that review (KiCad's untouched 4-layer default) and reads as current
truth out of context; the review's own S7 replaced it with JLCPCB JLC04161H-7628.

Co-Authored-By: Claude Opus 5 <noreply@anthropic.com>
Parts:
- removed R13: 1 M, Resistor_SMD:R_0402_1005Metric, symbol Device:R_US
- removed R16: 180 k, Resistor_SMD:R_0402_1005Metric, symbol Device:R_US
- U9: value TPS63020DSJR -> TPS63021DSJR; MP TPS63020DSJR -> TPS63021DSJR; MPN TPS63020DSJR -> TPS63021DSJR
Connections:
- net +3V3: now also U9.3 (FB)
