File: hardware/lora-daughterboard/lora-daughterboard.kicad_sch (KiCad schematic)
At the start: 74 parts, among them J2 USB4110GFA, J6 Conn_01x04, J8 CON-SMA-EDGE-S, U14 E220-900MM22S, U22 W25Q128JVSIQ, U28 ESP32-S3RH2, U3 TPS62913RPUR, Y5 SC-32S-32.768kHz-12.5pF, Y6 ECS-400-10-37B2-CKY-TR

Commit message: hardware: MPN + Mfr on every purchased part of the three ESP32 boards
Closes the LoRa pre-fab review's finding 3, extended to the sibling boards.
Every non-DNP symbol now names the exact part the cross-board BOM prices, so
the schematic can no longer imply a part that was never quoted.

401 of 401 purchasable parts carry an MPN. The only exemptions are the three
DNP v3.x provisions on the rocket-computer (R74/R75 499 k, R76 0 R): not
fitted, so never purchased, so correctly absent from the BOM.

Values normalised so each part resolves to one BOM line:

  LoRa R74  "10 K" -> "10 k"   capital K split one part across two lines
  LoRa D6   "LED"  -> "Green"  no colour recorded, so no MPN could attach
  Y1/Y3/Y5  "SC-32S-32.768kHz-12.5pF" -> "ABS07-32.768KHZ-T"

Two stale legacy MP fields disagreed with both the Value and the BOM and were
corrected -- a symbol carrying two part numbers is the wrong-part-order hazard
this pass exists to remove:

  rocket U19  TPS259824LNRGER -> ...RGET.  Same die and RGE-24 package; the
              suffix is reel quantity, and power-eco.md documents RGET.
  base   U9   TPS63021DSJR -> TPS63020DSJR.  These are NOT interchangeable:
              63021 is fixed 3.3 V, 63020 is adjustable. U9 pin 3 (FB) drives
              a real divider (R13 1 M / R16 180 k -> 0.5 x (1 + 1M/180k) =
              3.28 V), which only the adjustable part uses. BOM was right.

The ABS07 keeps the existing XTAL_SC-32S_3215 footprint: both parts are
2-pad 3.2 x 1.5 mm tuning forks, so the land is correct and only the
footprint's name now reads for the superseded vendor.

ERC clean on all three boards after the pass.

Co-Authored-By: Claude Opus 5 <noreply@anthropic.com>
Parts:
- C96: MPN CL05A105KO5NNNC -> CL05A106MQ5NUNC
- CR1, CR3: MPN (none) -> CUS10S30,H3F; Mfr (none) -> Toshiba
- CR2: MPN (none) -> SP0503BAHTG; Mfr (none) -> Littelfuse
- D4: MPN (none) -> APHHS1005QBC/D; Mfr (none) -> Kingbright
- D5: MPN (none) -> NCD0402R1; Mfr (none) -> NationStar
- D6: value LED -> Green; MPN (none) -> XL-1005UGC; Mfr (none) -> Xinglight
- FB1: MPN (none) -> 782853200; Mfr (none) -> Wurth
- FL1: MPN (none) -> DLW21SN670HQ2L; Mfr (none) -> Murata
- H1, H2, H3, H4: symbol Mechanical:MountingHole -> Mechanical:MountingHole_Pad
- J2: MPN (none) -> USB4110-GF-A; Mfr (none) -> GCT
- J6: MPN (none) -> BM04B-SRSS-TB; Mfr (none) -> JST
- J8: MPN (none) -> CON-SMA-EDGE-S; Mfr (none) -> generic
- L10: MPN (none) -> LQW15AN24NH00D; Mfr (none) -> Murata
- L11: MPN (none) -> LQG15HS2N0S02D; Mfr (none) -> Murata
- L8: MPN (none) -> VLS3012CX-2R2M-1; Mfr (none) -> TDK
- R1, R5: MPN (none) -> RC0402FR-075K11L; Mfr (none) -> Yageo
- R3, R4, R59, R60, R73: MPN (none) -> RC0402FR-0710KL; Mfr (none) -> Yageo
- R6: MPN (none) -> RC0402FR-0715K4L; Mfr (none) -> Yageo
- R7: MPN (none) -> RC0402FR-074K87L; Mfr (none) -> Yageo
- R74: value 10 K -> 10 k; MPN (none) -> RC0402FR-0710KL; Mfr (none) -> Yageo
- R75, R76: MPN (none) -> RC0402FR-0722RL; Mfr (none) -> Yageo
- R77, R78: MPN (none) -> RC0402FR-071KL; Mfr (none) -> Yageo
- R8: MPN (none) -> RC0402FR-077K5L; Mfr (none) -> Yageo
- S3: MPN (none) -> KMR221GLFS; Mfr (none) -> C&K
- U14: MPN (none) -> E220-900MM22S; Mfr (none) -> Ebyte
- U22: MPN (none) -> W25Q128JVSIQ; Mfr (none) -> Winbond
- U28: MPN (none) -> ESP32-S3RH2; Mfr (none) -> Espressif
- U3: MPN (none) -> TPS62913RPUR; Mfr (none) -> TI
- Y5: value SC-32S-32.768kHz-12.5pF -> ABS07-32.768KHZ-T; MPN (none) -> ABS07-32.768KHZ-T; Mfr (none) -> Abracon
- Y6: MPN (none) -> ECS-400-10-37B2-CKY-TR; Mfr (none) -> ECS
Connections:
- net GND: now also H1.1, H2.1, H3.1, H4.1
