File: hardware/gnss-sam10m8-18mm-hv/gnss-sam10m8-18mm-hv.kicad_sch (KiCad schematic)
At the start: 29 parts, among them J3 BM05B-SRSS-TB, U1 SAM-M10Q-00B, U3 TPS62913RPUR

Commit message: hardware: BOM-cost pass across all four boards
Component changes from a cross-board cost review. Per-board component cost
(USD @~100qty): rocket $86.21 -> $61.39, base station $35.91 -> $29.89, with
the LoRa daughterboard and GNSS SAM-M10Q board added to the shared BOM.

Memory architecture
  - Rocket: MR25H10 MRAM deleted; the log ring moves to in-package PSRAM.
    ESP32-S3 -> ESP32-S3RH2 (2 MB quad PSRAM, no in-package flash, same land
    pattern; SPICS1/GPIO26 was already unconnected on every board).
    Persistence across boots is knowingly given up.
  - Rocket NAND F35SQB004G-WWT -> GD5F2GQ5UEYIGR: pin- and footprint-identical
    (verified against the U11 land pattern), 4 Gbit -> 2 Gbit, $11.61 -> $3.50.
    Needs the 4096 -> 2048 B page migration in firmware.
  - Base station: dedicated log flash deleted entirely. It wrote one ~183 B CSV
    row per received packet at the 2 Hz downlink (~366 B/s, and only while a
    flight is active), so 256 MB was ~204 hours of headroom. The firmware
    already falls back to the existing SPIFFS partition, so this promotes a
    tested path rather than needing new code.
  - Boot flash W25Q64JVXGIQ -> W25Q128JVSIQ on all four positions: 16 MB for
    LESS money ($3.10 -> $2.21). SCHEMATIC ONLY - the boards still need
    "Update PCB from Schematic" plus re-placement, since SOIC-8 208mil is 2.2x
    the DFN's area. The DFN's 9th (exposed) pad was a redundant GND tie; pin 4
    is GND on all four, so nothing is lost.

Power
  - LoRa + GNSS keep TPS62913 (low-noise, RF rails). The rocket briefly moved
    to it and was REVERTED to TPS62152: the TPS62913 is forced-PWM with 5 mA
    quiescent, which would have raised the pad-idle floor ~6x against the
    light-sleep work.
  - Base load switch TPS22810 -> TPS22918 (identical footprint and pin order;
    pin 3 EN/UVLO -> ON is safe because it was driven as a plain enable).
    CT cap 10 nF -> 2.2 nF to match the rocket's ramp; R8 (QOD->VOUT) deleted.
  - LoRa gains a 7.5k S-CONF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
Parts:
- removed L1: ASPI-0530HI-2R2M-T2, Footprints:IND_ASPI-0530HI-2R2M-T2, symbol Custom:ASPI-0530HI-2R2M-T2
- added L8: VLS3012CX-2R2M-1, Footprints:IND_VLS3012CX-2R2M-1, symbol Custom:VLS3012CX-2R2M-1
Connections:
- net GND: no longer U3.10 (S-CONF)
- net at C7.1, C8.1, C9.1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: now also U3.10 (S-CONF)
- net at C11.1, C13.1, FB1.1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: now also L8.2
- net at U3.2 (SW): now also L8.1

Commit message: hardware: battery protection, boost swap, and a capacitor voltage audit
Base station power chain, all verified against exported netlists:

- Protection: MAX17303G+ gauge/protector and its NTMD6N02R2G FET pair
  replaced by DW01A + 2x FS8205A. The MAX17303 had no firmware driver and
  the board never had a working coulomb counter, so state of charge already
  came from the voltage curve in bs_battery_soc.h; it now reads a 1M/1M
  divider on GPIO1. The FETs move from the positive rail to the negative
  one because the DW01A has no charge pump, so board ground is now P-,
  separated from the cell's B- by the FET stack. Two FS8205A in parallel
  put the 150 mV overcurrent trip at ~4.8-6.0 A instead of ~2.4-3.0 A.
  TH1 moves onto the BQ21040's TS pin, replacing a fixed 10k that had been
  defeating thermal charge cutoff.

- V_LORA retargeted 7.49 V -> 4.95 V and LM5157QRTERQ1 -> TPS61023DRLR.
  Nothing needed 7.4 V (everything downstream is 3.3 V behind the
  TPS62913), while an RFD868x-class radio is 5 V nominal with a 6 V
  absolute maximum, so the old rail put it permanently out of reach. Being
  synchronous and internally compensated also dropped D2, C35-C38 and R10.
  Inductor stays the fleet 2.2 uH: inside TI's 0.37-2.9 uH range and the
  only value meeting their ripple-under-40%-of-average guidance at load.

- Keystone 1043P holder -> MYOUNG BH-18650-A5BJ001-2D. Terminal pitch
  72.30 vs 72.22 mm, so the battery nets did not move; BT2 is rotated 180
  degrees because this part's positive end is mirrored.

Across all four boards:

- Every crystal was mis-loaded. 32.768 kHz parts saw ~9 pF against a 6 pF
  spec and the 40 MHz saw 12.5 pF against 10 pF, both pulling slow. Moved
  to Seiko SC-32S (12.5 pF) with 22 pF load caps, and the 40 MHz caps to
  18 pF. The tolerance being paid for had been swamped several times over.

- Capacitor voltage audit, new Min V rating column in the BOM. Three parts
  were operating outside their rating on 8.4 V rails: 47 uF and 100 u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
Parts:
- J3: footprint CONN_BM05B-SRSS-TB_JST -> Footprints:CONN_BM05B-SRSS-TB_JST
Changed lines of the file:
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@@
 			)
 		)
-		(property "Footprint" "CONN_BM05B-SRSS-TB_JST"
+		(property "Footprint" "Footprints:CONN_BM05B-SRSS-TB_JST"
 			(at 40.005 71.755 0)
 			(hide yes)

Commit message: hardware: WIP -- 1k series R on cross-board UARTs, BS LoRa boost behind the load switch
*** Schematic-side only. Two of the three boards' layouts have not caught
    up, and the rocket-computer PCB is still mid-rework. Do not fabricate
    from this revision. ***

Three review follow-ups, all schematic:

1. Camera UART series resistors (rocket-computer, external_connections)
   R30, R32 = 1 k 0402 inserted in the camera link:
     Camera_RX  U17.61 -> R30 -> J4.3
     Camera_TX  U17.60 -> R32 -> J4.4
   Mitigation for the V9 review's H6: the peripheral ports are ground-side
   switched while their supply pins stay live, so an off-state peripheral
   floats toward VBATT and injects into P4 GPIOs through the signal lines.
   H6's recommendation was ">= 1 k series resistors or bus switches on
   every cross-connector signal". PCB: R30/R32 ARE placed, F.Cu
   (97.31,156.38) and (97.31,158.38).

2. GNSS UART series resistors (gnss-sam10m8-18mm-hv)
   R7, R8 = 1 k 0402, same pattern:
     GNSS_RX  U1.14 -> R7 -> J3.1
     GNSS_TX  U1.13 -> R8 -> J3.2
   PCB: R7/R8 are NOT placed. Needs Update PCB from Schematic.

3. LoRa boost moved behind the load switch (base-station, power)
   U2 (TPS61023, the V_LORA boost) VIN+EN and its inductor L8 and C34 move
   from VCC to the new V_SWITCH net, downstream of U22 (TPS22918).
   Net-(U22-QOD) is renamed V_SWITCH and now carries
   {C23, C34, C59, L8.1, U2.2, U2.3, U22.5, U22.6, U9.10, U9.11}.
   This closes the LoRa V3 review's finding 14: previously the base
   station could not power-cycle the radio daughterboard, because the
   boost's EN was tied to VCC and a boost passes VIN through its body
   diode regardless. Switching the boost input makes a real power cycle
   possible. PCB: not updated -- the net change needs re-routing.

DRC as merged (kicad-cli, severity-error, with parity):
  gnss-sam10m8   0 violations, 0 unconnected  -- but R7/R8 absent from copper
  base-station  10 violations (all malformed_courtyard on U15), 0 un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
Parts:
- added R7, R8: 1 k, Resistor_SMD:R_0402_1005Metric, symbol Device:R_US
Connections:
- net GNSS_RX: now also R7.1; no longer J3.1
- net GNSS_TX: now also R8.1; no longer J3.2
- new net: J3.1, R7.2
- new net: J3.2, R8.2
Changed lines of the file:
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@@
 	(wire
 		(pts
+			(xy 40.005 78.105) (xy 36.195 78.105)
+		)
+		(stroke
+			(width 0)
+			(type default)
+		)
+	)
+	(wire
+		(pts
 			(xy 16.51 129.54) (xy 21.59 129.54)
 		)
@@
 	(wire
 		(pts
+			(xy 40.005 69.215) (xy 36.195 69.215)
+		)
+		(stroke
+			(width 0)
+			(type default)
+		)
+	)
+	(wire
+		(pts
 			(xy 153.67 142.24) (xy 153.67 145.415)
 		)
@@
 	(wire
 		(pts
+			(xy 40.005 71.755) (xy 40.005 78.105)
+		)
+		(stroke
+			(width 0)
+			(type default)
+		)
+	)
+	(wire
+		(pts
 			(xy 159.385 130.81) (xy 171.45 130.81)
 		)
@@
 	(wire
 		(pts
+			(xy 36.195 69.215) (xy 36.195 70.485)
+		)
+		(stroke
+			(width 0)
+			(type default)
+		)
+	)
+	(wire
+		(pts
 			(xy 121.92 134.62) (xy 146.685 134.62)
 		)
@@
 	(global_label "GNSS_RX"
 		(shape input)
-		(at 40.005 71.755 180)
+		(at 28.575 78.105 180)
 		(fields_autoplaced yes)
 		(effects
@@
 		)
 		(property "Intersheetrefs" "${INTERSHEET_REFS}"
-			(at 28.5532 71.755 0)
+			(at 17.1232 78.105 0)
 			(hide yes)
 			(show_name no)
@@
 	(global_label "GNSS_TX"
 		(shape input)
-		(at 40.005 69.215 180)
+		(at 28.575 70.485 180)
 		(fields_autoplaced yes)
 		(effects
@@
 		)
 		(property "Intersheetrefs" "${INTERSHEET_REFS}"
-			(at 28.8556 69.215 0)
+			(at 17.4256 70.485 0)
 			(hide yes)
 			(show_name no)
@@
 	)
 	(symbol
+		(lib_id "Device:R_US")
+		(at 32.385 78.105 90)
+		(unit 1)
+		(body_style 1)
+		(exclude_from_sim no)
+		(in_bom yes)
+		(on_board yes)
+		(in_pos_files yes)
+		(dnp no)
+		(property "Reference" "R7"
+			(at 32.385 75.565 90)
+			(show_name no)
+			(do_not_autoplace no)
+			(effects
+				(font
+					(size 1.27 1.27)
+				)
+			)
+		)
+		(property "Value" "1 k"
+			(at 32.385 80.645 90)
+			(show_name no)
+			(do_not_autoplace no)
+			(effects
+				(font
+					(size 1.27 1.27)
+				)
+			)
+		)
+		(property "Footprint" "Resistor_SMD:R_0402_1005Metric"
+			(at 32.639 77.089 90)
+			(hide yes)
+			(show_name no)
+			(do_not_autoplace no)
+			(effects
+				(font
+					(size 1.27 1.27)
+				)
+			)
+		)
+		(property "Datasheet" ""
+			(at 32.385 78.105 0)
+			(hide yes)
+			(show_name no)
+			(do_not_autoplace no)
+			(effects
+				(font
+					(size 1.27 1.27)
+				)
+			)
+		)
+		(property "Description" "Resistor, US symbol"
+			(at 32.385 78.105 0)
+			(hide yes)
+			(show_name no)
+			(do_not_autoplace no)
+			(effects
+				(font
+					(size 1.27 1.27)
+				)
+			)
+		)
+		(pin "1"
+		)
+		(pin "2"
+		)
+		(instances
+			(project "gnss-sam10m8-18mm-hv"
+				(path "/a61d9c6a-d8dd-4945-858b-535894b4ed8b"
+					(reference "R7")
+					(unit 1)
+				)
+			)
+		)
+	)
+	(symbol
 		(lib_id "Custom:WE-CBA_0805")
 		(at 199.39 130.81 0)
@@
 					(unit 1)
 				)
+			)
+		)
+	)
+	(symbol
+		(lib_id "Device:R_US")
+		(at 32.385 70.485 90)
+		(unit 1)
+		(body_style 1)
+		(exclude_from_sim no)
+		(in_bom yes)
+		(on_board yes)
+		(in_pos_files yes)
+		(dnp no)
+		(property "Reference" "R8"
+			(at 32.385 67.945 90)
+			(show_name no)
+			(do_not_autoplace no)
+			(effects
+				(font
+					(size 1.27 1.27)
+				)
+			)
+		)
+		(property "Value" "1 k"
+			(at 32.385 73.025 90)
+			(show_name no)
+			(do_not_autoplace no)
+			(effects
+				(font
+					(size 1.27 1.27)
+				)
+			)
+		)
+		(property "Footprint" "Resistor_SMD:R_0402_1005Metric"
+			(at 32.639 69.469 90)
+			(hide yes)
+			(show_name no)
+			(do_not_autoplace no)
+			(effects
+				(font
+					(size 1.27 1.27)
+				)
+			)
+		)
+		(property "Datasheet" ""
+			(at 32.385 70.485 0)
+			(hide yes)
+			(show_name no)
+			(do_not_autoplace no)
+			(effects
+				(font
+					(size 1.27 1.27)
+				)
+			)
+		)
+		(property "Description" "Resistor, US symbol"
+			(at 32.385 70.485 0)
+			(hide yes)
+			(show_name no)
+			(do_not_autoplace no)
+			(effects
+				(font
+					(size 1.27 1.27)
+				)
+			)
+		)
+		(pin "1"
+		)
+		(pin "2"
+		)
+		(instances
+			(project "gnss-sam10m8-18mm-hv"
+				(path "/a61d9c6a-d8dd-4945-858b-535894b4ed8b"
+					(reference "R8")
+					(unit 1)
+				)

Commit message: hardware: declare filled+capped vias on the 6-layer boards; in-progress board edits
Two separate things, kept together because they land in the same board files.

1. Via protection, mine.  lora-daughterboard and rocket-computer both place
   vias in pads, and the fab fills those on 6-layer stackups -- but the board
   files still declared (filling no) (capping no), so nothing in the exported
   data said so.  Both now declare IPC-4761 Type VII (filled and capped),
   which is the process via-in-pad actually requires.  base-station is left at
   (filling no) (capping no): it is 4-layer and does not get the treatment.

2. In-progress layout work, the user's, carried along in the same files:

   rocket-computer  J7 removed (superseded by the J8 JST VH battery inlet);
                    C20/C22/C48/C49 crystal caps 18 pF -> 12 pF now reflected
                    in copper; 8 parts flipped side, 23 repositioned, routing
                    and via count adjusted to suit
   lora-daughterboard  routing and ground stitching (+8 vias, +10 segments)
   base-station     one via removed
   gnss-sam10m8-18mm-hv       C15 added; C11/C13 47 uF -> 22 uF
   gnss-px1105r-...-ext-ant   C16/R8/R9 added; C13/C14 47 uF -> 22 uF

The 47 -> 22 uF swap on both GNSS boards is already reflected in the
cross-board BOM: the 47 uF line is now rocket-computer only (1), and 22 uF
GNSS went 5 -> 8.

Co-Authored-By: Claude Opus 5 <noreply@anthropic.com>
Parts:
- added C15: 22 uF, Capacitor_SMD:C_0805_2012Metric, symbol Device:C
- C11, C13: value 47 uF -> 22 uF
Connections:
- net GND: now also C15.2
- net at C11.1, C13.1, FB1.1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: now also C15.1
Changed lines of the file:
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@@
 	)
 	(junction
+		(at 183.515 130.81)
+		(diameter 0)
+		(color 0 0 0 0)
+	)
+	(junction
 		(at 161.925 91.44)
 		(diameter 0)
@@
 	(wire
 		(pts
+			(xy 183.515 130.81) (xy 191.77 130.81)
+		)
+		(stroke
+			(width 0)
+			(type default)
+		)
+	)
+	(wire
+		(pts
 			(xy 161.925 31.115) (xy 167.64 31.115)
 		)
@@
 	(wire
 		(pts
-			(xy 171.45 130.81) (xy 191.77 130.81)
+			(xy 171.45 130.81) (xy 183.515 130.81)
 		)
 		(stroke
@@
 	)
 	(symbol
+		(lib_id "power:GND")
+		(at 183.515 138.43 0)
+		(unit 1)
+		(body_style 1)
+		(exclude_from_sim no)
+		(in_bom yes)
+		(on_board yes)
+		(in_pos_files yes)
+		(dnp no)
+		(fields_autoplaced yes)
+		(property "Reference" "#PWR018"
+			(at 183.515 144.78 0)
+			(hide yes)
+			(show_name no)
+			(do_not_autoplace no)
+			(effects
+				(font
+					(size 1.27 1.27)
+				)
+			)
+		)
+		(property "Value" "GND"
+			(at 183.515 142.875 0)
+			(show_name no)
+			(do_not_autoplace no)
+			(effects
+				(font
+					(size 1.27 1.27)
+				)
+			)
+		)
+		(property "Footprint" ""
+			(at 183.515 138.43 0)
+			(hide yes)
+			(show_name no)
+			(do_not_autoplace no)
+			(effects
+				(font
+					(size 1.27 1.27)
+				)
+			)
+		)
+		(property "Datasheet" ""
+			(at 183.515 138.43 0)
+			(hide yes)
+			(show_name no)
+			(do_not_autoplace no)
+			(effects
+				(font
+					(size 1.27 1.27)
+				)
+			)
+		)
+		(property "Description" "Power symbol creates a global label with name \"GND\" , ground"
+			(at 183.515 138.43 0)
+			(hide yes)
+			(show_name no)
+			(do_not_autoplace no)
+			(effects
+				(font
+					(size 1.27 1.27)
+				)
+			)
+		)
+		(pin "1"
+		)
+		(instances
+			(project "gnss-sam10m8-18mm-hv"
+				(path "/a61d9c6a-d8dd-4945-858b-535894b4ed8b"
+					(reference "#PWR018")
+					(unit 1)
+				)
+			)
+		)
+	)
+	(symbol
 		(lib_id "Mechanical:MountingHole")
 		(at 139.7 193.04 0)
@@
 	(symbol
 		(lib_id "Device:C")
+		(at 183.515 134.62 0)
+		(unit 1)
+		(body_style 1)
+		(exclude_from_sim no)
+		(in_bom yes)
+		(on_board yes)
+		(in_pos_files yes)
+		(dnp no)
+		(fields_autoplaced yes)
+		(property "Reference" "C15"
+			(at 187.325 133.3499 0)
+			(show_name no)
+			(do_not_autoplace no)
+			(effects
+				(font
+					(size 1.27 1.27)
+				)
+				(justify left)
+			)
+		)
+		(property "Value" "22 uF"
+			(at 187.325 135.8899 0)
+			(show_name no)
+			(do_not_autoplace no)
+			(effects
+				(font
+					(size 1.27 1.27)
+				)
+				(justify left)
+			)
+		)
+		(property "Footprint" "Capacitor_SMD:C_0805_2012Metric"
+			(at 184.4802 138.43 0)
+			(hide yes)
+			(show_name no)
+			(do_not_autoplace no)
+			(effects
+				(font
+					(size 1.27 1.27)
+				)
+			)
+		)
+		(property "Datasheet" ""
+			(at 183.515 134.62 0)
+			(hide yes)
+			(show_name no)
+			(do_not_autoplace no)
+			(effects
+				(font
+					(size 1.27 1.27)
+				)
+			)
+		)
+		(property "Description" "Unpolarized capacitor"
+			(at 183.515 134.62 0)
+			(hide yes)
+			(show_name no)
+			(do_not_autoplace no)
+			(effects
+				(font
+					(size 1.27 1.27)
+				)
+			)
+		)
+		(pin "1"
+		)
+		(pin "2"
+		)
+		(instances
+			(project "gnss-sam10m8-18mm-hv"
+				(path "/a61d9c6a-d8dd-4945-858b-535894b4ed8b"
+					(reference "C15")
+					(unit 1)
+				)
+			)
+		)
+	)
+	(symbol
+		(lib_id "Device:C")
 		(at 180.34 34.925 0)
 		(unit 1)
@@
 			)
 		)
-		(property "Value" "47 uF"
+		(property "Value" "22 uF"
 			(at 163.195 135.8899 0)
 			(show_name no)
@@
 			)
 		)
-		(property "Value" "47 uF"
+		(property "Value" "22 uF"
 			(at 175.26 135.8899 0)
 			(show_name no)

Commit message: hardware(gnss-sam10m8): D1/D3 colour was never recorded -- set to Green
Both LEDs carried the bare placeholder value "LED", the same gap that left the
LoRa board's D6 without a colour and therefore without a buyable part. D1 is
the timepulse indicator (U1.7 TIMEPULSE -> R1 -> D1 -> GND) and D3 the power
indicator (+3V3 -> R3 -> D3 -> GND).

Green is not a new decision: the cross-board BOM already prices 2 x
XL-1005UGC against the GNSS column. The board simply never said so, which is
how two LEDs of unspecified colour were about to go to fab alongside a BOM
buying green ones.

This was the last disagreement between the boards and the BOM. All four costed
boards now reconcile exactly: 427 fitted parts, 0 quantity mismatches, 0 parts
without a BOM row.

Co-Authored-By: Claude Opus 5 <noreply@anthropic.com>
Parts:
- D1, D3: value LED -> Green
Changed lines of the file:
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@@
 			)
 		)
-		(property "Value" "LED"
+		(property "Value" "Green"
 			(at 254.635 143.8275 0)
 			(show_name no)
@@
 			)
 		)
-		(property "Value" "LED"
+		(property "Value" "Green"
 			(at 177.4825 46.355 0)
 			(show_name no)

Commit message: hardware: SMF10A TVS on VSYS -- LoRa CR5 and both GNSS boards (schematics)
Closes the LoRa review's finding 12, and extends it to the two GNSS
daughterboards, which turned out to have the same gap in a worse form.

VSYS is fed straight from an externally-handled connector that hot-plugs onto a
live 2S pack, and clamps nothing before the TPS62913's 18 V VIN abs max:

  lora  VSYS = { CR1.1, CR3.1, FL1.1 }   an ORing Schottky damps the ring
  gnss  VSYS = { FL1.1, J.3 }            connector pin straight into the choke

The GNSS boards lack the one element that was damping the LoRa board, so they
sit closer to the limit -- ~14.4 V worst-case ring against ~12.6 V. Neither
breaches 18 V on the hot-plug transient alone; the argument for the part is ESD
on a human-handled connector whose power pin has no protection, while the USB
port beside it does.

Part: PTTC SMF10A, LCSC C5444308, 56k in stock, $0.086 at 50+.
V_RWM 10 V is 19% above the 8.4 V full-charge pack, and V_BR 11.1 V min stays
clear of it even at -40 C. V_C 17 V at 11.8 A sits under the 18 V abs max --
that is what selects this part. The next step up, SMF12A, clamps at 19.9 V,
ABOVE the abs max, so it would pass through the very event being clamped. 10 V
is the only SMF step that clears both ends of this rail's narrow window.

Symbol/footprint/3D were already in the project, unused, from the SS24FL line
that was never fitted -- same SOD-123FL package, pads named A/C. New
Custom:SMF10A reuses Footprints:SODFL3617X108N and 3dmodels/SS24FL.step, with a
zener-style cathode bar so it reads as a unidirectional TVS. Note the existing
SS24FL symbol pointed at "SS24FL:SODFL3617X108N" -- a library nickname this
project never defined -- which is likely why the part was unusable; the new
symbol uses the real "Footprints" nickname.

All three placed at rot 0, the one rotation whose pin transform is verified
against this file. Connectivity confirmed by netlist: cathode on VSYS, anode on
GND, ERC clean on all three boards. P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
Parts:
- added CR1: SMF10A, Footprints:SODFL3617X108N, symbol Custom:SMF10A
Connections:
- net GND: now also CR1.A
- net VSYS: now also CR1.C
