File: hardware/base-station-mini/battery.kicad_sch (KiCad schematic)
At the start: 23 parts, among them J2 USB4110GFA, Q1 FS8205A, Q2 FS8205A, Q3 FS8205A, U14 DW01A, U5 BQ21040DBVR

Commit message: hardware(minis): cost-reduction part swaps (Tier A + USB-C + QMC5883P)
rocket-computer-mini:
- pyro high-side P-FETs U6-U10: TPN4R712MD -> Winsok WSD20L50DN33 (incumbent
  unbuyable at build qty until the Q4-2026 Mouser restock; land compatibility
  closed by numeric overlay of the vendor package drawing vs the TSON Advance
  land vs the Toshiba outline -- identical 0.202 mm bottom-metal overlap;
  first-article gate: end-face wetting + bench-fire)
- pyro-ARM N-FET U9: CSD16323Q3 -> AOS AON7534 (same pinout, land verified)
- gate drivers Q3-Q6: DTC123JEBTL -> DTC123JETL (SOT-416 leads land fully)
- battery shunt R72: CSSH0805FT2L00 -> Yageo PA0805FRF870R002L
- magnetometer U3: IIS2MDC -> QST QMC5883P (new Custom symbol + LGA-16 3x3
  footprint from the vendor land; U3 relocated, C2/C4/C6 re-arranged; C6
  220 nF -> 4.7 uF 16 V 0603 for the C1 reservoir; 2x2 mm all-layer no-pour
  rule area under the die; stale X/Y axis silk removed -- new markings when
  the firmware axis mapping is decided; needs a new ~10-register driver)
- USB-C stays GCT: the HRO's through-hole shell legs land inside the pyro
  terminal's back-side SMD pads -- physically blocked at this location

base-station-mini:
- USB-C J2: GCT USB4110-GF-A -> HRO TYPE-C-31-M-12 (project footprint with
  symbol-matched pad names; NPTH-aligned placement, mating face within
  0.03 mm of the GCT; R14/R15 nudged 1.0 mm, one GND via moved, VBUS
  re-bridged; DRC 0 unconnected / 0 parity; shell-leg holes must be fully
  filled with solder at assembly)
- thermistor TH1: 103AT-2 -> MF52B 103F3435-100 (beta 3435 matched, charger
  TS window unchanged)
- LEDs D6/D9: Kingbright -> Xinglight

both minis:
- 22 uF 0805: CL21A226MOQNNNE -> CL21A226KOQNNNE (tighter K tolerance)
- bom.csv regenerated from the schematics; TSON footprint tags updated

Verification: rocket-mini ERC one error better than baseline, DRC 246
unconnected (3 better), parity equal, no new errors; base-mini ERC unchanged,
DRC clean.

Co-Authored-By: Cla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
Parts:
- D9: MPN WP710A10QBC/D -> XL-304UBC; Mfr Kingbright -> Xinglight
- J2: value USB4110GFA -> TYPE-C-31-M-12; footprint Footprints:GCT_USB4110GFA -> Footprints:USB_C_HRO_TYPE-C-31-M-12; Description_1 USB-C (USB TYPE-C) USB 2.0 Receptacle Connector 24 (16+8 Du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 -> USB-C (USB TYPE-C) USB 2.0 Receptacle Connector, 16 Positio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; MF GCT -> Korean Hroparts; MP USB4110GFA -> TYPE-C-31-M-12; MPN USB4110-GF-A -> TYPE-C-31-M-12; Mfr GCT -> Korean Hroparts
- TH1: value Thermistor - 4316-103AT-2-ND -> Thermistor 10k NTC B3435; MPN 103AT-2 -> MF52B 103F3435-100; Mfr Semitec -> Nanjing Shiheng
Changed lines of the file:
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@@
 			)
 		)
-		(property "MPN" "WP710A10QBC/D"
+		(property "MPN" "XL-304UBC"
 			(at 153.67 71.755 0)
 			(hide yes)
@@
 			)
 		)
-		(property "Mfr" "Kingbright"
+		(property "Mfr" "Xinglight"
 			(at 153.67 71.755 0)
 			(hide yes)
@@
 			)
 		)
-		(property "Value" "Thermistor - 4316-103AT-2-ND"
+		(property "Value" "Thermistor 10k NTC B3435"
 			(at 93.345 76.1999 0)
 			(hide yes)
@@
 			)
 		)
-		(property "MPN" "103AT-2"
+		(property "MPN" "MF52B 103F3435-100"
 			(at 90.17 74.93 0)
 			(hide yes)
@@
 			)
 		)
-		(property "Mfr" "Semitec"
+		(property "Mfr" "Nanjing Shiheng"
 			(at 90.17 74.93 0)
 			(hide yes)
@@
 			)
 		)
-		(property "Value" "USB4110GFA"
+		(property "Value" "TYPE-C-31-M-12"
 			(at 44.45 41.91 0)
 			(show_name no)
@@
 			)
 		)
-		(property "Footprint" "Footprints:GCT_USB4110GFA"
+		(property "Footprint" "Footprints:USB_C_HRO_TYPE-C-31-M-12"
 			(at 44.45 54.61 0)
 			(hide yes)
@@
 			)
 		)
-		(property "MF" "GCT"
+		(property "MF" "Korean Hroparts"
 			(at 44.45 54.61 0)
 			(hide yes)
@@
 			)
 		)
-		(property "Description_1" "USB-C (USB TYPE-C) USB 2.0 Receptacle Connector 24 (16+8 Dummy) Position Surface Mount, Right Angle; Through Hole"
+		(property "Description_1" "USB-C (USB TYPE-C) USB 2.0 Receptacle Connector, 16 Position, top-mount SMT signals + through-hole shell legs"
 			(at 44.45 54.61 0)
 			(hide yes)
@@
 			)
 		)
-		(property "MP" "USB4110GFA"
+		(property "MP" "TYPE-C-31-M-12"
 			(at 44.45 54.61 0)
 			(hide yes)
@@
 			)
 		)
-		(property "MPN" "USB4110-GF-A"
+		(property "MPN" "TYPE-C-31-M-12"
 			(at 44.45 54.61 0)
 			(hide yes)
@@
 			)
 		)
-		(property "Mfr" "GCT"
+		(property "Mfr" "Korean Hroparts"
 			(at 44.45 54.61 0)
 			(hide yes)

Commit message: BS-mini: TH1 becomes an 0603 chip, and stops reading the cell (#967)
TH1 was a two-pin 2.54 mm land for a leaded thermistor meant to be taped to
the 18650, so the BQ21040's TS pin read CELL temperature. The new holder
leaves no room for a part under the cell, so the sensor moves onto the
component side as a 0603 chip.

Electrically this is a non-event. Both parts are 10 k at 25 C with
B25/85 = 3435 K, so the TS window does not move and R53 (210 k, TS to GND —
TI's TTDM-defeat resistor) is unchanged. Checked against the datasheet
rather than assumed: at the 50 uA bias and the 275 mV / 1250 mV thresholds
the trips land at ~40.5 C hot and ~0.3 C cold, and R53's 2.7 C cold shift
reproduces TI's own "≈3 C error at cold" note for that resistor. Worth
recording that the hot trip is ~41 C, not the 45 C the parameter is named
for — TI defines those thresholds against a different curve. The sensor's
own self-heat is nil: 50 uA into 10 k is 25 uW against a 1.2 mW/C
dissipation factor, so 0.02 C.

WHAT IT COSTS, and the direction matters. The NTC now reads the ground
plane, not the cell, and a warm board makes the charger believe the pack is
warmer than it is. On the hot side that is conservative — charging is
inhibited early. On the COLD side it is not: board self-heat can mask a
genuinely cold cell and permit a sub-0 C charge, which is the failure the TS
pin exists to prevent. First article should compare the TS node against a
probe on the cell while charging, at room temperature and near 0 C; if the
offset is too large the answer is a wired probe on a connector, not a
different chip. The README section added here says so.

PLACEMENT is (74.80, 156.00) rot 90, the far end of the board from the
charger. Weighting dissipation over distance that is 37% less coupling than
the old land: 25 mm from the BQ21040 (was 13.5) and 27 mm from the
buck-boost (was 8.6). The top of the board scores 47% but is not cleanly
routable, and that is a fact about this board rather than about this pa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
Parts:
- TH1: footprint Connector_PinHeader_2.54mm:PinHeader_1x02_P2.54mm_Vertical -> Resistor_SMD:R_0603_1608Metric; MPN MF52B 103F3435-100 -> TX06F103F3435ER; Mfr Nanjing Shiheng -> Ohmite
Changed lines of the file:
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@@
 			)
 		)
-		(property "Footprint" "Connector_PinHeader_2.54mm:PinHeader_1x02_P2.54mm_Vertical"
+		(property "Footprint" "Resistor_SMD:R_0603_1608Metric"
 			(at 90.17 74.93 0)
 			(hide yes)
@@
 			)
 		)
-		(property "Description" "Temperature dependent resistor"
+		(property "Description" "Battery temperature sense for the BQ21040 TS pin - 10 k NTC at 25 C, B25/85 = 3435 K, 0603. R53 (210 k, TS to GND) is TI's TTDM-defeat resistor. BOARD-MOUNTED, not on the cell: placed at the far end of the board from the charger, buck and ESP32-S3 so board self-heating biases the reading as little as possible. Consequence: the JEITA window tracks PCB temperature, so a cold cell in a self-heated board can still be charged - see the board README."
 			(at 90.17 74.93 0)
 			(hide yes)
@@
 			)
 		)
-		(property "MPN" "MF52B 103F3435-100"
+		(property "MPN" "TX06F103F3435ER"
 			(at 90.17 74.93 0)
 			(hide yes)
@@
 			)
 		)
-		(property "Mfr" "Nanjing Shiheng"
+		(property "Mfr" "Ohmite"
 			(at 90.17 74.93 0)
 			(hide yes)
