File: hardware/base-station-mini/esp32_p3.kicad_sch (KiCad schematic)
At the start: 33 parts, among them J6 Conn_01x04, U1 W25Q128JVSIQ, U15 479480001, U3 ESP32-S3RH2, Y1 ABS07-32.768KHZ-T, Y2 ECS-400-10-37B2-CKY-TR

Commit message: hardware: base-station-mini gains on-board LoRa, TPS63021, rev V1
Turns the fork into a reduced-feature ground station. "Mini" is fewer features,
not a smaller board -- the outline stays base-station's 30.27 x 90.50 mm.

RADIO. The E220-900MM22S (U16) is on-board on SPI, replacing the UART header
that fed an external lora-daughterboard. Eight ESP32 signals wired via the L_*
labels already placed on the module side; LoRa_TX/LoRa_RX/LoRa_EN were dangling
single-node stubs and their GPIOs went straight back into the radio bus.

All eight land on the same GPIOs as the fabbed lora-daughterboard -- SCK/17,
CS/18, MOSI/21, MISO/33, BUSY/34, RXEN/35, RST/38, DIO1/2 -- so the radio_board
firmware pin map applies unchanged. L_DI02 stays a module-local DIO2->TXEN loop,
so the SX1262 drives its own RF switch and spends no GPIO.

POWER. +3V3 had no source at all after the converters came out. Now a
fixed-output TPS63021 with FB tied to VOUT, matching base-station at V6. The 5 V
V_LORA boost stays deleted -- the on-board module runs off +3V3.

RF. J8 is new copper that exists on no other board. The feed was 0.20 mm, right
for a 0.1 mm prepreg but not for this stackup's real 0.2104 mm; it is now 0.36 mm
with a 0.15 mm coplanar gap, the value base-station's S7 derived for the same
JLCPCB JLC04161H-7628 stack. Net-(U16-ANT) was also missing from the RF netclass
-- the only RF net unique to this board was the one net not declared as RF -- so
it is added and the zones refilled.

ALSO. BT2 placed on B.Cu at base-station's exact coordinates, verified pad for
pad. external_charger.kicad_sch deleted rather than left orphaned; it held the
last copies of SDA_SENS, SCL_SENS, PosADC, MidADC and 25 dead symbols. Rev V1,
never fabbed. bom.csv regenerated -- it was 109 refs against a 78-ref schematic
and had never listed U16 or J8.

State: 0 schematic-parity issues, 0 unconnected, 25 DRC all silkscreen.
Reviewed in prefab-review-2026-08-12.md; three items open before fab, none
blockers.

Co-Auth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
Parts:
- removed J6: Conn_01x04, Connector_JST:JST_SH_BM04B-SRSS-TB_1x04-1MP_P1.00mm_Vertical, symbol Connector_Generic:Conn_01x04
- removed R5, R6: 5.11 k, Resistor_SMD:R_0402_1005Metric, symbol Device:R_US
- added C20: 22 uF, Capacitor_SMD:C_0805_2012Metric, symbol Device:C
- added C22: 100 nF, Capacitor_SMD:C_0402_1005Metric, symbol Device:C
- added J8: CON-SMA-EDGE-S, Footprints:RFSOLUTIONS_CON-SMA-EDGE-S, symbol Custom:CON-SMA-EDGE-S
- added U16: E220-900MM22S, Footprints:E220-900MM22S, symbol Custom:E220-900MM22S
Connections:
- net +3V3: now also C20.2, C22.2, U16.1 (VCC)
- net GND: now also C20.1, C22.1, J8.G1, J8.G2, J8.G3, J8.G4, U16.16 (GND), U16.2 (GND), U16.7 (GND)
- net L_SCK: now reaches U3.23 (GPIO17)
- net L_SCK: now also U16.15 (SCK)
- net L_CS: now reaches U3.24 (GPIO18)
- net L_CS: now also U16.14 (NSS)
- net L_RST: now reaches U3.43 (GPIO38)
- net L_RST: now also U16.3 (NRST)
- net L_DI01: now reaches U3.7 (GPIO2)
- net L_DI01: now also U16.20 (DIO1)
- net LoRa_EN renamed L_MOSI
- net L_MOSI: now also U16.13 (MOSI)
- net LoRa_RX: no longer names the net of U3.41 (GPIO36)
- net LoRa_TX renamed L_RXEN
- net L_RXEN: now also U16.10 (RXEN)
- net MidADC: no longer names the net of U3.14 (GPIO9)
- net PosADC: no longer names the net of U3.13 (GPIO8)
- net SCL_SENS renamed L_BUSY
- net L_BUSY: now also U16.11 (BUSY)
- net SDA_SENS renamed L_MISO
- net L_MISO: now also U16.12 (MISO)
- new net: J8.1, U16.6 (ANT)
- new net L_DI02: U16.19 (DIO2), U16.9 (TXEN)

Commit message: hardware: cheaper flash across the fleet, and revs for the boards that had drifted
rocket-computer-mini U11: GD5F2GQ5UEYIGR (2 Gbit) -> GD5F1GQ5UEYIGR (1 Gbit).
Same GigaDevice family, same WSON-8 8x6 land, same pinout and 3.3 V rail, and
the ESP-IDF spi_nand_flash driver already carries device ID 0x51 (1024 blocks =
128 MB) -- a value/MPN change with no layout or firmware work. -$3.81/bd. Also
fixes U11's Datasheet field, which pointed at MX35UF4G24AD-Z4I8, a 1.8 V
Macronix part (flagged as an INFO finding in prefab-review-2026-08-05).

Boot NOR on all six placements: W25Q128JVSIQ -> GD25Q128ESIG (rocket-computer
U13+U16, base-station U1, base-station-mini U1, lora-daughterboard U22,
rocket-computer-mini U13). Identical SOIC-8 208 mil land and standard SPI-NOR
pinout (1 CS#, 2 SO/IO1, 3 WP#/IO2, 4 VSS, 5 SI/IO0, 6 SCLK, 7 HOLD#/IO3,
8 VCC), 2.7-3.6 V, 16 MB, and ESP-IDF has a first-party driver
(spi_flash_chip_gd.c, default y on S3) -- unlike the cheaper Puya part, which
would fall to the generic driver on a boot device. -$1.0471/pc over a 700 pc
line. WSON and 150 mil variants were swept and are 1.5-3.3x dearer for the same
die, so the 208 mil land stays. The shared 3D model is renamed to match; its
geometry is unchanged because the package is identical.

New revs on the boards that had changed since their fab tag without one:
rocket-computer V9 -> V10 and lora-daughterboard V3 -> V4 for this swap, and
gnss-px1105r V1 -> V2 for changes that predate it -- 8a95e02 refilled zones to
clear a 3V3-to-GND short in the stored artwork and da39e6e moved the board off
the default stackup, neither ever marked with a rev. base-station was already
V6; gnss-sam10m8 and servo-adapter are unchanged since fab; the two mini boards
have never been fabbed.

rocket-computer-mini/bom.csv regenerated from the schematic -- it was still the
parent board's BOM from the fork (243 designators against the schematic's 149;
U16 listed as a W25Q128 when it is the E220 radio; U5, the on-board GNSS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
Parts:
- U1: value W25Q128JVSIQ -> GD25Q128ESIG; MPN W25Q128JVSIQ -> GD25Q128ESIG; Mfr Winbond -> GigaDevice
Changed lines of the file:
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@@
 			)
 		)
-		(property "Value" "W25Q128JVSIQ"
+		(property "Value" "GD25Q128ESIG"
 			(at 65.405 106.045 0)
 			(show_name no)
@@
 			)
 		)
-		(property "MPN" "W25Q128JVSIQ"
+		(property "MPN" "GD25Q128ESIG"
 			(at 21.59 115.57 0)
 			(hide yes)
@@
 			)
 		)
-		(property "Mfr" "Winbond"
+		(property "Mfr" "GigaDevice"
 			(at 21.59 115.57 0)
 			(hide yes)

Commit message: hardware: name the SOIC-8 flash land for its package, not for a part number
SOIC-8_W25Q128JVSIQ.kicad_mod -> SOIC127P790X216-8N.kicad_mod, and the 3D model
with it, so neither carries the name of a device that is no longer fitted. The
descr had drifted further than the filename: it still read "Winbond
W25Q128JVSIQ ... LCSC C97521" over a GigaDevice part, and now describes the land
itself and says why it is not part-named.

The repo already has a casualty of part-named footprints -- IC_TPS259827LNRGER
holds the fitted TPS259824LNRGET, which prefab-review-2026-08-05 flagged as a
mismatch that "invites a wrong-variant order". Naming this land for its package
means the next change of fitted device needs no rename at all.

37 references updated across 5 PCBs, 5 schematics, 4 bom.csv and the footprint;
the footprint's internal name now matches its filename again.

The Custom:W25Q128JVSIQ symbol is deliberately left alone: its schematic copies
already differ from the shared Custom.kicad_sym (a known lib_symbol_mismatch),
so renaming it there is a separate and riskier job. Its stale
"W25Q128JVSIQ:SOIC127P790X216-8N" footprint nickname is now half correct, and
fixing it later is just dropping the dead library prefix.

Also rocket-computer-mini rev "rev1" -> "V1" -- it was the only board not using
the V notation.

Co-Authored-By: Claude Opus 5 <noreply@anthropic.com>
Parts:
- U1: footprint Footprints:SOIC-8_W25Q128JVSIQ -> Footprints:SOIC127P790X216-8N
Changed lines of the file:
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@@
 			)
 		)
-		(property "Footprint" "Footprints:SOIC-8_W25Q128JVSIQ"
+		(property "Footprint" "Footprints:SOIC127P790X216-8N"
 			(at 21.59 115.57 0)
 			(hide yes)

Commit message: hardware(minis): cost-reduction part swaps (Tier A + USB-C + QMC5883P)
rocket-computer-mini:
- pyro high-side P-FETs U6-U10: TPN4R712MD -> Winsok WSD20L50DN33 (incumbent
  unbuyable at build qty until the Q4-2026 Mouser restock; land compatibility
  closed by numeric overlay of the vendor package drawing vs the TSON Advance
  land vs the Toshiba outline -- identical 0.202 mm bottom-metal overlap;
  first-article gate: end-face wetting + bench-fire)
- pyro-ARM N-FET U9: CSD16323Q3 -> AOS AON7534 (same pinout, land verified)
- gate drivers Q3-Q6: DTC123JEBTL -> DTC123JETL (SOT-416 leads land fully)
- battery shunt R72: CSSH0805FT2L00 -> Yageo PA0805FRF870R002L
- magnetometer U3: IIS2MDC -> QST QMC5883P (new Custom symbol + LGA-16 3x3
  footprint from the vendor land; U3 relocated, C2/C4/C6 re-arranged; C6
  220 nF -> 4.7 uF 16 V 0603 for the C1 reservoir; 2x2 mm all-layer no-pour
  rule area under the die; stale X/Y axis silk removed -- new markings when
  the firmware axis mapping is decided; needs a new ~10-register driver)
- USB-C stays GCT: the HRO's through-hole shell legs land inside the pyro
  terminal's back-side SMD pads -- physically blocked at this location

base-station-mini:
- USB-C J2: GCT USB4110-GF-A -> HRO TYPE-C-31-M-12 (project footprint with
  symbol-matched pad names; NPTH-aligned placement, mating face within
  0.03 mm of the GCT; R14/R15 nudged 1.0 mm, one GND via moved, VBUS
  re-bridged; DRC 0 unconnected / 0 parity; shell-leg holes must be fully
  filled with solder at assembly)
- thermistor TH1: 103AT-2 -> MF52B 103F3435-100 (beta 3435 matched, charger
  TS window unchanged)
- LEDs D6/D9: Kingbright -> Xinglight

both minis:
- 22 uF 0805: CL21A226MOQNNNE -> CL21A226KOQNNNE (tighter K tolerance)
- bom.csv regenerated from the schematics; TSON footprint tags updated

Verification: rocket-mini ERC one error better than baseline, DRC 246
unconnected (3 better), parity equal, no new errors; base-mini ERC unchanged,
DRC clean.

Co-Authored-By: Cla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
Parts:
- C20: MPN CL21A226MOQNNNE -> CL21A226KOQNNNE
Changed lines of the file:
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@@
 			)
 		)
-		(property "MPN" "CL21A226MOQNNNE"
+		(property "MPN" "CL21A226KOQNNNE"
 			(at 46.99 153.67 0)
 			(hide yes)

Commit message: hardware(base-mini): the 22 uF 0805 follows the fleet back to the M-code
The last board still carrying the retired K grade. #1454 (V10) and #1455
(rocket-mini) moved the other two after the priced CrossBoard BOM retired the
CL21A226KOQNNNE line on 2026-08-28 — it had repriced up to $0.1257@2000 against
the M-code's $0.0725 — and merged both minis back onto the M part. The sheet has
billed this board on the M line ever since; only its schematic still said K.

All seven placements (C20, C42, C58, C59, C60, C61, C62) move to
CL21A226MOQNNNE across the two sheets that carry them, the board's fields, and
bom.csv. Same Samsung series, same 0805, same 16 V.

That is the whole fleet on one 22 uF 0805 line again: rocket-computer 12,
rocket-computer-mini 14, base-station 12, base-station-mini 7,
lora-daughterboard 8.

Measured: field-only. Netlist unchanged at 80 components and 91 nets.
kicad-cli sch erc --severity-all unchanged at 402. kicad-cli pcb drc
--severity-all --schematic-parity unchanged at 49. bom.csv reconciles to the
schematic. check_docs.py clean.

Co-Authored-By: Claude Opus 5 <noreply@anthropic.com>
Parts:
- C20: MPN CL21A226KOQNNNE -> CL21A226MOQNNNE
Changed lines of the file:
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@@
 			)
 		)
-		(property "MPN" "CL21A226KOQNNNE"
+		(property "MPN" "CL21A226MOQNNNE"
 			(at 46.99 153.67 0)
 			(hide yes)
