File: hardware/rocket-computer/rocket-computer.kicad_sch (KiCad schematic)
At the start: 15 parts, among them U1 FSUSB63UMX

Commit message: hardware: MPN + Mfr on every purchased part of the three ESP32 boards
Closes the LoRa pre-fab review's finding 3, extended to the sibling boards.
Every non-DNP symbol now names the exact part the cross-board BOM prices, so
the schematic can no longer imply a part that was never quoted.

401 of 401 purchasable parts carry an MPN. The only exemptions are the three
DNP v3.x provisions on the rocket-computer (R74/R75 499 k, R76 0 R): not
fitted, so never purchased, so correctly absent from the BOM.

Values normalised so each part resolves to one BOM line:

  LoRa R74  "10 K" -> "10 k"   capital K split one part across two lines
  LoRa D6   "LED"  -> "Green"  no colour recorded, so no MPN could attach
  Y1/Y3/Y5  "SC-32S-32.768kHz-12.5pF" -> "ABS07-32.768KHZ-T"

Two stale legacy MP fields disagreed with both the Value and the BOM and were
corrected -- a symbol carrying two part numbers is the wrong-part-order hazard
this pass exists to remove:

  rocket U19  TPS259824LNRGER -> ...RGET.  Same die and RGE-24 package; the
              suffix is reel quantity, and power-eco.md documents RGET.
  base   U9   TPS63021DSJR -> TPS63020DSJR.  These are NOT interchangeable:
              63021 is fixed 3.3 V, 63020 is adjustable. U9 pin 3 (FB) drives
              a real divider (R13 1 M / R16 180 k -> 0.5 x (1 + 1M/180k) =
              3.28 V), which only the adjustable part uses. BOM was right.

The ABS07 keeps the existing XTAL_SC-32S_3215 footprint: both parts are
2-pad 3.2 x 1.5 mm tuning forks, so the land is correct and only the
footprint's name now reads for the superseded vendor.

ERC clean on all three boards after the pass.

Co-Authored-By: Claude Opus 5 <noreply@anthropic.com>
Parts:
- C1: MPN (none) -> CL05B104KO5NNNC; Mfr (none) -> Samsung
- R1, R2: MPN (none) -> RC0402FR-07100KL; Mfr (none) -> Yageo
- R3: MPN (none) -> RC0402FR-0710RL; Mfr (none) -> Yageo
- S1: MPN (none) -> JS202011JCQN; Mfr (none) -> Same Sky (CUI)
- U1: MPN (none) -> FSUSB63UMX; Mfr (none) -> onsemi
Changed lines of the file:
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@@
+			)
+		)
+		(property "MPN" "CL05B104KO5NNNC"
+			(at 67.945 39.37 0)
+			(hide yes)
+			(show_name no)
+			(do_not_autoplace no)
+			(effects
+				(font
+					(size 1.27 1.27)
+				)
+			)
+		)
+		(property "Mfr" "Samsung"
+			(at 67.945 39.37 0)
+			(hide yes)
+			(show_name no)
+			(do_not_autoplace no)
+			(effects
+				(font
+					(size 1.27 1.27)
+				)
 			)
 		)
@@
 			)
 		)
+		(property "MPN" "FSUSB63UMX"
+			(at 41.91 55.245 0)
+			(hide yes)
+			(show_name no)
+			(do_not_autoplace no)
+			(effects
+				(font
+					(size 1.27 1.27)
+				)
+			)
+		)
+		(property "Mfr" "onsemi"
+			(at 41.91 55.245 0)
+			(hide yes)
+			(show_name no)
+			(do_not_autoplace no)
+			(effects
+				(font
+					(size 1.27 1.27)
+				)
+			)
+		)
 		(pin "4"
 		)
@@
 			)
 		)
+		(property "MPN" "RC0402FR-07100KL"
+			(at 52.705 85.09 0)
+			(hide yes)
+			(show_name no)
+			(do_not_autoplace no)
+			(effects
+				(font
+					(size 1.27 1.27)
+				)
+			)
+		)
+		(property "Mfr" "Yageo"
+			(at 52.705 85.09 0)
+			(hide yes)
+			(show_name no)
+			(do_not_autoplace no)
+			(effects
+				(font
+					(size 1.27 1.27)
+				)
+			)
+		)
 		(pin "1"
 		)
@@
 			)
 		)
+		(property "MPN" "RC0402FR-0710RL"
+			(at 67.945 31.115 0)
+			(hide yes)
+			(show_name no)
+			(do_not_autoplace no)
+			(effects
+				(font
+					(size 1.27 1.27)
+				)
+			)
+		)
+		(property "Mfr" "Yageo"
+			(at 67.945 31.115 0)
+			(hide yes)
+			(show_name no)
+			(do_not_autoplace no)
+			(effects
+				(font
+					(size 1.27 1.27)
+				)
+			)
+		)
 		(pin "1"
 		)
@@
 			)
 		)
+		(property "MPN" "RC0402FR-07100KL"
+			(at 18.415 46.355 0)
+			(hide yes)
+			(show_name no)
+			(do_not_autoplace no)
+			(effects
+				(font
+					(size 1.27 1.27)
+				)
+			)
+		)
+		(property "Mfr" "Yageo"
+			(at 18.415 46.355 0)
+			(hide yes)
+			(show_name no)
+			(do_not_autoplace no)
+			(effects
+				(font
+					(size 1.27 1.27)
+				)
+			)
+		)
 		(pin "1"
 		)
@@
 			)
 		)
+		(property "MPN" "JS202011JCQN"
+			(at 36.83 88.9 0)
+			(hide yes)
+			(show_name no)
+			(do_not_autoplace no)
+			(effects
+				(font
+					(size 1.27 1.27)
+				)
+			)
+		)
+		(property "Mfr" "Same Sky (CUI)"
+			(at 36.83 88.9 0)
+			(hide yes)
+			(show_name no)
+			(do_not_autoplace no)
+			(effects
+				(font
+					(size 1.27 1.27)
+				)
+			)
+		)

Commit message: hardware(rocket-computer): V9 pre-fab review close-out -- every finding fixed, measured, or waived
Closes the 2026-08-04..09 pre-manufacturing review (170 raw findings).
WORKLIST.md is the closing record: D-1..D-4 decided, H-1..H-10 and
M-1..M-25 dispositioned, Lows annotated, bench list is the remainder.

Power architecture:
- All four peripheral branches converted low-side N-FET -> integrated
  high-side switches (U26/U28 TPS22811LRPWR, U27/U29 TPS22810DRVR);
  U30 TPS22810DRVR gates the P4 domain. Every connector ground is now
  hard GND; the 12 EXP lines stay resistor-free by design (H-3/D-4).
  J3 and J4 power pins swapped ends -- fab notes B6/B7 carry the
  harness warnings.
- Q11 (CSD25404Q3) reverse-polarity P-FET at the battery input on a
  new TI-pattern footprint; CR2 re-purposed as connector ESD clamp
  upstream of it (M-9/M-10). Kelvin sense at R72 preserved.
- P4 rail self-latch: D9 (BAV170M) OR-gates S3 request with P4 hold,
  C105 rides the P4 through its own reset (H-4; firmware in #718).
- eFuse UVLO deglitch C94 (H-1); brownout decided as clean-reboot,
  ECO hold-up claims corrected in power-eco.md (H-8/D-3).
- Pyro gate-drive stiffened: R22 -> 5.11k, R78-R81 shunts (H-2).
- Servo budget decided at 3 A set by the In2 stretch; ILIM left open
  at 11.6 A; SERVO_IMON flight data gates any increase (D-1).

Component and BOM:
- TPS2121 ILIM 18.7k -> 49.9k (real protection at 2.26 A typ, M-5).
- IMON scaling: R85 -> 2.2k (3 A camera), R88 -> 1k (servo open).
- C27 VDD_SPI 10u -> 1u per HDG (M-4); switch VIN bypass 100n -> 1u;
  C40/C76 consolidation; C65 MPN fixed (was a 390 pF part number
  under a 100 nF value -- would have misassembled the buck bypass).
- SW2/SW3 on the R-667995 tact switch, footprint imported and pads
  renumbered to match; FB-network DNP parts carry MPNs for the v3.x
  flip (M-22); bom.csv regenerated: 79 lines / 243 placements, every
  part carries an MPN. Priced BOMs evicted from board dirs (they live
  in Documents/Circuit Board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
Parts:
- added FID2, FID3, FID4: Fiducial, Fiducial:Fiducial_0.5mm_Mask1mm, symbol Mechanical:Fiducial
Changed lines of the file:
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@@
+	)
+	(symbol
+		(lib_id "Mechanical:Fiducial")
+		(at 148.59 191.77 0)
+		(unit 1)
+		(body_style 1)
+		(exclude_from_sim no)
+		(in_bom no)
+		(on_board yes)
+		(in_pos_files yes)
+		(dnp no)
+		(fields_autoplaced yes)
+		(property "Reference" "FID4"
+			(at 151.765 190.4999 0)
+			(show_name no)
+			(do_not_autoplace no)
+			(effects
+				(font
+					(size 1.27 1.27)
+				)
+				(justify left)
+			)
+		)
+		(property "Value" "Fiducial"
+			(at 151.765 193.0399 0)
+			(show_name no)
+			(do_not_autoplace no)
+			(effects
+				(font
+					(size 1.27 1.27)
+				)
+				(justify left)
+			)
+		)
+		(property "Footprint" "Fiducial:Fiducial_0.5mm_Mask1mm"
+			(at 148.59 191.77 0)
+			(hide yes)
+			(show_name no)
+			(do_not_autoplace no)
+			(effects
+				(font
+					(size 1.27 1.27)
+				)
+			)
+		)
+		(property "Datasheet" ""
+			(at 148.59 191.77 0)
+			(hide yes)
+			(show_name no)
+			(do_not_autoplace no)
+			(effects
+				(font
+					(size 1.27 1.27)
+				)
+			)
+		)
+		(property "Description" "Fiducial Marker"
+			(at 148.59 191.77 0)
+			(hide yes)
+			(show_name no)
+			(do_not_autoplace no)
+			(effects
+				(font
+					(size 1.27 1.27)
+				)
+			)
+		)
+		(instances
+			(project "rocket-computer"
+				(path "/ae61c2c4-72e9-4776-93ae-2e716b9dc70f"
+					(reference "FID4")
+					(unit 1)
+				)
+			)
+		)
 	)
 	(symbol
@@
 	)
 	(symbol
+		(lib_id "Mechanical:Fiducial")
+		(at 132.715 184.785 0)
+		(unit 1)
+		(body_style 1)
+		(exclude_from_sim no)
+		(in_bom no)
+		(on_board yes)
+		(in_pos_files yes)
+		(dnp no)
+		(fields_autoplaced yes)
+		(property "Reference" "FID2"
+			(at 135.89 183.5149 0)
+			(show_name no)
+			(do_not_autoplace no)
+			(effects
+				(font
+					(size 1.27 1.27)
+				)
+				(justify left)
+			)
+		)
+		(property "Value" "Fiducial"
+			(at 135.89 186.0549 0)
+			(show_name no)
+			(do_not_autoplace no)
+			(effects
+				(font
+					(size 1.27 1.27)
+				)
+				(justify left)
+			)
+		)
+		(property "Footprint" "Fiducial:Fiducial_0.5mm_Mask1mm"
+			(at 132.715 184.785 0)
+			(hide yes)
+			(show_name no)
+			(do_not_autoplace no)
+			(effects
+				(font
+					(size 1.27 1.27)
+				)
+			)
+		)
+		(property "Datasheet" ""
+			(at 132.715 184.785 0)
+			(hide yes)
+			(show_name no)
+			(do_not_autoplace no)
+			(effects
+				(font
+					(size 1.27 1.27)
+				)
+			)
+		)
+		(property "Description" "Fiducial Marker"
+			(at 132.715 184.785 0)
+			(hide yes)
+			(show_name no)
+			(do_not_autoplace no)
+			(effects
+				(font
+					(size 1.27 1.27)
+				)
+			)
+		)
+		(instances
+			(project "rocket-computer"
+				(path "/ae61c2c4-72e9-4776-93ae-2e716b9dc70f"
+					(reference "FID2")
+					(unit 1)
+				)
+			)
+		)
+	)
+	(symbol
 		(lib_id "Mechanical:MountingHole")
 		(at 37.465 193.04 0)
@@
 					(unit 1)
 				)
+			)
+		)
+	)
+	(symbol
+		(lib_id "Mechanical:Fiducial")
+		(at 148.59 184.15 0)
+		(unit 1)
+		(body_style 1)
+		(exclude_from_sim no)
+		(in_bom no)
+		(on_board yes)
+		(in_pos_files yes)
+		(dnp no)
+		(fields_autoplaced yes)
+		(property "Reference" "FID3"
+			(at 151.765 182.8799 0)
+			(show_name no)
+			(do_not_autoplace no)
+			(effects
+				(font
+					(size 1.27 1.27)
+				)
+				(justify left)
+			)
+		)
+		(property "Value" "Fiducial"
+			(at 151.765 185.4199 0)
+			(show_name no)
+			(do_not_autoplace no)
+			(effects
+				(font
+					(size 1.27 1.27)
+				)
+				(justify left)
+			)
+		)
+		(property "Footprint" "Fiducial:Fiducial_0.5mm_Mask1mm"
+			(at 148.59 184.15 0)
+			(hide yes)
+			(show_name no)
+			(do_not_autoplace no)
+			(effects
+				(font
+					(size 1.27 1.27)
+				)
+			)
+		)
+		(property "Datasheet" ""
+			(at 148.59 184.15 0)
+			(hide yes)
+			(show_name no)
+			(do_not_autoplace no)
+			(effects
+				(font
+					(size 1.27 1.27)
+				)
+			)
+		)
+		(property "Description" "Fiducial Marker"
+			(at 148.59 184.15 0)
+			(hide yes)
+			(show_name no)
+			(do_not_autoplace no)
+			(effects
+				(font
+					(size 1.27 1.27)
+				)
+			)
+		)
+		(instances
+			(project "rocket-computer"
+				(path "/ae61c2c4-72e9-4776-93ae-2e716b9dc70f"
+					(reference "FID3")
+					(unit 1)
+				)

Commit message: hardware: consolidate five resistor lines onto fleet values (rocket, base-station)
Cross-board BOM line reduction; netlist-verified functions, no ratio-
critical or safety-analyzed parts touched:

- rocket R3 10R -> 22R: FSUSB63 VCC supply filter, uA load; 22R is a
  three-board fleet line, retires the 10R line
- rocket R85 2.2k -> 2k: TPS22811 CAM_IMON gain load; joins the base's
  2k line, retires 2.2k. FIRMWARE: IMON scale changes by x0.909
- base R17 18.7k -> 100k: TPS61023 EN pull-up, value non-critical;
  retires the fleet's last 18.7k line
- base R40/R42 300k/100k -> 1M/180k: battery ADC divider re-ratioed
  onto fleet values (8.4V -> 1.281V at GPIO8, was 2.1V; source
  impedance 152k against the 100nF reservoir C55, pack drain drops
  21uA -> 7uA). FIRMWARE: scale constant 4.000 -> 6.5556; retires 300k
- PCB field sync included (R85's board-side MPN still carried the
  pre-fix 3.3k code; now consistent both sides)

Deliberately NOT consolidated after review: U9 stays CSD16323Q3 (pyro
arm FET -- WORKLIST H-2 glitch-margin analysis is against this part's
threshold; H-9 fire-return layout built into its drain pad); base L6
stays SRP4020TA-1R5M (it is the MP2672 switching inductor, not a
filter -- a VLS3012 would saturate).

ERC profiles unchanged both boards; DRC error-severity: base clean,
rocket = the three accepted courtyard overlaps. bom.csv regenerated.

Co-Authored-By: Claude Fable 5 <noreply@anthropic.com>
Parts:
- R3: value 10 -> 22; MPN RC0402FR-0710RL -> RC0402FR-0722RL
Changed lines of the file:
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@@
 			)
 		)
-		(property "Value" "10"
+		(property "Value" "22"
 			(at 66.04 30.48 90)
 			(show_name no)
@@
 			)
 		)
-		(property "MPN" "RC0402FR-0710RL"
+		(property "MPN" "RC0402FR-0722RL"
 			(at 67.945 31.115 0)
 			(hide yes)

Commit message: hardware(V10): the #678 sweep — NRETRY to ground, LEDs at 1 k, H2 grounded, the missing bypasses, and the U9 pin-9 parity fix (#1360)
Schematic, library and BOM only; the board is untouched. Record:
hardware/rocket-computer/v10-power-parity-2026-09-11.md section 6.4.

## Owner decisions (2026-09-11)

- NRETRY to ground: C45 (1 uF, ~1800 retries, past the datasheet's last
  quantization bucket) deleted, U19 pin 11 tied to GND. With C46 2.2 nF
  still on RETRY_DLY the TPS25982 fault table reads "auto-retry
  indefinitely with finite delay" -- a finite count ends in latch-off,
  which a flight computer must never do.
- Status LEDs: R65, R66, R70 10 k -> 1 k (stocked line). ~1.5 mA green,
  ~1.3 mA red, ~0.4 mA blue instead of 0.05-0.15 mA.
- H2, the plated mounting ring 0.6 mm from the antenna body, on no net:
  H2 becomes Mechanical:MountingHole_Pad with pin 1 on GND. The other
  seven holes are unchanged; the pad's zone connection is the layout
  pass's.

## Simple adds from the same list

- C44 soft-start 390 pF -> 10 nF (the buck started in current limit into
  its output capacitance; ~5 ms now, datasheet class).
- R141 10 k pull-up on S3 GPIO0 to +3V3, on the wire to the boot button.
- C146 / C147 100 nF at the IMU and baro VDD pins (their nearest 100 nF
  was the magnetometer's at 3-4 mm), on V_MCU_SWTCH.
- C148 10 uF on the S3 RF supply net, converter side of L4 (the guide
  asks 10 uF per RF pin; there was only C33 100 nF).
- ISM6HG256_INT2: single-pin label replaced by a no-connect flag.
- U9 CSD16323Q3 symbol pin 9 renumbered 5 in Custom.kicad_sym and in the
  cached copies on this board and the mini: the shared TSON footprint
  numbers its drain tab as a second pad 5, so the symbol now matches it
  and the permanent "no pad for pin 9" parity warning is gone on both
  boards. Netlists unchanged.
- power-eco.md Change 2 pin table rewritten to the as-built designators
  and values (ITIMER/dVdt/NRETRY had drifted; the input clamp is gone).

Not changed, recorded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
Parts:
- H2: value MountingHole -> MountingHole_Pad; symbol Mechanical:MountingHole -> Mechanical:MountingHole_Pad
Connections:
- net GND: now also H2.1
Changed lines of the file:
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@@
 	)
 	(symbol
-		(lib_id "Mechanical:MountingHole")
+		(lib_id "Mechanical:MountingHole_Pad")
 		(at 17.78 193.675 0)
 		(unit 1)
@@
 			)
 		)
-		(property "Value" "MountingHole"
+		(property "Value" "MountingHole_Pad"
 			(at 20.32 194.9449 0)
 			(show_name no)
@@
 			)
 		)
-		(property "Description" "Mounting Hole without connection"
+		(property "Description" "Mounting Hole with connection"
 			(at 17.78 193.675 0)
 			(hide yes)
@@
 				)
 			)
+		)
+		(pin "1"
 		)
 		(instances
@@
 	)
 	(embedded_fonts no)
+	(symbol
+		(lib_id "power:GND")
+		(at 17.78 196.215 0)
+		(unit 1)
+		(body_style 1)
+		(exclude_from_sim no)
+		(in_bom yes)
+		(on_board yes)
+		(in_pos_files yes)
+		(dnp no)
+		(fields_autoplaced yes)
+		(property "Reference" "#PWR0710"
+			(at 17.78 202.565 0)
+			(hide yes)
+			(show_name no)
+			(do_not_autoplace no)
+			(effects
+				(font
+					(size 1.27 1.27)
+				)
+			)
+		)
+		(property "Value" "GND"
+			(at 17.78 201.295 0)
+			(show_name no)
+			(do_not_autoplace no)
+			(effects
+				(font
+					(size 1.27 1.27)
+				)
+			)
+		)
+		(property "Footprint" ""
+			(at 17.78 196.215 0)
+			(hide yes)
+			(show_name no)
+			(do_not_autoplace no)
+			(effects
+				(font
+					(size 1.27 1.27)
+				)
+			)
+		)
+		(property "Datasheet" ""
+			(at 17.78 196.215 0)
+			(hide yes)
+			(show_name no)
+			(do_not_autoplace no)
+			(effects
+				(font
+					(size 1.27 1.27)
+				)
+			)
+		)
+		(property "Description" "Power symbol creates a global label with name \"GND\" , ground"
+			(at 17.78 196.215 0)
+			(hide yes)
+			(show_name no)
+			(do_not_autoplace no)
+			(effects
+				(font
+					(size 1.27 1.27)
+				)
+			)
+		)
+		(pin "1"
+		)
+		(instances
+			(project "rocket-computer"
+				(path "/ae61c2c4-72e9-4776-93ae-2e716b9dc70f"
+					(reference "#PWR0710")
+					(unit 1)
+				)
+			)
+		)
+	)
 )

Commit message: rocket-computer: the V10 ERC error floor goes from 62 to 0 without touching a net (#680)
The 62 errors were noise that buried anything real: 38 deliberately unused
pins without no-connect flags, 12 power inputs on nets with no power output,
and 12 pin-type clashes from shared symbols whose grounds were typed as power
outputs and whose tied-off open-drain pins were typed as outputs.

Pin types are fixed in the shared library and in every cached copy that
instantiates the symbol: IC grounds are power inputs; one power output per
net (eFuse OUT 17 drives VBATT, the P4's internal-LDO outputs drive VDDO_*,
the S3's VDD_SPI is a regulator output in the in-package-flash configuration
every board here uses); tied-off open-drain pins are passive; the TPS62152's
hidden thermal pad is no longer a hidden power input (the source of the
GND/PGND multiple-net-names warning). Six PWR_FLAGs mark the nets fed
through an inductor or resistor, plus GND. 38 no-connect flags. AONR21321
joins the library. Six stray wire stubs and an orphan VBATT symbol go.

Netlists are byte-identical before and after on all five boards touched.
V10 62 -> 0 errors; through the shared symbols the mini goes 40 -> 33, the
base stations 47 -> 46 and 40 -> 39, the LoRa daughterboard 34 -> 33. The
mini's remainder is its own (QMC5883P/BMP581 grounds, its flags) and is
listed in the note.

Co-Authored-By: Claude Fable 5.1 <noreply@anthropic.com>
Connections:
- no-connect marks 0 -> 6
Changed lines of the file:
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@@
 	(wire
 		(pts
-			(xy 67.945 35.56) (xy 57.15 35.56)
+			(xy 67.945 35.56) (xy 62.23 35.56)
+		)
+		(stroke
+			(width 0)
+			(type default)
+		)
+	)
+	(wire
+		(pts
+			(xy 62.23 35.56) (xy 57.15 35.56)
 		)
 		(stroke
@@
 		)
 	)
+	(junction
+		(at 62.23 35.56)
+		(diameter 0)
+		(color 0 0 0 0)
+	)
+	(symbol
+		(lib_id "power:PWR_FLAG")
+		(at 62.23 35.56 0)
+		(unit 1)
+		(body_style 1)
+		(exclude_from_sim no)
+		(in_bom yes)
+		(on_board yes)
+		(in_pos_files yes)
+		(dnp no)
+		(property "Reference" "#FLG01"
+			(at 62.23 33.655 0)
+			(hide yes)
+			(show_name no)
+			(do_not_autoplace no)
+			(effects
+				(font
+					(size 1.27 1.27)
+				)
+			)
+		)
+		(property "Value" "PWR_FLAG"
+			(at 60.325 33.655 0)
+			(show_name no)
+			(do_not_autoplace no)
+			(effects
+				(font
+					(size 1.27 1.27)
+				)
+				(justify right)
+			)
+		)
+		(property "Footprint" ""
+			(at 62.23 35.56 0)
+			(hide yes)
+			(show_name no)
+			(do_not_autoplace no)
+			(effects
+				(font
+					(size 1.27 1.27)
+				)
+			)
+		)
+		(property "Datasheet" ""
+			(at 62.23 35.56 0)
+			(hide yes)
+			(show_name no)
+			(do_not_autoplace no)
+			(effects
+				(font
+					(size 1.27 1.27)
+				)
+			)
+		)
+		(property "Description" "Special symbol for telling ERC where power comes from"
+			(at 62.23 35.56 0)
+			(hide yes)
+			(show_name no)
+			(do_not_autoplace no)
+			(effects
+				(font
+					(size 1.27 1.27)
+				)
+			)
+		)
+		(pin "1"
+		)
+		(instances
+			(project "rocket-computer"
+				(path "/ae61c2c4-72e9-4776-93ae-2e716b9dc70f"
+					(reference "#FLG01")
+					(unit 1)
+				)
+			)
+		)
+	)
+	(no_connect
+		(at 57.15 57.785)
+	)
+	(no_connect
+		(at 57.15 47.625)
+	)
+	(no_connect
+		(at 24.13 86.36)
+	)
+	(no_connect
+		(at 24.13 88.9)
+	)
+	(no_connect
+		(at 24.13 91.44)
+	)
+	(no_connect
+		(at 49.53 86.36)
+	)
 )
