File: hardware/servo-adapter/servo-adapter.kicad_pcb (KiCad board)
At the start: 4 copper layers, 24.4 x 16.4 mm, 9 parts, among them J1 Conn_01x06_Pin, J2 6130XX21021_61300621021, J3 6130XX21021_61300621021

Commit message: hardware(servo-adapter): layout for C5 and R1-R4; C1-C4 to the fleet 22 uF 0805
Layout (the owner's): C5 and R1-R4 placed and routed. DRC reports no
unconnected items.

Schematic: C1-C4 move to the fleet's 22 uF 0805 (Samsung CL21A226MOQNNNE,
16 V). This is the same part the V9/V10 already run on the 8.4 V rail;
more can be added if needed. MinVRating 16 V matches how the fleet records
this part.

Not yet consistent: the board was saved before the 0805 change, so C1-C4
are still 1210 on the PCB. Schematic parity flags the footprint and the
MPN, and Update PCB from Schematic resolves both. DRC errors that are new
with this layout:
- C5's courtyard overlaps D1, R13 and J1.
- R1-R4 sit inside J1's courtyard. C1-C4 already did on the fabbed board.
- One GND via is inside the board-edge clearance.

Co-Authored-By: Claude Opus 5.5 <noreply@anthropic.com>
Parts:
- added C5: TCJE337M016R0050, Footprints:CAPMP7.6X4.3_3.1N_KEM, F.Cu at (90.2, 72.2)
- added R1: 330, Resistor_SMD:R_0402_1005Metric, F.Cu at (80.4, 79.0)
- added R2: 330, Resistor_SMD:R_0402_1005Metric, F.Cu at (83.8, 79.1)
- added R3: 330, Resistor_SMD:R_0402_1005Metric, F.Cu at (89.0, 79.1)
- added R4: 330, Resistor_SMD:R_0402_1005Metric, F.Cu at (94.9, 79.3)
- C1, C2, C3, C4: value 100 uF -> 22 uF
- moved D1 3.33 mm to (95.2, 70.7)
- moved R13 1.29 mm to (95.2, 71.6), turned to 0 degrees
Connections:
- J1 pad 2: Servo4 -> Servo4_In
- J1 pad 3: Servo3 -> Servo3_In
- J1 pad 4: Servo2 -> Servo2_In
- J1 pad 5: Servo1 -> Servo1_In
Routing:
- net Servo4_In: track 0.00 -> 5.43 mm
- net Servo4: track 9.83 -> 4.72 mm
- net Servo3: track 9.22 -> 5.16 mm
- net Servo3_In: track 0.00 -> 3.81 mm
- net Servo1: track 5.73 -> 2.20 mm
- net Servo2: track 8.92 -> 5.51 mm
- net GND: track 5.08 -> 1.92 mm, vias 13 -> 14
- net Servo1_In: track 0.00 -> 2.50 mm
- net Servo2_In: track 0.00 -> 2.40 mm

Commit message: hardware(servo-adapter): C1-C4 swapped to the 0805 footprint on the board
The owner's board update. Schematic parity is now clean (8 -> 0): C1-C4
are C_0805_2012Metric with CL21A226MOQNNNE on both sides. DRC reports no
unconnected items.

Zone fills are STALE: the F.Cu GND pour was not refilled after the swap.
The stored copper still touches pad 1 (LiPoPos) of C1-C4, which DRC reports
as 4 clearance + 4 solder-mask-bridge errors and which would plot as a
LiPoPos-GND short. A refill clears exactly those 8 and adds nothing
(checked on a scratch copy). Refill before any fab output.

Co-Authored-By: Claude Opus 5.5 <noreply@anthropic.com>
Parts:
- C1, C2, C3, C4: footprint Capacitor_SMD:C_1210_3225Metric -> Capacitor_SMD:C_0805_2012Metric
