File: hardware/tinker-mantis/tinker-mantis.kicad_pcb (KiCad board)
At the start: 8 copper layers, 22.3 x 75 mm, 277 parts, among them J1 BM05B-SRSS-TB, J2 JL212R-SMT-35005BP1, J3 878321620, J4 B4B-PH-SM4-TB, J5 Conn_01x04, J6 USB4110GFA, J8 JST_B2P-VH, Q11 AONR21321, Q12 DTC123J, Q13 DTA123J, Q14 DTC123J, Q3 DTC123J, Q4 DTC123J, Q5 DTC123J, Q6 DTC123J, SW2 R-667995, SW3 R-667995, U1 FSUSB63UMX, U10 WSD20L50DN33, U11 GD5F2GQ5UEYIGR, U13 W25Q128JVYIQ, U15 ESP32-S3RH2, U16 W25Q128JVYIQ, U17 ESP32-P4NRW32, U18 TPS62152RGTR, U19 TPS259824LNRGET, U2 ISM6HG256XTR, U20 TLV62569DRLR, U21 TPS2121RUXR, U22 AANI-CH-0070, U23 INA230AIRGTR, U26 TPS22811LRPWR, U27 TPS22810DRVR, U28 TPS22811LRPWR, U29 TPS22810DRVR, U3 QMC5883P, U30 TPS22810DRVR, U4 BMP581, U47 TPS61094DSS, U6 WSD20L50DN33, U7 WSD20L50DN33, U8 WSD20L50DN33, U9 AON7534, Y1 ABS07-32.768KHZ-T, Y2 ECS-400-10-37B2-CKY-TR, Y3 ABS07-32.768KHZ-T, Y4 ECS-400-10-37B2-CKY-TR

Commit message: hardware(Tinker-Mantis): the V10 layout review and its fixes -- return vias, pin-1 marks, INT1 off the P4 crystal, V10 fab notes, and a glitch filter on the OC's I2C slave
The owner's V10 layout as saved on 2026-09-29, with the fixes from the 2026-09-29 layout review
(hardware/tinker-mantis/layout-review-2026-09-29.md). The items left for a future revision are
tracked in #1556.

Board (tinker-mantis.kicad_pcb):
- The owner's 2026-09-29 saves: VDD3P3 widened, antenna-cutout stitching, the C53 and V_SCAP_ADC
  vias, an In2 ribbon re-route, ESP_VDD_HP widened, and U18/U27/U29/U30 updated from the library.
- Six GND return vias. The U4 via moves into pad 9, and the via under U2 is deleted.
- FID3 moves to the top-left corner of the bottom side. R41, R47 and R22 get thermal relief on
  their GND pads. C27 and C145 are swapped.
- ISM6HG256_INT1 is re-routed away from the P4 crystal. Its run within 0.30 mm of XTAL_N goes
  from 4.50 mm to 0.07 mm.
- Pin-1 dots are added to the board copies of U17, U15, U23, U1, U6-U10, J1 and J3; U2, U26 and
  U28's dots move to where they print. S1's "F" moves clear of C44, and two orphan "+" marks are
  deleted.
- The OC_ARM_EN via moves clear of J2.5. The dangling SERVO_ACT stub is deleted, and D9 and U47
  point at the repo's 3D models.
- User.Drawings holds block A of the new fab notes.

Project: missing_courtyard, pth/npth_inside_courtyard and footprint_type_mismatch are raised
from ignore to warning (#1365 E).

Library: U_LGA-14L_2p5X3p0X0p83_STM's pin-1 circle moves from B.SilkS to F.SilkS. The Beetle's
U2 now reports lib_footprint_mismatch until an Update Footprint; its dot prints on the bottom too.

Docs:
- FABRICATION-NOTES.md is rewritten for V10: block A for the fab (stack, ENIG, filled and capped
  vias, mask dams, and A9, no tabs on the top edge) and block B for assembly (0.08 mm foil,
  reflow order, C130, J3's pin 1 and the mounting hardware).
- SOLDER-PASTE-CONVENTION.md gets a tinker-mantis row.
- WORKLIST M-17 re-affirm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
Parts:
- moved FID3 29.0 mm to (73.3, 97.3)
- moved C145 0.97 mm to (83.3, 150.1)
- moved C27 0.97 mm to (84.3, 150.1)
Routing:
- net CAM_IMON: track 60.9 -> 53.7 mm
- net PYRO1_FIRE: track 83.5 -> 79.8 mm
- net M_SCK: track 26.8 -> 23.1 mm
- net P4_EN_HOLD: track 77.8 -> 74.9 mm
- net PYRO1_CONT: track 69.0 -> 71.6 mm
- net PG_RAIL: track 23.4 -> 25.0 mm
- net Net-(R54-Pad1): track 83.3 -> 84.6 mm
- net PYRO2_FIRE: track 65.2 -> 66.4 mm
- net FC_ARM: track 65.2 -> 66.4 mm
- net LoRa_ACT: track 87.5 -> 86.4 mm
- net OUT_D+: track 17.1 -> 18.1 mm
- net IND_2: track 67.2 -> 68.2 mm
- net BMP585_CS: track 11.0 -> 10.2 mm
- net LoRa_RX: track 81.8 -> 82.5 mm
- net PYRO2_CONT: track 103.3 -> 102.6 mm
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Other:
- board text added: "TINKERROCKET TINKER-MANTIS (ROCKET COMPUTER V10) - FABRICATION NOTES BOARD 22.35 x 75.00 mm, 8 LAYER, 1.630 mm STACK. TWO INTERNAL SLOTS 8.0 x 3.0 mm, ROUTED; THEY ARE PART OF THE OUTLINE. A1. STACKUP: JLCPCB JLC08161H-2116, EIGHT LAYER, 1.630 mm. 1 oz OUTER / 0.5 oz INNER. BUILD TO THIS TEMPLATE. OUTER PREPREG 2116 AT 0.1164 mm (er 4.16), CORES 0.300 mm (er 4.41), INNER PREPREG 1080 x2 AT 0.1528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"
- board text removed: "TINKERROCKET ROCKET COMPUTER - FABRICATION NOTES BOARD 22.35 x 75.00 mm, 6 LAYER, 1.546 mm STACK. 1. STACKUP: JLCPCB JLC06161H-3313, 1 oz OUTER / 0.5 oz INNER. BUILD TO THIS TEMPLATE. JLC LISTS TWO TEMPLATES UNDER THIS NAME - USE THE DEFAULT, WITH THE 2116 MIDDLE PREPREG AT 0.1164 mm (NOT THE 0.1088 mm VARIANT). 2. SURFACE FINISH: ENIG. REQUIRED FOR THE 0.35 mm PITCH QFN-104 (U17), THE 0.4 mm QFN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"
