File: hardware/tinker-mantis/tinker-mantis.kicad_sch (KiCad schematic)
At the start: 18 parts, among them U1 FSUSB63UMX

Commit message: hardware(Tinker-Base, Mantis, Beetle): J2 becomes the GCT USB4110-GF-A the other boards use, placed where the HRO sat, and S1's maker is C&K
Tinker-Base J2 moves from the HRO TYPE-C-31-M-12 to the GCT USB4110-GF-A that the
Mantis, Beetle, LoRa and Space Bug boards use (owner, 2026-10-03).

- Schematic: J2 already used the Custom:USB4110GFA symbol. Only its footprint and
  part fields change (Value, MF, MP, MPN, Mfr, Description_1), copied from the
  Mantis/Beetle/LoRa instances. Both footprints name their pads after the
  symbol's pin numbers, so the netlist is identical.
- PCB: the GCT footprint sits where the HRO did, with its front face on the HRO's
  (1.11 mm past the board edge). The signal pads land on the same x positions,
  the pegs move 0.03 mm, and every existing track still ends on a pad. The SMD
  shell tabs connect solid to the F.Cu ground pour. Two new GND vias between the
  tabs tie the shell to In1.Cu and B.Cu ground, which the HRO's plated slots
  reached directly. BT2's + pad stays 0.84 mm from J2. DRC: 0 errors (24
  silkscreen/library warnings, 26 before), 0 unconnected, 0 parity issues; the
  fills are a refill fixed point.
- FABRICATION-NOTES: J2 is fully SMT now. The slot annular-ring minimum and the
  hand-solder instructions go; the V1 HRO procedure is kept in the "why" notes.
  The README status records the change and the V1 order.
- The V1 boards ordered on 2026-09-29 (tag tinker-base-v1.0.0) have the HRO land
  and still take TYPE-C-31-M-12.

S1 slide switch (JS202011JCQN) on the Mantis and Beetle: Mfr Same Sky (CUI) -> C&K.
It is a C&K JS-series part, and its SnapEDA MF/MANUFACTURER fields already said
so. Run Update PCB on those two boards to carry the field over.

bom.csv rows were updated and checked against each schematic designator by
designator; tools/check_board_parity.py and tools/check_docs.py pass.

Co-Authored-By: Claude Opus 5.5 <noreply@anthropic.com>
Parts:
- S1: Mfr Same Sky (CUI) -> C&K
Changed lines of the file:
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@@
 			)
 		)
-		(property "Mfr" "Same Sky (CUI)"
+		(property "Mfr" "C&K"
 			(at 36.83 88.9 0)
 			(hide yes)
