File: hardware/tinker-mantis/esp32s3_outputs.kicad_sch (KiCad schematic)
At the start: 46 parts, among them J5 Conn_01x04, SW3 R-667995, U11 GD5F2GQ5UEYIGR, U13 W25Q128JVYIQ, U15 ESP32-S3RH2, U22 AANI-CH-0070, U29 TPS22810DRVR, Y1 ABS07-32.768KHZ-T, Y2 ECS-400-10-37B2-CKY-TR

Commit message: hardware(Tinker-Beetle V2, Tinker-Mantis V11, LoRa V4): the ESP32-S3s take their boot flash in the package, and the Beetle's V2 work to date (#1684)
Every in-work board's ESP32-S3RH2 + external W25Q128JVYIQ becomes an
ESP32-S3FH4R2 (4 MB quad flash + the same 2 MB quad PSRAM in the package,
same QFN-56 and pinout). The boot NOR and its 100 nF go; pads 30-35 carry
no-connect flags. The S3FN8 was not used: the Beetle FC's raw-GNSS filter
keeps ~219 KB in PSRAM and the OC's log ring is 512 KB there.

- Tinker-Beetle V2: U15/U32 -> FH4R2; U13, U33, C26, C115 removed.
- Tinker-Mantis V11: out computer U15 -> FH4R2; U13, C26 removed. The P4's
  boot flash U16 stays (no P4 has in-package flash).
- LoRa daughterboard V4: U28 -> FH4R2; U22, C18 removed. radio_board already
  declares 4 MB with PSRAM off, so its firmware needs no change.

The Beetle folder also carries the rest of its uncommitted V2 work, which
shares these files: TPS1HC08-Q1 eFuse pyro switches (U6-U8, U10, R144-R147;
Q3-Q6 gone), the PX1105R (U12) with its GVLB208.A antenna, the MMC5983MA
magnetometer on the sensor SPI, the Molex 0479480001 BLE antenna, the WAGO
2601-1105 battery terminal (J2), the SHOU HAN vertical USB-C (J6), no FC
32.768 kHz crystal (Y3), the BAT54XV2T1G power-switch OR (D9/D12) and the
BOM consolidation. The libraries gain the symbols and footprints those use
(MMC5983MA's GND pins become power inputs).

Checked: tools/check_board_parity.py passes on every board. ERC and
netlists match the working copy they came from. PCB DRC with schematic
parity: LoRa 0 unconnected, Mantis 4, Beetle 190 (its V2 layout is in
progress). Firmware for the 4 MB partition tables (Beetle V2, Mantis V11
OC) is not part of this.

Not included: Tinker-Base V2 (FH4R2 + U23 log flash, GCT USB4110-GF-A J2,
330 ohm LED resistors). Its PCB has not been updated yet, so it fails the
board-parity check.

Co-authored-by: Claude Opus 5.5 <noreply@anthropic.com>
Parts:
- removed C26: 100 nF, Capacitor_SMD:C_0402_1005Metric, symbol Device:C
- removed U13: W25Q128JVYIQ, Footprints:24-WLCSP_Y_WIN, symbol Custom:W25Q128JVYIQ
- U15: value ESP32-S3RH2 -> ESP32-S3FH4R2; MPN ESP32-S3RH2 -> ESP32-S3FH4R2
Connections:
- net OUT_SPI_CLK: no longer names the net of U15.33 (SPICLK)
- net OUT_SPI_CS0: no longer names the net of U15.32 (SPICS0)
- net OUT_SPI_D: no longer names the net of U15.35 (SPID)
- net OUT_SPI_HD: no longer names the net of U15.30 (SPIHD)
- net OUT_SPI_Q: no longer names the net of U15.34 (SPIQ)
- net OUT_SPI_WP: no longer names the net of U15.31 (SPIWP)
- no-connect marks 10 -> 16
