File: hardware/gnss-sdr-dev/gnss-sdr-dev.kicad_sch (KiCad schematic)
At the start: 9 parts

Commit message: hardware(gnss-sdr-dev): the rest of the board routed except the P4's new pins, and the Mantis flight-data NAND added -- FPGA fanout and supplies, sample lines and clock, power entry, IMU, USB-HS connector side; silkscreen references hidden
Silkscreen:
- Reference designators hidden on every part, the new ones included.

Flight-data flash (new sheet "Data flash", flash.kicad_sch):
- U701 is the Mantis U11 part and footprint, GD5F2GQ5UEYIGR (2 Gbit SPI NAND, WSON-8 8x6).
- R701 pulls CS up through reset and boot. R702/R703 pull HOLD#/WP# up, as on the Mantis. C701 is 100 nF.
- It uses the P4's four free GPIOs: GPIO0 = CS, GPIO9 = MISO, GPIO33 = SCK, GPIO34 = MOSI.
  - GPIO34 is the P4's JTAG-source strap, so it only drives the NAND's input and has no pull.
- ERC: 0 errors. The two new warnings are pin-type warnings like those already on the sheet.
- Placed east of the P4 at (147.6, 139). Its locals are routed; its P4 links are not (see below).

Rules:
- New 0.1 mm clearance inside U501's courtyard (0.8 mm BGA), written like the fine-pitch rule for U6/U7/U9/U10.
- Zone fills keep the board default.

Planes:
- +3V3_MCU plane on In4 over the digital side.
- +1V1_FPGA island on B.Cu: the ball field, a finger to each core decoupler, and a strip east of R501-R512 down to the 1.1 V buck.

FPGA:
- Via-in-pad on every supply, ground and interior signal ball.
- Fixed escape lanes run between the ball columns below and south-west of the field.
- Routed:
  - 1.1 V, 2.5 V (on In4, along the east edge) and VCCAUX.
  - The eight sample lines from the shield's escape vias, with their DNP edge-rate shunts.
  - The 27 MHz sample clock out of the shield.
  - Logic-analyzer header (13 of 14 lines), JTAG, status LEDs, config flash and its pull-ups.
  - The CFG_0/1/2 mode straps, on B.Cu under the strap resistors.

Power entry and the west:
- Battery/host connector, input filter, VSS/VSYS/+BATT, VIN to the GNSS LDO and on to the P4 buck's filter.
- GNSS LDO output, +3V3_GNSS and +1V8_LNA, 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
Other:
- added sheet Data flash (flash.kicad_sch)
- note added: "From the Tinker-Mantis: 2 Gbit SPI NAND for flight logging, on the P4's four free GPIOs"
Changed lines of the file:
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@@
+		)
+	)
+	(text "From the Tinker-Mantis: 2 Gbit SPI NAND for flight\nlogging, on the P4's four free GPIOs"
+		(exclude_from_sim no)
+		(at 158.75 213.36 0)
+		(effects
+			(font
+				(size 1.5 1.5)
+			)
+			(justify left bottom)
+		)
+	)
+	(sheet
+		(at 154.94 203.2)
+		(size 101.6 27.94)
+		(exclude_from_sim no)
+		(in_bom yes)
+		(on_board yes)
+		(dnp no)
+		(fields_autoplaced yes)
+		(stroke
+			(width 0.1524)
+			(type solid)
+		)
+		(fill
+			(color 0 0 0 0)
+		)
+		(property "Sheetname" "Data flash"
+			(at 154.94 201.9 0)
+			(show_name no)
+			(do_not_autoplace no)
+			(effects
+				(font
+					(size 2.5 2.5)
+					(thickness 0.6)
+					(bold yes)
+				)
+				(justify left bottom)
+			)
+		)
+		(property "Sheetfile" "flash.kicad_sch"
+			(at 154.94 232.44 0)
+			(show_name no)
+			(do_not_autoplace no)
+			(effects
+				(font
+					(size 1.27 1.27)
+				)
+				(justify left top)
+			)
+		)
+		(instances
+			(project "gnss-sdr-dev"
+				(path "/18c5be81-d8c2-4b08-92bf-000bb4e79507"
+					(page "12")
+				)
+			)
 		)
 	)

Commit message: hardware(gnss-sdr-dev): one USB-C port through a Mantis-style FSUSB63 switch, USB-C #1's chain removed; part values hidden; the owner's placement in progress
USB (owner: put the two USB ports on the Mantis's switch, remove the unused parts; the owner places the new ones):
- One USB-C, J601, keeps its USBLC6 ESD (U601) and common-mode choke (FL601).
  - J601's chain is the one rated for 480 Mbps. USB-C #1's SP0503 ESD has too much capacitance for high speed.
- U602 FSUSB63UMX sits after FL601:
  - HSD2 -> USB_D+/USB_D- -> R22/R23 -> the P4's USB-Serial/JTAG (flashing, console).
  - HSD3 -> USB_HS_DP/USB_HS_DM -> the P4's HS PHY (sample streaming).
  - HSD1 is unused.
- As on the Mantis (U1, S1, R1-R3, C1):
  - SEL1 is pulled up by R603 (100 k).
  - SEL0 is pulled up by R604 (100 k) and grounded by slide switch S601 (JS202011JCQN). Closed selects USB-Serial/JTAG; open selects the HS PHY.
  - VCC comes from +3V3_MCU through R605 (22 ohm) with C602 (100 nF).
- Removed: J5 (USB-C #1), D7, R20, R21, C73 and D9, plus the 94 tracks and vias that only served them (all in J5's corner).
  - The USB sheet keeps D8, the battery OR into VSYS.
- Text blocks reworded to match, at the owner's request.
- Not yet on the board: U602, S601, R603-R605 and C602 come in with the owner's Update PCB.
  - Until then tools/check_board_parity.py fails on those six. The owner chose to push now.

Board:
- Value fields hidden on every footprint. They were all on F.Fab, so the silkscreen is unchanged.
- The owner's placement in progress (their 19:48 save): 33 parts moved, their tracks ripped up.
  - J601's chain moves to the right edge.
  - Also moved: the 1.1 V buck and its parts, the NAND, the IMU and its caps, and the FPGA configuration pull-ups.
- DRC: 4 errors, all from the in-progress placement:
  - R512 pad 2 against the GND via at (160.15, 134.4);
  - C71/C72 clearance and courtyards;
  - R501/R503 courtyards.
- Parity: the six new parts.

Checks: ERC 0 errors, 16 warnings (6 fewer than bef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
Other:
- note added: "From the Space Bug M8T: battery OR into VSYS"
- note added: "USB-C through an FSUSB63 switch: USB-Serial/JTAG (flashing) or the HS PHY (sample streaming)"
- note removed: "From the Space Bug M8T: USB-C #1, USB-Serial/JTAG (flashing), VBUS into VSYS"
- note removed: "USB-C #2 on the P4 high-speed PHY: sample streaming"
Changed lines of the file:
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@@
 		)
 	)
-	(text "From the Space Bug M8T: USB-C #1, USB-Serial/JTAG\n(flashing), VBUS into VSYS"
+	(text "From the Space Bug M8T: battery OR into VSYS"
 		(exclude_from_sim no)
 		(at 158.75 162.56 0)
@@
 		)
 	)
-	(text "USB-C #2 on the P4 high-speed PHY:\nsample streaming"
+	(text "USB-C through an FSUSB63 switch: USB-Serial/JTAG\n(flashing) or the HS PHY (sample streaming)"
 		(exclude_from_sim no)
 		(at 283.21 162.56 0)
