File: hardware/gnss-sdr-dev/fpga_power.kicad_sch (KiCad schematic)
At the start: 28 parts, among them U501 LFE5U-25F-6BG256

Commit message: hardware(gnss-sdr-dev): the design review's before-assembly fixes -- FL401 a 2 A shielded power-line choke, U601 a 0.5 pF HS ESD array with a VBUS TVS, and the value fixes
The boards were not ordered yet, so the copper can still change. Schematic only: the PCB is not updated yet (the
owner runs Update PCB and places FL401, U601 and the new D602), so DRC parity stays red until then.

Parts:
- FL401: Bourns SRF3225TP-501Y (2 A, 0.1 ohm max, 60 V, 500 ohm at 100 MHz, -40 to +105 C, shielded) replaces the
  DLW21SN670HQ2L, a 320 mA USB data-line choke that carried the whole board's input current. No 0805 choke reaches
  0.8 A. New footprint FIL_SRF3225TP (Bourns layout), a CadQuery model and a Custom symbol.
- U601: TI TPD4E05U06DQAR, 0.5 pF. The ESP32-P4 guide allows 1 pF on the high-speed lines; the USBLC6-2SC6 was
  2.5-3.5 pF. USON-10 with D+ on pins 1 and 10 and D- on 2 and 9, for flow-through routing; channel 2 is unused.
- D602 (new): LESD5D5.0CT1G on VBUS_HS, as on Espressif's ESP32-P4-Function-EV-Board. The new U601 has no VBUS pin.
- C403 2.2 -> 22 nF: the GNSS LDO now ramps after the FPGA rails. The front ends no longer drive the ECP5's left
  banks (not hot-socket rated) while those are unpowered.
- R104 10 -> 2.2 ohm: at least 3.15 V at the antenna at 30 mA, and no overload into a shorted feed.
- R503/R504 1 k -> 0 ohm: the configuration straps Lattice asks for (< 500 ohm).
- FB501 470 -> 120 ohm bead (BLM18PG121SN1D), inside the ECP5 checklist's range.
- C105 1 -> 100 nF (the BGA524N6 asks for > 10 nF); C408 1 -> 2.2 uF on the LP5907 output.
- U301 (MAX2771) marked do-not-fit: owner stock, fitted by hand.
- U701's Datasheet field now points at the GD5F2GQ5UE datasheet.
- FABRICATION-NOTES.md: U8 joins the parts with no pin-1 mark, U301 joins the do-not-fit list, and the U9 sentence is
  corrected (U9 makes +3V3_MCU; the FPGA core buck is U403).

ERC: 0 errors and the same 15 warnings. The netlist changes only for the parts above.

The bring-up and firmware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
Parts:
- FB501: value BLM18PG471SN1D -> BLM18PG121SN1D; symbol Custom:BLM18PG471SN1D -> Custom:BLM18PG121SN1D; MPN BLM18PG471SN1D -> BLM18PG121SN1D
Changed lines of the file:
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@@
 	)
 	(symbol
-		(lib_id "Custom:BLM18PG471SN1D")
+		(lib_id "Custom:BLM18PG121SN1D")
 		(at 43.18 55.88 0)
 		(unit 1)
@@
 			)
 		)
-		(property "Value" "BLM18PG471SN1D"
+		(property "Value" "BLM18PG121SN1D"
 			(at 43.18 59.055 0)
 			(show_name no)
@@
 			)
 		)
-		(property "Description" "Ferrite bead 470 ohm @ 100 MHz, 1 A, 0603"
+		(property "Description" "Ferrite bead 120 ohm @ 100 MHz, 2 A, 0603"
 			(at 43.18 55.88 0)
 			(hide yes)
@@
 			)
 		)
-		(property "MPN" "BLM18PG471SN1D"
+		(property "MPN" "BLM18PG121SN1D"
 			(at 43.18 55.88 0)
 			(hide yes)
