File: hardware/gnss-sdr-dev/power.kicad_sch (KiCad schematic)
At the start: 27 parts, among them J401 BM05B-SRSS-TB, U401 ADP7142ARDZ-3.3, U402 LP5907MFX-1.8, U403 TPS62A02APDDC, U404 TLV75725PDBV

Commit message: hardware(gnss-sdr-dev): the design review's before-assembly fixes -- FL401 a 2 A shielded power-line choke, U601 a 0.5 pF HS ESD array with a VBUS TVS, and the value fixes
The boards were not ordered yet, so the copper can still change. Schematic only: the PCB is not updated yet (the
owner runs Update PCB and places FL401, U601 and the new D602), so DRC parity stays red until then.

Parts:
- FL401: Bourns SRF3225TP-501Y (2 A, 0.1 ohm max, 60 V, 500 ohm at 100 MHz, -40 to +105 C, shielded) replaces the
  DLW21SN670HQ2L, a 320 mA USB data-line choke that carried the whole board's input current. No 0805 choke reaches
  0.8 A. New footprint FIL_SRF3225TP (Bourns layout), a CadQuery model and a Custom symbol.
- U601: TI TPD4E05U06DQAR, 0.5 pF. The ESP32-P4 guide allows 1 pF on the high-speed lines; the USBLC6-2SC6 was
  2.5-3.5 pF. USON-10 with D+ on pins 1 and 10 and D- on 2 and 9, for flow-through routing; channel 2 is unused.
- D602 (new): LESD5D5.0CT1G on VBUS_HS, as on Espressif's ESP32-P4-Function-EV-Board. The new U601 has no VBUS pin.
- C403 2.2 -> 22 nF: the GNSS LDO now ramps after the FPGA rails. The front ends no longer drive the ECP5's left
  banks (not hot-socket rated) while those are unpowered.
- R104 10 -> 2.2 ohm: at least 3.15 V at the antenna at 30 mA, and no overload into a shorted feed.
- R503/R504 1 k -> 0 ohm: the configuration straps Lattice asks for (< 500 ohm).
- FB501 470 -> 120 ohm bead (BLM18PG121SN1D), inside the ECP5 checklist's range.
- C105 1 -> 100 nF (the BGA524N6 asks for > 10 nF); C408 1 -> 2.2 uF on the LP5907 output.
- U301 (MAX2771) marked do-not-fit: owner stock, fitted by hand.
- U701's Datasheet field now points at the GD5F2GQ5UE datasheet.
- FABRICATION-NOTES.md: U8 joins the parts with no pin-1 mark, U301 joins the do-not-fit list, and the U9 sentence is
  corrected (U9 makes +3V3_MCU; the FPGA core buck is U403).

ERC: 0 errors and the same 15 warnings. The netlist changes only for the parts above.

The bring-up and firmware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
Parts:
- C403: value 2.2 nF -> 22 nF; MPN CC0402KRX7R9BB222 -> CL05B223KB5NNNC; Mfr Yageo -> Samsung
- C408: value 1 uF -> 2.2 uF; MPN GRM155R61A105KE15D -> CL05A225MQ5NSNC; Mfr Murata -> Samsung
- FL401: value DLW21SN670HQ2L -> SRF3225TP-501Y; footprint Footprints:FIL_DLW21SN670HQ2L -> Footprints:FIL_SRF3225TP; symbol Custom:DLW21SN670HQ2L -> Custom:SRF3225TP-501Y; MPN DLW21SN670HQ2L -> SRF3225TP-501Y; Mfr Murata -> Bourns
Changed lines of the file:
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@@
 	)
 	(symbol
-		(lib_id "Custom:DLW21SN670HQ2L")
+		(lib_id "Custom:SRF3225TP-501Y")
 		(at 160.02 60.96 0)
 		(unit 1)
@@
 			)
 		)
-		(property "Value" "DLW21SN670HQ2L"
+		(property "Value" "SRF3225TP-501Y"
 			(at 154.94 67.31 0)
 			(show_name no)
@@
 			)
 		)
-		(property "Footprint" "Footprints:FIL_DLW21SN670HQ2L"
+		(property "Footprint" "Footprints:FIL_SRF3225TP"
 			(at 160.02 60.96 0)
 			(hide yes)
@@
 			)
 		)
-		(property "Datasheet" ""
+		(property "Datasheet" "https://www.bourns.com/docs/Product-Datasheets/SRF3225TP.pdf"
 			(at 160.02 60.96 0)
 			(hide yes)
@@
 			)
 		)
-		(property "Description" "Common-mode choke on the host supply/return (VSYS/VSS -> VIN/GND)"
+		(property "Description" "Common-mode choke on the host supply/return (VSYS/VSS -> VIN/GND), shielded power-line type, 2 A"
 			(at 160.02 60.96 0)
 			(hide yes)
@@
 			)
 		)
-		(property "MPN" "DLW21SN670HQ2L"
+		(property "MPN" "SRF3225TP-501Y"
 			(at 160.02 60.96 0)
 			(hide yes)
@@
 			)
 		)
-		(property "Mfr" "Murata"
+		(property "Mfr" "Bourns"
 			(at 160.02 60.96 0)
 			(hide yes)
@@
 			)
 		)
-		(property "Value" "2.2 nF"
+		(property "Value" "22 nF"
 			(at 63.5 144.78 0)
 			(show_name no)
@@
 			)
 		)
-		(property "Description" "Capacitor 2.2 nF X7R"
+		(property "Description" "Capacitor 22 nF X7R"
 			(at 60.96 143.51 0)
 			(hide yes)
@@
 			)
 		)
-		(property "MPN" "CC0402KRX7R9BB222"
+		(property "MPN" "CL05B223KB5NNNC"
 			(at 60.96 143.51 0)
 			(hide yes)
@@
 			)
 		)
-		(property "Mfr" "Yageo"
+		(property "Mfr" "Samsung"
 			(at 60.96 143.51 0)
 			(hide yes)
@@
 			)
 		)
-		(property "Value" "1 uF"
+		(property "Value" "2.2 uF"
 			(at 101.6 180.34 0)
 			(show_name no)
@@
 			)
 		)
-		(property "Description" "Capacitor 1 uF X5R"
+		(property "Description" "Capacitor 2.2 uF X5R"
 			(at 99.06 179.07 0)
 			(hide yes)
@@
 			)
 		)
-		(property "MPN" "GRM155R61A105KE15D"
+		(property "MPN" "CL05A225MQ5NSNC"
 			(at 99.06 179.07 0)
 			(hide yes)
@@
 			)
 		)
-		(property "Mfr" "Murata"
+		(property "Mfr" "Samsung"
 			(at 99.06 179.07 0)
 			(hide yes)

Commit message: hardware: the 1 uF 0402 caps consolidate on the 16 V CL05A105KO5NNNC, with the pending part and layout work
Every GRM155R61A105KE15D (Murata, 10 V X5R) becomes the Samsung CL05A105KO5NNNC (16 V X5R) on
space-bug-m8t, gnss-sdr-dev and the legacy gnss-px1105r board -- 34 symbols and their 34 footprints.
Same 0402 footprint, so only the MPN and Mfr change. The higher-rated part is already the 1 uF used
on the Tinker boards, so the BOMs now carry one 1 uF line instead of two.

Pending work committed alongside:
- space-bug-m8t: the 10 uF bulk caps go to CL21A226MOQNNNE, added CL05A106MQ5NUNC, RC0402FR-071KL and
  R-667995 parts, schematic, layout and DRC rule updates, and the new FABRICATION-NOTES.md
- gnss-sdr-dev: the 5.1 nH inductors go from LQG15HS5N1S02D to LQW15AN5N1C00D, added 1 k and 100 k
  resistors, and schematic and layout updates
- legacy gnss-px1105r: the 10 uF caps go to CL21A226MOQNNNE, plus schematic and layout updates
- tinker-beetle: the 390 pF caps go to GRM1555C1H391JA01D, the 100 k resistors to RC0402FR-07100KL,
  and the 2.2 uH inductor from XGL4020-222ME to SRP4020FA-2R2M
- gnss-sam10m8-18mm-hv: the 100 pF cap goes from CL05C101JB5NNNC to GRM1555C1H101JA01D
- the Taoglas CGGBP.25.4.A.02 antenna footprint, and project-file housekeeping

Co-Authored-By: Claude Opus 5.5 <noreply@anthropic.com>
Parts:
- added R405: 100 k, Resistor_SMD:R_0402_1005Metric, symbol Device:R_US
- C407, C412, C413: MPN GRM155R61A105KE15D -> CL05A105KO5NNNC; Mfr Murata -> Samsung
Connections:
- net +3V3_MCU: now also R405.1
- net +BATT: now also D401.1 (A1), FL401.1
- net VSYS: now also C401.1, C402.1, U401.7 (VIN), U401.8 (VIN__1); no longer D401.1 (A1), FL401.1
- net GNSS_EN: now reaches U403.5 (PG)
- net GNSS_EN: now also U401.5 (EN), R405.2
- removed net VIN: C401.1, C402.1, FL401.2, U401.5 (EN), U401.7 (VIN), U401.8 (VIN__1)
- new net +BATT_F: FL401.2
- no-connect marks 3 -> 2
Changed lines of the file:
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@@
 	)
 	(junction
-		(at 175.26 55.88)
-		(diameter 0)
-		(color 0 0 0 0)
-	)
-	(junction
 		(at 146.05 121.92)
 		(diameter 0)
@@
 	)
 	(junction
-		(at 63.5 124.46)
-		(diameter 0)
-		(color 0 0 0 0)
-	)
-	(junction
 		(at 50.8 121.92)
 		(diameter 0)
@@
 		(at 86.36 177.8)
 	)
-	(no_connect
-		(at 261.62 134.62)
-	)
 	(wire
 		(pts
@@
 	(wire
 		(pts
-			(xy 38.1 121.92) (xy 50.8 121.92)
-		)
-		(stroke
-			(width 0)
-			(type default)
-		)
-	)
-	(wire
-		(pts
 			(xy 81.28 185.42) (xy 81.28 187.96)
 		)
@@
 	(wire
 		(pts
-			(xy 175.26 55.88) (xy 182.88 55.88)
-		)
-		(stroke
-			(width 0)
-			(type default)
-		)
-	)
-	(wire
-		(pts
 			(xy 68.58 78.74) (xy 78.74 78.74)
 		)
@@
 	(wire
 		(pts
-			(xy 63.5 124.46) (xy 63.5 137.16)
-		)
-		(stroke
-			(width 0)
-			(type default)
-		)
-	)
-	(wire
-		(pts
 			(xy 231.14 185.42) (xy 243.84 185.42)
 		)
@@
 		)
 	)
-	(wire
-		(pts
-			(xy 170.18 55.88) (xy 175.26 55.88)
-		)
-		(stroke
-			(width 0)
-			(type default)
-		)
-	)
 	(global_label "+3V3_MCU"
 		(shape input)
@@
 			)
 		)
-		(property "Value" "VSYS"
+		(property "Value" "+BATT"
 			(at 129.54 52.07 0)
 			(show_name no)
@@
 			)
 		)
-		(property "MPN" "GRM155R61A105KE15D"
+		(property "MPN" "CL05A105KO5NNNC"
 			(at 231.14 189.23 0)
 			(hide yes)
@@
 			)
 		)
-		(property "Mfr" "Murata"
+		(property "Mfr" "Samsung"
 			(at 231.14 189.23 0)
 			(hide yes)
@@
 			)
 		)
-		(property "Description" "Common-mode choke on the host supply/return (VSYS/VSS -> VIN/GND), shielded power-line type, 2 A"
+		(property "Description" "Common-mode choke on the host connector supply/return (+BATT/VSS -> +BATT_F/GND), ahead of D8; shielded power-line type, 2 A"
 			(at 160.02 60.96 0)
 			(hide yes)
@@
 			)
 		)
-		(property "Value" "VIN"
+		(property "Value" "VSYS"
 			(at 30.48 118.11 0)
 			(show_name no)
@@
 			)
 		)
-		(property "MPN" "GRM155R61A105KE15D"
+		(property "MPN" "CL05A105KO5NNNC"
 			(at 269.24 189.23 0)
 			(hide yes)
@@
 			)
 		)
-		(property "Mfr" "Murata"
+		(property "Mfr" "Samsung"
 			(at 269.24 189.23 0)
 			(hide yes)
@@
 			)
 		)
-		(property "MPN" "GRM155R61A105KE15D"
+		(property "MPN" "CL05A105KO5NNNC"
 			(at 60.96 179.07 0)
 			(hide yes)
@@
 			)
 		)
-		(property "Mfr" "Murata"
+		(property "Mfr" "Samsung"
 			(at 60.96 179.07 0)
 			(hide yes)
@@
 	(symbol
 		(lib_id "power:PWR_FLAG")
-		(at 175.26 55.88 0)
+		(at 44.45 121.92 0)
 		(unit 1)
 		(body_style 1)
@@
 		(fields_autoplaced yes)
 		(property "Reference" "#FLG_Power_9"
-			(at 175.26 62.23 0)
+			(at 44.45 128.27 0)
 			(hide yes)
 			(show_name no)
@@
 		)
 		(property "Value" "PWR_FLAG"
-			(at 175.26 52.07 0)
+			(at 44.45 118.11 0)
 			(show_name no)
 			(do_not_autoplace no)
@@
 		)
 		(property "Footprint" ""
-			(at 175.26 55.88 0)
+			(at 44.45 121.92 0)
 			(hide yes)
 			(show_name no)
@@
 		)
 		(property "Datasheet" ""
-			(at 175.26 55.88 0)
+			(at 44.45 121.92 0)
 			(hide yes)
 			(show_name no)
@@
 		)
 		(property "Description" ""
-			(at 175.26 55.88 0)
+			(at 44.45 121.92 0)
 			(hide yes)
 			(show_name no)
@@
 			)
 		)
-		(property "Value" "VIN"
+		(property "Value" "+BATT_F"
 			(at 182.88 52.07 0)
 			(show_name no)
@@
 		)
 	)
+	(label "GNSS_EN"
+		(at 63.5 137.16 90)
+		(effects
+			(font
+				(size 1.27 1.27)
+			)
+			(justify left bottom)
+		)
+	)
+	(wire
+		(pts
+			(xy 261.62 134.62) (xy 264.16 134.62)
+		)
+		(stroke
+			(width 0)
+			(type default)
+		)
+	)
+	(wire
+		(pts
+			(xy 264.16 134.62) (xy 264.16 144.78)
+		)
+		(stroke
+			(width 0)
+			(type default)
+		)
+	)
+	(label "GNSS_EN"
+		(at 264.16 144.78 0)
+		(effects
+			(font
+				(size 1.27 1.27)
+			)
+			(justify left bottom)
+		)
+	)
+	(symbol
+		(lib_id "Device:R_US")
+		(at 43.18 146.05 90)
+		(unit 1)
+		(body_style 1)
+		(exclude_from_sim no)
+		(in_bom yes)
+		(on_board yes)
+		(in_pos_files yes)
+		(dnp no)
+		(property "Reference" "R405"
+			(at 43.18 142.24 90)
+			(show_name no)
+			(do_not_autoplace no)
+			(effects
+				(font
+					(size 1.27 1.27)
+				)
+			)
+		)
+		(property "Value" "100 k"
+			(at 43.18 149.86 90)
+			(show_name no)
+			(do_not_autoplace no)
+			(effects
+				(font
+					(size 1.27 1.27)
+				)
+			)
+		)
+		(property "Footprint" "Resistor_SMD:R_0402_1005Metric"
+			(at 43.18 146.05 0)
+			(hide yes)
+			(show_name no)
+			(do_not_autoplace no)
+			(effects
+				(font
+					(size 1.27 1.27)
+				)
+			)
+		)
+		(property "Datasheet" ""
+			(at 43.18 146.05 0)
+			(hide yes)
+			(show_name no)
+			(do_not_autoplace no)
+			(effects
+				(font
+					(size 1.27 1.27)
+				)
+			)
+		)
+		(property "Description" "Resistor 100 k"
+			(at 43.18 146.05 0)
+			(hide yes)
+			(show_name no)
+			(do_not_autoplace no)
+			(effects
+				(font
+					(size 1.27 1.27)
+				)
+			)
+		)
+		(property "MPN" "RC0402FR-07100KL"
+			(at 43.18 146.05 0)
+			(hide yes)
+			(show_name no)
+			(do_not_autoplace no)
+			(effects
+				(font
+					(size 1.27 1.27)
+				)
+			)
+		)
+		(property "Mfr" "Yageo"
+			(at 43.18 146.05 0)
+			(hide yes)
+			(show_name no)
+			(do_not_autoplace no)
+			(effects
+				(font
+					(size 1.27 1.27)
+				)
+			)
+		)
+		(pin "1"
+		)
+		(pin "2"
+		)
+		(instances
+			(project "gnss-sdr-dev"
+				(path "/18c5be81-d8c2-4b08-92bf-000bb4e79507/ebe8985f-054b-42ea-8c33-d916c783b295"
+					(reference "R405")
+					(unit 1)
+				)
+			)
+		)
+	)
+	(label "GNSS_EN"
+		(at 46.99 146.05 0)
+		(effects
+			(font
+				(size 1.27 1.27)
+			)
+			(justify left bottom)
+		)
+	)
+	(global_label "+3V3_MCU"
+		(shape input)
+		(at 39.37 146.05 180)
+		(fields_autoplaced yes)
+		(effects
+			(font
+				(size 1.27 1.27)
+			)
+			(justify right)
+		)
+		(property "Intersheetrefs" "${INTERSHEET_REFS}"
+			(at 39.37 146.05 0)
+			(hide yes)
+			(show_name no)
+			(do_not_autoplace no)
+			(effects
+				(font
+					(size 1.27 1.27)
+				)
+				(justify right)
+			)
+		)
+	)
+	(wire
+		(pts
+			(xy 170.18 55.88) (xy 182.88 55.88)
+		)
+		(stroke
+			(width 0)
+			(type default)
+		)
+	)
+	(wire
+		(pts
+			(xy 38.1 121.92) (xy 44.45 121.92)
+		)
+		(stroke
+			(width 0)
+			(type default)
+		)
+	)
+	(wire
+		(pts
+			(xy 44.45 121.92) (xy 50.8 121.92)
+		)
+		(stroke
+			(width 0)
+			(type default)
+		)
+	)
+	(junction
+		(at 44.45 121.92)
+		(diameter 0)
+		(color 0 0 0 0)
+	)
 )
