File: hardware/gnss-sdr-dev/rf_frontend.kicad_sch (KiCad schematic)
At the start: 35 parts, among them J101 CON-SMA-EDGE-S, U101 BGA524N6, U102 BGA855N6, U103 TPS2553DBV

Commit message: hardware(gnss-sdr-dev): the design review's before-assembly fixes -- FL401 a 2 A shielded power-line choke, U601 a 0.5 pF HS ESD array with a VBUS TVS, and the value fixes
The boards were not ordered yet, so the copper can still change. Schematic only: the PCB is not updated yet (the
owner runs Update PCB and places FL401, U601 and the new D602), so DRC parity stays red until then.

Parts:
- FL401: Bourns SRF3225TP-501Y (2 A, 0.1 ohm max, 60 V, 500 ohm at 100 MHz, -40 to +105 C, shielded) replaces the
  DLW21SN670HQ2L, a 320 mA USB data-line choke that carried the whole board's input current. No 0805 choke reaches
  0.8 A. New footprint FIL_SRF3225TP (Bourns layout), a CadQuery model and a Custom symbol.
- U601: TI TPD4E05U06DQAR, 0.5 pF. The ESP32-P4 guide allows 1 pF on the high-speed lines; the USBLC6-2SC6 was
  2.5-3.5 pF. USON-10 with D+ on pins 1 and 10 and D- on 2 and 9, for flow-through routing; channel 2 is unused.
- D602 (new): LESD5D5.0CT1G on VBUS_HS, as on Espressif's ESP32-P4-Function-EV-Board. The new U601 has no VBUS pin.
- C403 2.2 -> 22 nF: the GNSS LDO now ramps after the FPGA rails. The front ends no longer drive the ECP5's left
  banks (not hot-socket rated) while those are unpowered.
- R104 10 -> 2.2 ohm: at least 3.15 V at the antenna at 30 mA, and no overload into a shorted feed.
- R503/R504 1 k -> 0 ohm: the configuration straps Lattice asks for (< 500 ohm).
- FB501 470 -> 120 ohm bead (BLM18PG121SN1D), inside the ECP5 checklist's range.
- C105 1 -> 100 nF (the BGA524N6 asks for > 10 nF); C408 1 -> 2.2 uF on the LP5907 output.
- U301 (MAX2771) marked do-not-fit: owner stock, fitted by hand.
- U701's Datasheet field now points at the GD5F2GQ5UE datasheet.
- FABRICATION-NOTES.md: U8 joins the parts with no pin-1 mark, U301 joins the do-not-fit list, and the U9 sentence is
  corrected (U9 makes +3V3_MCU; the FPGA core buck is U403).

ERC: 0 errors and the same 15 warnings. The netlist changes only for the parts above.

The bring-up and firmware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
Parts:
- C105: value 1 nF -> 100 nF; MPN GRM1555C1H102JA01D -> CL05B104KO5NNNC; Mfr Murata -> Samsung
- R104: value 10 -> 2.2; MPN RC0402FR-0710RL -> RC0402FR-072R2L
Changed lines of the file:
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@@
 			)
 		)
-		(property "Value" "1 nF"
+		(property "Value" "100 nF"
 			(at 142.24 187.96 0)
 			(show_name no)
@@
 			)
 		)
-		(property "Description" "Capacitor 1 nF C0G"
+		(property "Description" "Capacitor 100 nF X7R"
 			(at 139.7 186.69 0)
 			(hide yes)
@@
 			)
 		)
-		(property "MPN" "GRM1555C1H102JA01D"
+		(property "MPN" "CL05B104KO5NNNC"
 			(at 139.7 186.69 0)
 			(hide yes)
@@
 			)
 		)
-		(property "Mfr" "Murata"
+		(property "Mfr" "Samsung"
 			(at 139.7 186.69 0)
 			(hide yes)
@@
 			)
 		)
-		(property "Value" "10"
+		(property "Value" "2.2"
 			(at 107.95 56.515 90)
 			(show_name no)
@@
 			)
 		)
-		(property "Description" "Resistor 10"
+		(property "Description" "Resistor 2.2"
 			(at 107.95 53.34 0)
 			(hide yes)
@@
 			)
 		)
-		(property "MPN" "RC0402FR-0710RL"
+		(property "MPN" "RC0402FR-072R2L"
 			(at 107.95 53.34 0)
 			(hide yes)

Commit message: hardware: the 1 uF 0402 caps consolidate on the 16 V CL05A105KO5NNNC, with the pending part and layout work
Every GRM155R61A105KE15D (Murata, 10 V X5R) becomes the Samsung CL05A105KO5NNNC (16 V X5R) on
space-bug-m8t, gnss-sdr-dev and the legacy gnss-px1105r board -- 34 symbols and their 34 footprints.
Same 0402 footprint, so only the MPN and Mfr change. The higher-rated part is already the 1 uF used
on the Tinker boards, so the BOMs now carry one 1 uF line instead of two.

Pending work committed alongside:
- space-bug-m8t: the 10 uF bulk caps go to CL21A226MOQNNNE, added CL05A106MQ5NUNC, RC0402FR-071KL and
  R-667995 parts, schematic, layout and DRC rule updates, and the new FABRICATION-NOTES.md
- gnss-sdr-dev: the 5.1 nH inductors go from LQG15HS5N1S02D to LQW15AN5N1C00D, added 1 k and 100 k
  resistors, and schematic and layout updates
- legacy gnss-px1105r: the 10 uF caps go to CL21A226MOQNNNE, plus schematic and layout updates
- tinker-beetle: the 390 pF caps go to GRM1555C1H391JA01D, the 100 k resistors to RC0402FR-07100KL,
  and the 2.2 uH inductor from XGL4020-222ME to SRP4020FA-2R2M
- gnss-sam10m8-18mm-hv: the 100 pF cap goes from CL05C101JB5NNNC to GRM1555C1H101JA01D
- the Taoglas CGGBP.25.4.A.02 antenna footprint, and project-file housekeeping

Co-Authored-By: Claude Opus 5.5 <noreply@anthropic.com>
Parts:
- L104, L105: MPN LQG15HS5N1S02D -> LQW15AN5N1C00D
Changed lines of the file:
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@@
 			)
 		)
-		(property "MPN" "LQG15HS5N1S02D"
+		(property "MPN" "LQW15AN5N1C00D"
 			(at 76.2 238.76 0)
 			(hide yes)
@@
 			)
 		)
-		(property "MPN" "LQG15HS5N1S02D"
+		(property "MPN" "LQW15AN5N1C00D"
 			(at 45.72 238.76 0)
 			(hide yes)
