File: hardware/gnss-sdr-dev/usb.kicad_sch (KiCad schematic)
At the start: 7 parts, among them J5 USB4110GFA

Commit message: hardware(gnss-sdr-dev): one USB-C port through a Mantis-style FSUSB63 switch, USB-C #1's chain removed; part values hidden; the owner's placement in progress
USB (owner: put the two USB ports on the Mantis's switch, remove the unused parts; the owner places the new ones):
- One USB-C, J601, keeps its USBLC6 ESD (U601) and common-mode choke (FL601).
  - J601's chain is the one rated for 480 Mbps. USB-C #1's SP0503 ESD has too much capacitance for high speed.
- U602 FSUSB63UMX sits after FL601:
  - HSD2 -> USB_D+/USB_D- -> R22/R23 -> the P4's USB-Serial/JTAG (flashing, console).
  - HSD3 -> USB_HS_DP/USB_HS_DM -> the P4's HS PHY (sample streaming).
  - HSD1 is unused.
- As on the Mantis (U1, S1, R1-R3, C1):
  - SEL1 is pulled up by R603 (100 k).
  - SEL0 is pulled up by R604 (100 k) and grounded by slide switch S601 (JS202011JCQN). Closed selects USB-Serial/JTAG; open selects the HS PHY.
  - VCC comes from +3V3_MCU through R605 (22 ohm) with C602 (100 nF).
- Removed: J5 (USB-C #1), D7, R20, R21, C73 and D9, plus the 94 tracks and vias that only served them (all in J5's corner).
  - The USB sheet keeps D8, the battery OR into VSYS.
- Text blocks reworded to match, at the owner's request.
- Not yet on the board: U602, S601, R603-R605 and C602 come in with the owner's Update PCB.
  - Until then tools/check_board_parity.py fails on those six. The owner chose to push now.

Board:
- Value fields hidden on every footprint. They were all on F.Fab, so the silkscreen is unchanged.
- The owner's placement in progress (their 19:48 save): 33 parts moved, their tracks ripped up.
  - J601's chain moves to the right edge.
  - Also moved: the 1.1 V buck and its parts, the NAND, the IMU and its caps, and the FPGA configuration pull-ups.
- DRC: 4 errors, all from the in-progress placement:
  - R512 pad 2 against the GND via at (160.15, 134.4);
  - C71/C72 clearance and courtyards;
  - R501/R503 courtyards.
- Parity: the six new parts.

Checks: ERC 0 errors, 16 warnings (6 fewer than bef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
Parts:
- removed C73: 1 uF, Capacitor_SMD:C_0402_1005Metric, symbol Device:C
- removed D7: SP0503BAHTG, Footprints:TVS-SP05_LTF, symbol Custom:SP0503BAHTG
- removed D9: CUS10S30, Footprints:USC_TOS, symbol Custom:CUS10S30_H3F
- removed J5: USB4110GFA, Footprints:GCT_USB4110GFA, symbol Custom:USB4110GFA
- removed R20, R21: 5.11 k, Resistor_SMD:R_0402_1005Metric, symbol Device:R_US
Connections:
- no-connect marks 2 -> 0
Other:
- note removed: "USB-C"

Commit message: hardware: the 1 uF 0402 caps consolidate on the 16 V CL05A105KO5NNNC, with the pending part and layout work
Every GRM155R61A105KE15D (Murata, 10 V X5R) becomes the Samsung CL05A105KO5NNNC (16 V X5R) on
space-bug-m8t, gnss-sdr-dev and the legacy gnss-px1105r board -- 34 symbols and their 34 footprints.
Same 0402 footprint, so only the MPN and Mfr change. The higher-rated part is already the 1 uF used
on the Tinker boards, so the BOMs now carry one 1 uF line instead of two.

Pending work committed alongside:
- space-bug-m8t: the 10 uF bulk caps go to CL21A226MOQNNNE, added CL05A106MQ5NUNC, RC0402FR-071KL and
  R-667995 parts, schematic, layout and DRC rule updates, and the new FABRICATION-NOTES.md
- gnss-sdr-dev: the 5.1 nH inductors go from LQG15HS5N1S02D to LQW15AN5N1C00D, added 1 k and 100 k
  resistors, and schematic and layout updates
- legacy gnss-px1105r: the 10 uF caps go to CL21A226MOQNNNE, plus schematic and layout updates
- tinker-beetle: the 390 pF caps go to GRM1555C1H391JA01D, the 100 k resistors to RC0402FR-07100KL,
  and the 2.2 uH inductor from XGL4020-222ME to SRP4020FA-2R2M
- gnss-sam10m8-18mm-hv: the 100 pF cap goes from CL05C101JB5NNNC to GRM1555C1H101JA01D
- the Taoglas CGGBP.25.4.A.02 antenna footprint, and project-file housekeeping

Co-Authored-By: Claude Opus 5.5 <noreply@anthropic.com>
Connections:
- net +BATT renamed +BATT_F
Changed lines of the file:
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@@
 			)
 		)
-		(property "Value" "+BATT"
+		(property "Value" "+BATT_F"
 			(at 149.86 59.69 0)
 			(show_name no)
