File: hardware/tinker-base/battery.kicad_sch (KiCad schematic)
At the start: 23 parts, among them J2 TYPE-C-31-M-12, Q1 FS8205A, Q2 FS8205A, Q3 FS8205A, U14 DW01A, U5 BQ21040DBVR

Commit message: hardware(Tinker-Base): V1 design review and fixes -- the antenna window clear on every layer, 21 ground vias, L5/C25/fiducials, R52 1.2 k, and fab notes for the order
Stacked on #1545 (the Beetle/Mantis parts). The V1 JLC package was plotted from
exactly this board (md5 1fe1e414).

The review is new: hardware/tinker-base/design-review-2026-09-28.md. It has a
table of the fixes applied, and of the items left undone with the reason for each.

Layout (tinker-base.kicad_pcb):
- U15 antenna. F.Cu keeps the feed notch. A second rule area clears In1, In2 and
  B.Cu under the whole 4.6 x 3.0 mm window. Before this, In1 GND, In2 +3V3 and
  B.Cu GND filled under the feed pads. Nine GND fence vias.
- 21 GND vias: nine beside signal vias (signal vias more than 1 mm from a
  ground via: 14 -> 5), nine in U3's exposed pad between its paste windows, one
  for C16/C24 and two for U16's ground pads. Five old vias removed.
- J8 moved so its pads start 0.30 mm inside the edge. L5 (330 nH) runs from the
  SMA line to GND beside it.
- C25 (100 nF) on V_SWITCH at U9.
- J2's signal pads trimmed to HRO's land, in the library too. BT2.P to J2 goes
  from 0.40 to 0.84 mm.
- S3 gets an F.Cu keep-out over its body, and its GPIO0 via moves out from
  under it.
- Thermal reliefs on J2's shell legs and D6's cathode. Pin-1 dots on U3, U5, U22,
  CR1 and U16. FID1-FID3 added, R13/R16 refs hidden, and a B.Silk "-" at BT2's
  N end.
- Zones refilled. A second kicad-cli refill reproduces them byte for byte.

Schematic:
- L5, C25 and FID1-FID3 added.
- R52 680 -> 1.2 k. The charge current drops from 0.79 A to about 0.45 A, so the
  charger's heat no longer trips the board-mounted NTC from room temperature.
- Title blocks, rev V1, on all four sheets.
- bom.csv regenerated.

Library:
- IC_ESP32-S3 and 8L_WSON_8x6x3p4x4p3_MAC go back to their window polygons.
  4078070b had added paste pads on top of those polygons.
- USB_C_HRO_TYPE-C-31-M-12 pads trimmed.
- ANT_AANI-CH-0070_ABR's description states the r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
Parts:
- R52: value 680 -> 1.2 k; MPN RC0402FR-07680RL -> RC0402FR-071K2L
Other:
- company: (none) -> TinkerRocket
- title: (none) -> tinker-base: Battery
Changed lines of the file:
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@@
 	(generator_version "10.0")
 	(paper "A4")
+	(title_block
+		(title "tinker-base: Battery")
+		(date "2026-09-28")
+		(rev "V1")
+		(company "TinkerRocket")
+	)
 	(text "1S Battery"
 		(exclude_from_sim no)
@@
 			)
 		)
-		(property "Value" "680"
+		(property "Value" "1.2 k"
 			(at 95.885 81.915 90)
 			(show_name no)
@@
 			)
 		)
-		(property "MPN" "RC0402FR-07680RL"
+		(property "MPN" "RC0402FR-071K2L"
 			(at 98.425 81.915 0)
 			(hide yes)

Commit message: hardware(Tinker-Base, Mantis, Beetle): J2 becomes the GCT USB4110-GF-A the other boards use, placed where the HRO sat, and S1's maker is C&K
Tinker-Base J2 moves from the HRO TYPE-C-31-M-12 to the GCT USB4110-GF-A that the
Mantis, Beetle, LoRa and Space Bug boards use (owner, 2026-10-03).

- Schematic: J2 already used the Custom:USB4110GFA symbol. Only its footprint and
  part fields change (Value, MF, MP, MPN, Mfr, Description_1), copied from the
  Mantis/Beetle/LoRa instances. Both footprints name their pads after the
  symbol's pin numbers, so the netlist is identical.
- PCB: the GCT footprint sits where the HRO did, with its front face on the HRO's
  (1.11 mm past the board edge). The signal pads land on the same x positions,
  the pegs move 0.03 mm, and every existing track still ends on a pad. The SMD
  shell tabs connect solid to the F.Cu ground pour. Two new GND vias between the
  tabs tie the shell to In1.Cu and B.Cu ground, which the HRO's plated slots
  reached directly. BT2's + pad stays 0.84 mm from J2. DRC: 0 errors (24
  silkscreen/library warnings, 26 before), 0 unconnected, 0 parity issues; the
  fills are a refill fixed point.
- FABRICATION-NOTES: J2 is fully SMT now. The slot annular-ring minimum and the
  hand-solder instructions go; the V1 HRO procedure is kept in the "why" notes.
  The README status records the change and the V1 order.
- The V1 boards ordered on 2026-09-29 (tag tinker-base-v1.0.0) have the HRO land
  and still take TYPE-C-31-M-12.

S1 slide switch (JS202011JCQN) on the Mantis and Beetle: Mfr Same Sky (CUI) -> C&K.
It is a C&K JS-series part, and its SnapEDA MF/MANUFACTURER fields already said
so. Run Update PCB on those two boards to carry the field over.

bom.csv rows were updated and checked against each schematic designator by
designator; tools/check_board_parity.py and tools/check_docs.py pass.

Co-Authored-By: Claude Opus 5.5 <noreply@anthropic.com>
Parts:
- J2: value TYPE-C-31-M-12 -> USB4110GFA; footprint Footprints:USB_C_HRO_TYPE-C-31-M-12 -> Footprints:GCT_USB4110GFA; Description_1 USB-C (USB TYPE-C) USB 2.0 Receptacle Connector, 16 Positio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 -> USB-C (USB TYPE-C) USB 2.0 Receptacle Connector 24 (16+8 Du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; MF Korean Hroparts -> GCT; MP TYPE-C-31-M-12 -> USB4110GFA; MPN TYPE-C-31-M-12 -> USB4110-GF-A; Mfr Korean Hroparts -> GCT
Changed lines of the file:
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@@
 			)
 		)
-		(property "Value" "TYPE-C-31-M-12"
+		(property "Value" "USB4110GFA"
 			(at 44.45 41.91 0)
 			(show_name no)
@@
 			)
 		)
-		(property "Footprint" "Footprints:USB_C_HRO_TYPE-C-31-M-12"
+		(property "Footprint" "Footprints:GCT_USB4110GFA"
 			(at 44.45 54.61 0)
 			(hide yes)
@@
 			)
 		)
-		(property "MF" "Korean Hroparts"
+		(property "MF" "GCT"
 			(at 44.45 54.61 0)
 			(hide yes)
@@
 			)
 		)
-		(property "Description_1" "USB-C (USB TYPE-C) USB 2.0 Receptacle Connector, 16 Position, top-mount SMT signals + through-hole shell legs"
+		(property "Description_1" "USB-C (USB TYPE-C) USB 2.0 Receptacle Connector 24 (16+8 Dummy) Position Surface Mount, Right Angle; Through Hole"
 			(at 44.45 54.61 0)
 			(hide yes)
@@
 			)
 		)
-		(property "MP" "TYPE-C-31-M-12"
+		(property "MP" "USB4110GFA"
 			(at 44.45 54.61 0)
 			(hide yes)
@@
 			)
 		)
-		(property "MPN" "TYPE-C-31-M-12"
+		(property "MPN" "USB4110-GF-A"
 			(at 44.45 54.61 0)
 			(hide yes)
@@
 			)
 		)
-		(property "Mfr" "Korean Hroparts"
+		(property "Mfr" "GCT"
 			(at 44.45 54.61 0)
 			(hide yes)
