File: hardware/tinker-base/power.kicad_sch (KiCad schematic)
At the start: 19 parts, among them U22 TPS22918DBVR, U9 TPS63020DSJR

Commit message: hardware(Tinker-Base): V1 design review and fixes -- the antenna window clear on every layer, 21 ground vias, L5/C25/fiducials, R52 1.2 k, and fab notes for the order (#1546)
* hardware(Tinker-Base): V1 design review and fixes -- the antenna window clear on every layer, 21 ground vias, L5/C25/fiducials, R52 1.2 k, and fab notes for the order

Stacked on #1545 (the Beetle/Mantis parts). The V1 JLC package was plotted from
exactly this board (md5 1fe1e414).

The review is new: hardware/tinker-base/design-review-2026-09-28.md. It has a
table of the fixes applied, and of the items left undone with the reason for each.

Layout (tinker-base.kicad_pcb):
- U15 antenna. F.Cu keeps the feed notch. A second rule area clears In1, In2 and
  B.Cu under the whole 4.6 x 3.0 mm window. Before this, In1 GND, In2 +3V3 and
  B.Cu GND filled under the feed pads. Nine GND fence vias.
- 21 GND vias: nine beside signal vias (signal vias more than 1 mm from a
  ground via: 14 -> 5), nine in U3's exposed pad between its paste windows, one
  for C16/C24 and two for U16's ground pads. Five old vias removed.
- J8 moved so its pads start 0.30 mm inside the edge. L5 (330 nH) runs from the
  SMA line to GND beside it.
- C25 (100 nF) on V_SWITCH at U9.
- J2's signal pads trimmed to HRO's land, in the library too. BT2.P to J2 goes
  from 0.40 to 0.84 mm.
- S3 gets an F.Cu keep-out over its body, and its GPIO0 via moves out from
  under it.
- Thermal reliefs on J2's shell legs and D6's cathode. Pin-1 dots on U3, U5, U22,
  CR1 and U16. FID1-FID3 added, R13/R16 refs hidden, and a B.Silk "-" at BT2's
  N end.
- Zones refilled. A second kicad-cli refill reproduces them byte for byte.

Schematic:
- L5, C25 and FID1-FID3 added.
- R52 680 -> 1.2 k. The charge current drops from 0.79 A to about 0.45 A, so the
  charger's heat no longer trips the board-mounted NTC from room temperature.
- Title blocks, rev V1, on all four sheets.
- bom.csv regenerated.

Library:
- IC_ESP32-S3 and 8L_WSON_8x6x3p4x4p3_MAC go b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
Parts:
- added C25, C26: 100 nF, Capacitor_SMD:C_0402_1005Metric, symbol Device:C
Connections:
- net +3V3: now also C26.1
- net GND: now also C25.2, C26.2
- net V_SWITCH: now also C25.1
Other:
- company: (none) -> TinkerRocket
- title: (none) -> tinker-base: Power Switch

Commit message: hardware(Tinker-Base V2): in-package flash, a log flash, the GCT USB-C, 330 R LED resistors and a fixed 3.3 V buck, schematic and layout (#1685)
V2 of the base station, in work (title blocks V2; V1 is tag tinker-base-v1.0.0).

- U3 is an ESP32-S3FH4R2 (4 MB flash + 2 MB PSRAM in the package); the WLCSP
  boot NOR U1 and its C1 are gone.
- U23, a GD25Q128ESIGR log flash, on GPIO4-7 (SPI3, the V2 base station's NAND
  pins), with R58-R60 pull-ups and C89.
- J2 is the GCT USB4110-GF-A, placed so its front face sits where HRO's did.
- R41/R54 LED resistors 330 R.
- U9 is the TPS62152RGTR fixed 3.3 V buck (as the Beetle/Mantis), replacing the
  TPS63020 and its R13/R16 divider. The first V1 board ran +3V3 at 6.4 V; its
  U9 symbol carried a stale MP = TPS63021DSJR. DEF to GND for 3.3 V; C90 soft
  start. The fab notes ask for LCSC C2070611 by code.
- PCB brought up to the schematic: buck re-laid, U23 placed and routed (SCK
  hops to B.Cu), U1's escapes removed, Volt_Read re-routed on B.Cu, J2 on the
  GCT land. DRC with schematic parity: 0 errors, 0 unconnected, 0 parity
  issues; 26 warnings as at V1's sign-off. check_board_parity passes.

Not done: gerbers/position file, bom.csv and the fab-notes order block (for a
V2 order), and the base-station firmware for the 4 MB table and the external
log flash. README *Status* has the details.

Co-authored-by: Claude Opus 5.5 <noreply@anthropic.com>
Parts:
- removed R13: 1 M, Resistor_SMD:R_0402_1005Metric, symbol Device:R_US
- removed R16: 180 k, Resistor_SMD:R_0402_1005Metric, symbol Device:R_US
- added C90: 10 nF, Capacitor_SMD:C_0402_1005Metric, symbol Device:C
- R54: value 150 -> 330; MPN RC0402FR-07150RL -> RC0402FR-07330RL
- U9: value TPS63020DSJR -> TPS62152RGTR; footprint Footprints:IC_TPS63021DSJR -> Footprints:QFN50P300X300X100-17N; symbol Custom:TPS63020DSJR -> Custom:TPS62152RGTR; AVAILABILITY Good -> (none); Check_prices https://www.snapeda.com/parts/TPS63021DSJR/Texas+Instrument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 -> https://www.snapeda.com/parts/TPS62152RGTR/Texas+Instrument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; DIGIKEY-PURCHASE-URL https://snapeda.com/shop?store=DigiKey&id=296571 -> (none); DigiKey_Part_Number (none) -> 296-43621-1-ND; MAXIMUM_PACKAGE_HEIGHT 1.00mm -> (none); MFANUFACTURER Texas Instruments -> (none); MOUSER-PURCHASE-URL https://snapeda.com/shop?store=Mouser&id=296571 -> (none); MP TPS63021DSJR -> TPS62152RGTR; MPN TPS63020DSJR -> TPS62152RGTR; PACKAGE VSON-14 Texas Instruments -> (none); PARTREV I -> (none); PRICE None -> (none); Package VSON-14 Texas Instruments -> VQFN-16 Texas Instruments; STANDARD Manufacturer Recommendations -> (none); SnapEDA_Link https://www.snapeda.com/parts/TPS63021DSJR/Texas+Instrument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 -> https://www.snapeda.com/parts/TPS62152RGTR/Texas+Instrument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; TEXAS_INSTRUMENTS-PURCHASE-URL https://snapeda.com/shop?store=Texas+Instruments&id=296571 -> (none)
Connections:
- net +3V3: now also L9.2, U9.14 (VOS), U9.7 (FSW); no longer U9.4 (VOUT_4), U9.5 (VOUT_5)
- net GND: now also U9.16 (PGND), U9.17 (EP), U9.5 (FB), U9.6 (AGND), U9.8 (DEF), C90.2; no longer U9.13 (PS/SYNC), U9.2 (GND)
- net V_SWITCH: now also U9.13 (EN); no longer U9.1 (VINA)
- net at U9.3 (SW): now also L9.1, U9.1 (SW), U9.2 (SW)
- new net: C90.1, U9.9 (SS-TR)
- no-connect marks 0 -> 1
Other:
- note added: "Power 3.3 V @ 1 A"
- note removed: "Power 3.3 V @ 1.5 A"
- moved on the sheet: C25, L9
