File: hardware/space-bug-m8t/esp32_p4.kicad_sch (KiCad schematic)
At the start: 65 parts, among them U6 ESP32-P4NRW32X, U7 W25Q128JVYIQ, U8 TLV62569DRLR, U9 TPS62152RGTR, Y1 ECS-400-10-37B2-CKY-TR

Commit message: hardware: the 1 uF 0402 caps consolidate on the 16 V CL05A105KO5NNNC, with the pending part and layout work
Every GRM155R61A105KE15D (Murata, 10 V X5R) becomes the Samsung CL05A105KO5NNNC (16 V X5R) on
space-bug-m8t, gnss-sdr-dev and the legacy gnss-px1105r board -- 34 symbols and their 34 footprints.
Same 0402 footprint, so only the MPN and Mfr change. The higher-rated part is already the 1 uF used
on the Tinker boards, so the BOMs now carry one 1 uF line instead of two.

Pending work committed alongside:
- space-bug-m8t: the 10 uF bulk caps go to CL21A226MOQNNNE, added CL05A106MQ5NUNC, RC0402FR-071KL and
  R-667995 parts, schematic, layout and DRC rule updates, and the new FABRICATION-NOTES.md
- gnss-sdr-dev: the 5.1 nH inductors go from LQG15HS5N1S02D to LQW15AN5N1C00D, added 1 k and 100 k
  resistors, and schematic and layout updates
- legacy gnss-px1105r: the 10 uF caps go to CL21A226MOQNNNE, plus schematic and layout updates
- tinker-beetle: the 390 pF caps go to GRM1555C1H391JA01D, the 100 k resistors to RC0402FR-07100KL,
  and the 2.2 uH inductor from XGL4020-222ME to SRP4020FA-2R2M
- gnss-sam10m8-18mm-hv: the 100 pF cap goes from CL05C101JB5NNNC to GRM1555C1H101JA01D
- the Taoglas CGGBP.25.4.A.02 antenna footprint, and project-file housekeeping

Co-Authored-By: Claude Opus 5.5 <noreply@anthropic.com>
Parts:
- removed TP1: 3V3, TestPoint:TestPoint_Pad_D1.0mm, symbol Connector:TestPoint
- removed TP2: GND, TestPoint:TestPoint_Pad_D1.0mm, symbol Connector:TestPoint
- removed TP3: EN, TestPoint:TestPoint_Pad_D1.0mm, symbol Connector:TestPoint
- removed TP4: BOOT, TestPoint:TestPoint_Pad_D1.0mm, symbol Connector:TestPoint
- removed TP7: TXD0, TestPoint:TestPoint_Pad_D1.0mm, symbol Connector:TestPoint
- removed TP8: RXD0, TestPoint:TestPoint_Pad_D1.0mm, symbol Connector:TestPoint
- added C137: 10 uF, Capacitor_SMD:C_0402_1005Metric, symbol Device:C
- added R24: 1 k, Resistor_SMD:R_0402_1005Metric, symbol Device:R_US
- added SW1: R-667995, Footprints:R-667995_MIT, symbol Switch:SW_Push
- C29, C62, C63, C66, C67, C68, C69: MPN GRM155R61A105KE15D -> CL05A105KO5NNNC; Mfr Murata -> Samsung
Connections:
- net +3V3_MCU: now also C137.1
- net BOOT: now also R24.1
- net GND: now also C137.2, SW1.1
- new net: R24.2, SW1.2
Other:
- moved on the sheet: C42, C43, C44, C45, C46, C47, C48, C49, C50, C51, C52, C53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
