File: hardware/space-bug-m8t/space-bug-m8t.kicad_sch (KiCad schematic)
At the start: 41 parts, among them J4 BM05B-SRSS-TB, Q1 DTC123J, U1 NEO-M8T, U2 ADP7142ARDZ-3.3, U3 BGA524N6, U5 LP5907MFX-1.8

Commit message: hardware: the 1 uF 0402 caps consolidate on the 16 V CL05A105KO5NNNC, with the pending part and layout work
Every GRM155R61A105KE15D (Murata, 10 V X5R) becomes the Samsung CL05A105KO5NNNC (16 V X5R) on
space-bug-m8t, gnss-sdr-dev and the legacy gnss-px1105r board -- 34 symbols and their 34 footprints.
Same 0402 footprint, so only the MPN and Mfr change. The higher-rated part is already the 1 uF used
on the Tinker boards, so the BOMs now carry one 1 uF line instead of two.

Pending work committed alongside:
- space-bug-m8t: the 10 uF bulk caps go to CL21A226MOQNNNE, added CL05A106MQ5NUNC, RC0402FR-071KL and
  R-667995 parts, schematic, layout and DRC rule updates, and the new FABRICATION-NOTES.md
- gnss-sdr-dev: the 5.1 nH inductors go from LQG15HS5N1S02D to LQW15AN5N1C00D, added 1 k and 100 k
  resistors, and schematic and layout updates
- legacy gnss-px1105r: the 10 uF caps go to CL21A226MOQNNNE, plus schematic and layout updates
- tinker-beetle: the 390 pF caps go to GRM1555C1H391JA01D, the 100 k resistors to RC0402FR-07100KL,
  and the 2.2 uH inductor from XGL4020-222ME to SRP4020FA-2R2M
- gnss-sam10m8-18mm-hv: the 100 pF cap goes from CL05C101JB5NNNC to GRM1555C1H101JA01D
- the Taoglas CGGBP.25.4.A.02 antenna footprint, and project-file housekeeping

Co-Authored-By: Claude Opus 5.5 <noreply@anthropic.com>
Parts:
- C27, C28: MPN GRM155R61A105KE15D -> CL05A105KO5NNNC; Mfr Murata -> Samsung
- C7: value 10 uF -> 22 uF; MPN CL21A106KOQNNNE -> CL21A226MOQNNNE
