File: hardware/tinker-beetle/power.kicad_sch (KiCad schematic)
At the start: 72 parts, among them J3 JST_B2B-PH-SM4-TB, J6 USB4110GFA, Q11 AONR21321, U18 TPS62152RGTR, U19 TPS259631DDAR, U21 TPS2121RUXR, U30 TPS22810DRVR, U47 TPS61094DSS

Commit message: hardware: L11 becomes the Bourns SRP4020FA-2R2M on Bourns's own land; the XGL4020 land had its pads 0.49 mm too far out (#1538)
The TPS61094 hold-up inductor (L11, Mantis and Beetle) moves from the
Coilcraft XGL4020-222ME to the Bourns SRP4020FA-2R2M. The Coilcraft 4020
family is hard to buy: Mouser does not list the XGL4020, its XFL4020-222MEC
had 132 pieces on a 40-week lead, and Digi-Key only has marketplace
listings. Mouser had 11,042 of the Bourns part on 2026-09-27.

Electrically it meets the same need. In backup the boost runs into its
2.6 A (max) valley limit by design, so the worst peak is ~3.1 A with the
ripple at L -30 %. There the Bourns part is ~10 % down and the XGL4020
~12 %. DCR max 23.5 vs 21.5 mOhm; both are soft-saturating metal-powder
cores, unlike the rejected ferrite VLS3012CX.

The old land was misdrawn. In Coilcraft doc 1529, 2.37 mm is the pitch
between the pad centre lines, not the gap, so L_XGL4020_4.0x4.0mm put its
pads at +-1.675 mm instead of +-1.185 mm. Only ~0.42 of the XGL4020's
0.82 mm terminals, and ~0.50 of the Bourns part's 0.88 mm, reached copper.
That footprint and its model are deleted. The new IND_SRP4020FA-2R2M is
Bourns's Recommended Layout (1.4 x 3.4 mm pads, 3.8 mm overall, 1.0 mm
gap). Both the Bourns terminals and the Coilcraft XGL/XFL4020 terminals sit
fully on it. The 3D model is CadQuery-built from the datasheet's
dimensions (build script alongside).

Schematic only: L11's Footprint, MPN and Mfr fields change on both
boards, and bom.csv follows. Netlists are otherwise identical (nets
unchanged), ERC counts are unchanged (Mantis 933, Beetle 737), both BOMs
reconcile 0/0/0, and check_board_parity passes. DRC's only new items are
L11's footprint/MPN parity and the old library footprint no longer being
found. They clear when the PCBs are updated from the schematic, which is
the owner's layout step. On the current Mantis board, four vias and one
F.Cu track sit where the new pads go. The hold-up doc records the change.

Co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
Parts:
- L11: footprint Footprints:L_XGL4020_4.0x4.0mm -> Footprints:IND_SRP4020FA-2R2M; MPN XGL4020-222ME -> SRP4020FA-2R2M; Mfr Coilcraft -> Bourns
Changed lines of the file:
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@@
 			)
 		)
-		(property "Footprint" "Footprints:L_XGL4020_4.0x4.0mm"
+		(property "Footprint" "Footprints:IND_SRP4020FA-2R2M"
 			(at 231.14 72.39 0)
 			(hide yes)
@@
 			)
 		)
-		(property "MPN" "XGL4020-222ME"
+		(property "MPN" "SRP4020FA-2R2M"
 			(at 231.14 72.39 0)
 			(hide yes)
@@
 			)
 		)
-		(property "Mfr" "Coilcraft"
+		(property "Mfr" "Bourns"
 			(at 231.14 72.39 0)
 			(hide yes)

Commit message: hardware: the 1 uF 0402 caps consolidate on the 16 V CL05A105KO5NNNC, with the pending part and layout work
Every GRM155R61A105KE15D (Murata, 10 V X5R) becomes the Samsung CL05A105KO5NNNC (16 V X5R) on
space-bug-m8t, gnss-sdr-dev and the legacy gnss-px1105r board -- 34 symbols and their 34 footprints.
Same 0402 footprint, so only the MPN and Mfr change. The higher-rated part is already the 1 uF used
on the Tinker boards, so the BOMs now carry one 1 uF line instead of two.

Pending work committed alongside:
- space-bug-m8t: the 10 uF bulk caps go to CL21A226MOQNNNE, added CL05A106MQ5NUNC, RC0402FR-071KL and
  R-667995 parts, schematic, layout and DRC rule updates, and the new FABRICATION-NOTES.md
- gnss-sdr-dev: the 5.1 nH inductors go from LQG15HS5N1S02D to LQW15AN5N1C00D, added 1 k and 100 k
  resistors, and schematic and layout updates
- legacy gnss-px1105r: the 10 uF caps go to CL21A226MOQNNNE, plus schematic and layout updates
- tinker-beetle: the 390 pF caps go to GRM1555C1H391JA01D, the 100 k resistors to RC0402FR-07100KL,
  and the 2.2 uH inductor from XGL4020-222ME to SRP4020FA-2R2M
- gnss-sam10m8-18mm-hv: the 100 pF cap goes from CL05C101JB5NNNC to GRM1555C1H101JA01D
- the Taoglas CGGBP.25.4.A.02 antenna footprint, and project-file housekeeping

Co-Authored-By: Claude Opus 5.5 <noreply@anthropic.com>
Parts:
- C44: MPN CL05C391JB5NNNC -> GRM1555C1H391JA01D
- R44: MPN RT0402BRD07100KL -> RC0402FR-07100KL
Changed lines of the file:
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@@
 			)
 		)
-		(property "MPN" "CL05C391JB5NNNC"
+		(property "MPN" "GRM1555C1H391JA01D"
 			(at 55.245 122.555 0)
 			(hide yes)
@@
 			)
 		)
-		(property "MPN" "RT0402BRD07100KL"
+		(property "MPN" "RC0402FR-07100KL"
 			(at 51.435 156.21 0)
 			(hide yes)
