File: hardware/tinker-beetle/pyro.kicad_sch (KiCad schematic)
At the start: 42 parts, among them J2 JL212R-SMT-35005BP1, Q12 DTC123J, Q13 DTA123J, Q14 DTC123J, Q3 DTC123J, Q4 DTC123J, Q5 DTC123J, Q6 DTC123J, U10 WSD20L50DN33, U6 WSD20L50DN33, U7 WSD20L50DN33, U8 WSD20L50DN33, U9 AON7534

Commit message: hardware(Tinker-Beetle V2, Tinker-Mantis V11, LoRa V4): the ESP32-S3s take their boot flash in the package, and the Beetle's V2 work to date (#1684)
Every in-work board's ESP32-S3RH2 + external W25Q128JVYIQ becomes an
ESP32-S3FH4R2 (4 MB quad flash + the same 2 MB quad PSRAM in the package,
same QFN-56 and pinout). The boot NOR and its 100 nF go; pads 30-35 carry
no-connect flags. The S3FN8 was not used: the Beetle FC's raw-GNSS filter
keeps ~219 KB in PSRAM and the OC's log ring is 512 KB there.

- Tinker-Beetle V2: U15/U32 -> FH4R2; U13, U33, C26, C115 removed.
- Tinker-Mantis V11: out computer U15 -> FH4R2; U13, C26 removed. The P4's
  boot flash U16 stays (no P4 has in-package flash).
- LoRa daughterboard V4: U28 -> FH4R2; U22, C18 removed. radio_board already
  declares 4 MB with PSRAM off, so its firmware needs no change.

The Beetle folder also carries the rest of its uncommitted V2 work, which
shares these files: TPS1HC08-Q1 eFuse pyro switches (U6-U8, U10, R144-R147;
Q3-Q6 gone), the PX1105R (U12) with its GVLB208.A antenna, the MMC5983MA
magnetometer on the sensor SPI, the Molex 0479480001 BLE antenna, the WAGO
2601-1105 battery terminal (J2), the SHOU HAN vertical USB-C (J6), no FC
32.768 kHz crystal (Y3), the BAT54XV2T1G power-switch OR (D9/D12) and the
BOM consolidation. The libraries gain the symbols and footprints those use
(MMC5983MA's GND pins become power inputs).

Checked: tools/check_board_parity.py passes on every board. ERC and
netlists match the working copy they came from. PCB DRC with schematic
parity: LoRa 0 unconnected, Mantis 4, Beetle 190 (its V2 layout is in
progress). Firmware for the 4 MB partition tables (Beetle V2, Mantis V11
OC) is not part of this.

Not included: Tinker-Base V2 (FH4R2 + U23 log flash, GCT USB4110-GF-A J2,
330 ohm LED resistors). Its PCB has not been updated yet, so it fails the
board-parity check.

Co-authored-by: Claude Opus 5.5 <noreply@anthropic.com>
Parts:
- removed Q3, Q4, Q5, Q6: DTC123J, Footprints:TRANS_SOT-416_EMT3-EMT3F_ROHM, symbol Transistor_BJT:DTC123J
- added C153, C154, C155, C156: 100 nF, Capacitor_SMD:C_0402_1005Metric, symbol Device:C
- added R144, R145, R146, R147: 33.2 k, Resistor_SMD:R_0402_1005Metric, symbol Device:R_US
- J2: value JL212R-SMT-35005BP1 -> 2601-1105; footprint Footprints:CUI_TBLH11-350-05-BK -> Footprints:WAGO_2601-1105; symbol Custom:TBLH11-350-05-BK -> Custom:WAGO_2601-1105; MANUFACTURER CUI Devices -> (none); MAXIMUM_PACKAGE_HEIGHT 8.8mm -> (none); MPN JL212R-SMT-35005BP1 -> 2601-1105; Mfr JILN -> WAGO; PARTREV 1.0 -> (none); STANDARD Manufacturer Recommendations -> (none)
- R132, R21: value 100 -> 22; MPN RC0402FR-07100RL -> RC0402FR-0722RL
- U10, U6, U7, U8: value WSD20L50DN33 -> TPS1HC08-Q1; footprint Footprints:TSON Advance_TOS -> Footprints:VAH0011B; symbol Custom:WSD20L50DN33 -> Custom:TPS1HC08-Q1; MPN WSD20L50DN33 -> TPS1HC08PQVAHRQ1; Mfr Winsok -> Texas Instruments
Connections:
- net GND: now also U10.4 (GND), U6.4 (GND), U7.4 (GND), U8.4 (GND), C153.2, C154.2, C155.2, C156.2, R144.2, R145.2, R146.2, R147.2
- net PYRO1_EXT: now also J2.5, U8.1 (VOUT), U8.11 (VOUT); no longer J2.1_1 (1), J2.1_2 (1__1), U8.5 (DRAIN), U8.6 (DRAIN), U8.7 (DRAIN), U8.8 (DRAIN)
- net PYRO1_FIRE: now also R15.2
- net PYRO2_EXT: now also J2.4, U6.1 (VOUT), U6.11 (VOUT); no longer J2.2_1 (2), J2.2_2 (2__1), U6.5 (DRAIN), U6.6 (DRAIN), U6.7 (DRAIN), U6.8 (DRAIN)
- net PYRO2_FIRE: now also R16.2
- net PYRO3_EXT: now also J2.3, U7.1 (VOUT), U7.11 (VOUT); no longer J2.3_1 (3), J2.3_2 (3__1), U7.5 (DRAIN), U7.6 (DRAIN), U7.7 (DRAIN), U7.8 (DRAIN)
- net PYRO3_FIRE: now also R17.2
- net PYRO4_EXT: now also J2.2, U10.1 (VOUT), U10.11 (VOUT); no longer J2.4_1 (4), J2.4_2 (4__1), U10.5 (DRAIN), U10.6 (DRAIN), U10.7 (DRAIN), U10.8 (DRAIN)
- net PYRO4_FIRE: now also R23.2
- net PYRO_GND: now also J2.1; no longer J2.5_1 (5), J2.5_2 (5__1)
- net VBAT_CON: now also C153.1, C154.1, C155.1, C156.1; no longer R15.2, R16.2, R17.2, R23.2, U10.1 (SOURCE), U10.3 (SOURCE), U6.1 (SOURCE), U6.3 (SOURCE), U7.1 (SOURCE), U7.3 (SOURCE), U8.1 (SOURCE), U8.3 (SOURCE)
- net at R16.1: now also U6.7 (EN); no longer U6.4 (GATE)
- net at R17.1: now also U7.7 (EN); no longer U7.4 (GATE)
- net at R23.1: now also U10.7 (EN); no longer U10.4 (GATE)
- net at R15.1: now also U8.7 (EN); no longer U8.4 (GATE)
- new net: R145.1, U6.3 (ILIM)
- new net: R146.1, U7.3 (ILIM)
- new net: R144.1, U8.3 (ILIM)
- new net: R147.1, U10.3 (ILIM)
- no-connect marks 0 -> 12
Other:
- moved on the sheet: R15, R16, R17, R23
