File: hardware/spin-rig-controller/io.kicad_sch (KiCad schematic)
At the start: 47 parts, among them J301 CL57T CONTROL, J302 ENCODER, J303 INDEX, J304 GNSS, U301 SN74ACT244PWR, U302 AM26LV32EIDR, U303 SN74LVC1G17DBVR, U304 SN74LVC2G125DCTR

Commit message: hardware(spin-rig-controller): the driver's own plugs -- XT60 pack input, CL57T 3.5 mm headers in its pin order, and an encoder pass-through
After the first review, the connectors change so the assembly plugs together instead of being wired up:
- J101 is an XT60PW-M (right angle, top edge), matching the rig's pack and anti-spark switch;
- J103 (driver feed), J301 (control) and the new J305 (encoder out) are 3.5 mm Phoenix MC headers that take
  the CL57T's own pluggable plugs, in its order: P4 +VDC GND; P1 PUL+ PUL- DIR+ DIR- ENA+ ENA- ALM BRK COM-;
  P2 EB+ EB- EA+ EA- VCC EGND. The silkscreen names every pin;
- the motor's encoder extension lead lands on J302 (right edge) and passes through to J305; the AM26LV32E
  reads A and B on the way. J302 is numbered from the bottom so the six traces nest around the corner;
- J303, J304 and J104 become through-hole JST PH. J102 (brake resistor) is now the only VH connector, which
  ends the three look-alike power connectors.

The CL57T V4.x has no in-position output: its ALM and BRK are open-collector to a shared COM- (CL57T V4.0
manual, CL42T/CL86T V4.1 manuals). The input that read PEND now reads BRK (DRV_BRK, GPIO2), and ENC_Z is
dropped (the encoder has no index; GPIO35 is free). The Qwiic connector moves beside the INA238.

Through-hole parts (design.HAND) are out of the JLC BOM and CPL; make_fab.py lists them in -hand.csv
(29 extended part types now, about $23 of JLC parts a board). The router's leftovers are closed by
gen/hand_fixes.py, planned against the copper around each (gen/region.py lists a window's copper).
ERC 0 errors (the shared SP0503 symbol's 4 warnings); DRC 0 errors, 0 unconnected, schematic parity clean;
tools/check_board_parity.py passes. Still to measure: the CL57T's terminal pitch (3.5 mm assumed). Not ordered.

Co-Authored-By: Claude Opus 5.5 <noreply@anthropic.com>
Parts:
- removed R315: 120, Resistor_SMD:R_0402_1005Metric, symbol Device:R
- added J305: ENCODER OUT, Connector_Phoenix_MC:PhoenixContact_MC_1,5_6-G-3.5_1x06_P3.50mm_Horizontal, symbol Connector_Generic:Conn_01x06
- J301: footprint Connector_JST:JST_PH_B10B-PH-SM4-TB_1x10-1MP_P2.00mm_Vertical -> Connector_Phoenix_MC:PhoenixContact_MC_1,5_9-G-3.5_1x09_P3.50mm_Horizontal; symbol Connector_Generic:Conn_01x10 -> Connector_Generic:Conn_01x09; LCSC C264997 -> C3581423; MPN B10B-PH-SM4-TB(LF)(SN) -> 1844281; Mfr JST -> Phoenix Contact
- J302: value ENCODER -> ENCODER IN; footprint Connector_JST:JST_PH_B8B-PH-SM4-TB_1x08-1MP_P2.00mm_Vertical -> Connector_Phoenix_MC:PhoenixContact_MC_1,5_6-G-3.5_1x06_P3.50mm_Horizontal; symbol Connector_Generic:Conn_01x08 -> Connector_Generic:Conn_01x06; LCSC C495548 -> C3580663; MPN B8B-PH-SM4-TB(LF)(SN) -> 1844252; Mfr JST -> Phoenix Contact
- J303: footprint Connector_JST:JST_PH_B4B-PH-SM4-TB_1x04-1MP_P2.00mm_Vertical -> Connector_JST:JST_PH_B4B-PH-K_1x04_P2.00mm_Vertical; LCSC C160354 -> (none); MPN B4B-PH-SM4-TB(LF)(SN) -> B4B-PH-K-S(LF)(SN)
- J304: footprint Connector_JST:JST_PH_B3B-PH-SM4-TB_1x03-1MP_P2.00mm_Vertical -> Connector_JST:JST_PH_B3B-PH-K_1x03_P2.00mm_Vertical; LCSC C160353 -> (none); MPN B3B-PH-SM4-TB(LF)(SN) -> B3B-PH-K-S(LF)(SN)
Connections:
- net ENC_A_N: now also J302.3 (Pin_3), J305.4 (Pin_4); no longer J302.2 (Pin_2)
- net ENC_A_P: now also J302.4 (Pin_4), J305.3 (Pin_3); no longer J302.1 (Pin_1)
- net ENC_B_N: now also J302.5 (Pin_5), J305.2 (Pin_2); no longer J302.4 (Pin_4)
- net ENC_B_P: now also J302.6 (Pin_6), J305.1 (Pin_1); no longer J302.3 (Pin_3)
- net ENC_GND: now also J302.1 (Pin_1), J305.6 (Pin_6); no longer J302.7 (Pin_7)
- net GND: now also J301.9 (Pin_9); no longer J301.10 (Pin_10), J301.8 (Pin_8)
- net ENC_Z: no longer names the net of U302.11 (3Y)
- net ENC_Z_N: no longer names the net of U302.9 (3B)
- net ENC_Z_N: no longer J302.6 (Pin_6)
- net ENC_Z_P: no longer names the net of U302.10 (3A)
- net ENC_Z_P: no longer J302.5 (Pin_5)
- net PEND renamed DRV_BRK
- net PEND_P renamed BRK_P
- net BRK_P: now also J301.8 (Pin_8); no longer J301.9 (Pin_9)
- new net ENC_VCC: J302.2 (Pin_2), J305.5 (Pin_5)
- no-connect marks 10 -> 12
Other:
- note added: "Encoder pass-through and tap (the receiver listens in parallel with the driver)"
- note removed: "Encoder tap (in parallel with the driver's encoder input)"
- moved on the sheet: C301, C302, C303, C304, R301, R302, R303, R304, R305, R306, R307, R308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

Commit message: hardware(spin-rig-controller): 67 x 90 mm over the Pi 4B -- covers the Pi but its port end, same connectors, one-sided 4-layer
The 110 x 80 board left a lot of empty copper. It now sits over the Pi on the
same 11 mm standoffs and the Pi's four M2.5 holes, with a 25 mm strip at the
top (XT60, input stage, encoder-out) and an 11 mm strip down the right (the
driver headers, index, GNSS) as the only overhang. Every connector and the
encoder pass-through stay; all SMD parts stay on the top side.

- design.py: the three M3 holes and the fiducials dropped (Economic
  assembly doesn't use them).
- make_pcb.py: new placement around U201_XY/U104_XY; the buck's BOOT/RT/EN
  runs and the ESP32's bottom fan-out are now locked pre-routes relative to
  those parts; In2's 5 V plane is the bottom 22 mm; Pi feed re-laid.
- fixup.py: the ESP32's 1.5 mm stitching grid follows U201_XY.
- silk.py: the title shrinks or turns to fit; pin labels and header names
  packed for the right edge.
- hand_fixes.py: re-planned for this routing result.
- README and FABRICATION-NOTES: 67 x 90, 540 vias, new pin-1 table and
  tooling-hole spots.

DRC 0 errors / 0 warnings / 0 unconnected, schematic parity clean, ERC 0
errors (the shared SP0503 symbol's 4 warnings), parity gate 167 symbols.

Co-Authored-By: Claude Opus 5.5 <noreply@anthropic.com>
Parts:
- TP301, TP302, TP303, TP304, TP305, TP306: footprint TestPoint:TestPoint_Pad_D1.5mm -> TestPoint:TestPoint_Pad_D1.0mm
Changed lines of the file:
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@@
 			)
 		)
-		(property "Footprint" "TestPoint:TestPoint_Pad_D1.5mm"
+		(property "Footprint" "TestPoint:TestPoint_Pad_D1.0mm"
 			(at 339.09 246.38 0)
 			(hide yes)
@@
 			)
 		)
-		(property "Footprint" "TestPoint:TestPoint_Pad_D1.5mm"
+		(property "Footprint" "TestPoint:TestPoint_Pad_D1.0mm"
 			(at 355.6 246.38 0)
 			(hide yes)
@@
 			)
 		)
-		(property "Footprint" "TestPoint:TestPoint_Pad_D1.5mm"
+		(property "Footprint" "TestPoint:TestPoint_Pad_D1.0mm"
 			(at 370.84 246.38 0)
 			(hide yes)
@@
 			)
 		)
-		(property "Footprint" "TestPoint:TestPoint_Pad_D1.5mm"
+		(property "Footprint" "TestPoint:TestPoint_Pad_D1.0mm"
 			(at 387.35 246.38 0)
 			(hide yes)
@@
 			)
 		)
-		(property "Footprint" "TestPoint:TestPoint_Pad_D1.5mm"
+		(property "Footprint" "TestPoint:TestPoint_Pad_D1.0mm"
 			(at 403.86 246.38 0)
 			(hide yes)
@@
 			)
 		)
-		(property "Footprint" "TestPoint:TestPoint_Pad_D1.5mm"
+		(property "Footprint" "TestPoint:TestPoint_Pad_D1.0mm"
 			(at 419.1 246.38 0)
 			(hide yes)
