File: hardware/gnss-px100-18mm-hv/receiver.kicad_sch (KiCad schematic)
At the start: 64 parts, among them J1 CON-SMA-EDGE-S, U1 PX100-5C-01A, U3 BGA855N6, U4 BGA855N6, Y1 TG2520SMN 26 MHz, Y2 32.768 kHz

Commit message: hardware(gnss-px100): L13 not fitted and C37 1.3 pF -- the L5 arm no longer grounds the PX100's LNA_IN2 for DC
Both SkyTraq references (PX100-5C and -5S data sheets) feed each LNA
input through a shunt capacitor at the band SAW and a series inductor,
so the pin has no DC path to ground. The L5 arm as drawn had one: FL7's
6.8 nH output shunt (L13) and the 12 nH series L15 tied pin 37 to
ground. If the PX100 biases its LNA inputs through the pins, that kills
the L5 LNA. The TinkerNav PX100 V2 grounds both inputs the same way and
never tracked anything; no TinkerNav PX100 has worked.

L13 is now not fitted and C37 goes from 4 pF to 1.3 pF (Murata
GJM1555C1H1R3BB01D, LCSC C161309). At 1176.45 MHz, 4 pF in parallel
with 6.8 nH is +9.7 mS, a 1.31 pF capacitor. Across 1164-1189 MHz the
two differ by about 0.4 mS, less than C37's own +/-0.1 pF tolerance.
The change is parts only, so it applies to the ordered V1 boards too.

The README gains the reasoning, a "no working PX100 to copy" note in
place of the TinkerNav evidence paragraph, and a bring-up step that
meters pins 37 and 40. The fab notes flag L13 as not fitted, give C37's
new part, and say to build from the in-work schematic rather than the
tag. The sheet's stage-2 note is rewritten and moved down so it clears
the ground symbols. ERC, netlist (only C37's value) and DRC with parity
are unchanged.

Co-Authored-By: Claude Opus 5.5 <noreply@anthropic.com>
Parts:
- C37: value 4 pF -> 1.3 pF; Dist_PN C161323 -> C161309; MPN GJM1555C1H4R0BB01D -> GJM1555C1H1R3BB01D
- L13: now not fitted
Other:
- note added: "Stage 2, SkyTraq's split: lumped Wilkinson L10/L11 6.8 nH, C34/C35 1.5 pF, R10 100 ohm, C33 2.7 pF (centred on L1). FL6 is 50 ohm with no matching; FL7 (Murata) needs its 10 nH input shunt (L12). C36+L14 and C37+L15 are SkyTraq's input matches into the PX100 LNAs, which keep both LNA inputs free of any DC path. L13 (FL7's 6.8 nH output shunt) is NOT fitted: with L15 in series it would ground LNA_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"
- note removed: "Stage 2, SkyTraq's split: lumped Wilkinson L10/L11 6.8 nH, C34/C35 1.5 pF, R10 100 ohm, C33 2.7 pF (centred on L1). FL6 is 50 ohm with no matching; FL7 (Murata) needs its 10 nH (L12) and 7 nH (L13, 6.8 nH fitted) shunts. C36+L14 and C37+L15 are SkyTraq's input matches into the PX100 LNAs."
Changed lines of the file:
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@@
 		)
 	)
-	(text "Stage 2, SkyTraq's split: lumped Wilkinson L10/L11 6.8 nH, C34/C35 1.5 pF, R10 100 ohm, C33 2.7 pF (centred on L1).\nFL6 is 50 ohm with no matching; FL7 (Murata) needs its 10 nH (L12) and 7 nH (L13, 6.8 nH fitted) shunts.\nC36+L14 and C37+L15 are SkyTraq's input matches into the PX100 LNAs."
+	(text "Stage 2, SkyTraq's split: lumped Wilkinson L10/L11 6.8 nH, C34/C35 1.5 pF, R10 100 ohm, C33 2.7 pF (centred on L1).\nFL6 is 50 ohm with no matching; FL7 (Murata) needs its 10 nH input shunt (L12).\nC36+L14 and C37+L15 are SkyTraq's input matches into the PX100 LNAs, which keep both LNA inputs free of any DC path.\nL13 (FL7's 6.8 nH output shunt) is NOT fitted: with L15 in series it would ground LNA_IN2 for DC.\nC37 is 1.3 pF, the same admittance at 1176.45 MHz as the reference 4 pF in parallel with 6.8 nH."
 		(exclude_from_sim no)
-		(at 195.58 99.06 0)
+		(at 195.58 102.87 0)
 		(effects
 			(font
@@
 		(on_board yes)
 		(in_pos_files yes)
-		(dnp no)
+		(dnp yes)
 		(property "Reference" "L13"
 			(at 320.04 82.55 0)
@@
 			)
 		)
-		(property "Value" "4 pF"
+		(property "Value" "1.3 pF"
 			(at 330.2 85.09 0)
 			(show_name no)
@@
 			)
 		)
-		(property "MPN" "GJM1555C1H4R0BB01D"
+		(property "MPN" "GJM1555C1H1R3BB01D"
 			(at 327.66 83.82 0)
 			(hide yes)
@@
 			)
 		)
-		(property "Dist_PN" "C161323"
+		(property "Dist_PN" "C161309"
 			(at 327.66 83.82 0)
 			(hide yes)

Commit message: hardware(gnss-px100): C48 becomes a 0 ohm link -- the TCXO drives TCXO_I directly, as in SkyTraq's reference
C48 was a 1 nF DC cut between Y1's clipped-sine output and the PX100's
TCXO_I (pin 4). It came from the TCXO data sheets: Epson specifies its
output through a 10 nF DC cut. SkyTraq's reference (PX100-5C data sheet)
wires the TCXO straight to pin 4, and so do the TinkerNav PX100s. Their
RF never worked, but they boot, with an ECS TCXO whose clipped-sine
output drives the same 10 kohm // 10 pF load. So pin 4 is known to
take a TCXO's DC level, while nothing shows it biases itself behind a
series capacitor.

C48 keeps its designator and its 0402 capacitor pads, so the ordered
V1 copper is unchanged. It is drawn as Device:R_Small (the same 2.54 mm
pin offsets as C_Small, so no wire moves) and is now a UNI-ROYAL
0402WGF0000TCE 0 ohm jumper (LCSC C17168). The README and fab notes
give the reasoning and the bring-up fallback: if the PX100 stays silent
or pin 4 shows no clean 26 MHz, refit 1 nF. The sheet's Y1 note says
the same. ERC, netlist (only C48's value) and DRC with parity are
unchanged.

Co-Authored-By: Claude Opus 5.5 <noreply@anthropic.com>
Parts:
- C48: value 1 nF -> 0R; symbol Device:C_Small -> Device:R_Small; Dist_PN C76947 -> C17168; MPN GRM1555C1H102JA01D -> 0402WGF0000TCE; Mfr Murata -> UNI-ROYAL
Other:
- note added: "Y1: Epson TG2520SMN 26 MHz, +/-0.5 ppm, fed by the PX100's own TCXO LDO (pin 3). Its long side is the g-sensitive X axis (0.4 ppb/g typ): keep it along board x, across the thrust. C48 is a 0 ohm link: the TCXO drives TCXO_I directly, as in SkyTraq's reference (refit 1 nF if the clock fails). Y2: 32.768 kHz, no load capacitors."
- note removed: "Y1: Epson TG2520SMN 26 MHz, +/-0.5 ppm, fed by the PX100's own TCXO LDO (pin 3). Its long side is the g-sensitive X axis (0.4 ppb/g typ): keep it along board x, across the thrust. C48 is the DC-cut its output needs. Y2: 32.768 kHz, no load capacitors."
Changed lines of the file:
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@@
 		)
 	)
-	(text "Y1: Epson TG2520SMN 26 MHz, +/-0.5 ppm, fed by the\nPX100's own TCXO LDO (pin 3). Its long side is the\ng-sensitive X axis (0.4 ppb/g typ): keep it along board x,\nacross the thrust. C48 is the DC-cut its output needs.\nY2: 32.768 kHz, no load capacitors."
+	(text "Y1: Epson TG2520SMN 26 MHz, +/-0.5 ppm, fed by the\nPX100's own TCXO LDO (pin 3). Its long side is the\ng-sensitive X axis (0.4 ppb/g typ): keep it along board x,\nacross the thrust. C48 is a 0 ohm link: the TCXO drives TCXO_I\ndirectly, as in SkyTraq's reference (refit 1 nF if the clock fails).\nY2: 32.768 kHz, no load capacitors."
 		(exclude_from_sim no)
 		(at 110.49 205.74 0)
@@
 	)
 	(symbol
-		(lib_id "Device:C_Small")
+		(lib_id "Device:R_Small")
 		(at 142.24 157.48 90)
 		(unit 1)
@@
 			)
 		)
-		(property "Value" "1 nF"
+		(property "Value" "0R"
 			(at 142.24 154.94 90)
 			(show_name no)
@@
 			)
 		)
-		(property "MPN" "GRM1555C1H102JA01D"
+		(property "MPN" "0402WGF0000TCE"
 			(at 142.24 157.48 0)
 			(hide yes)
@@
 			)
 		)
-		(property "Mfr" "Murata"
+		(property "Mfr" "UNI-ROYAL"
 			(at 142.24 157.48 0)
 			(hide yes)
@@
 			)
 		)
-		(property "Dist_PN" "C76947"
+		(property "Dist_PN" "C17168"
 			(at 142.24 157.48 0)
 			(hide yes)
