File: hardware/px100-test-board/px100-test-board.kicad_pcb (KiCad board)
At the start: 4 copper layers, 75 x 52 mm, 164 parts, among them J1 CON-SMA-EDGE-S, J101 USB4110GFA, J201 ESP32 SPARE, J301 PX100 PINS, Q301 MMBT3904, Q302 MMBT3904, SW201 BOOT, SW202 RESET, SW301 PX RESET, SW302 PX BOOT, U1 PX100-5C-01A, U101 FSUSB63UMX, U103 AP2112K-3.3TRG1, U104 ADP7142ARDZ-3.3, U201 ESP32-S3FN8, U301 CP2102N-A02-GQFN24, Y1 TG2520SMN 26 MHz, Y2 32.768 kHz, Y201 40 MHz

Commit message: hardware(px100-test-board): ESP32-S3FH4R2 in place of the FN8 -- the Beetle JLC build's part
Same QFN-56 footprint and pinout, so the layout is untouched: only U201's
value, MPN and LCSC fields change (C3013940, 2,862 at JLC on 2026-10-29).
The FH4R2 has 4 MB of flash and 2 MB of quad PSRAM in the package; its
flash pins (GPIO27-32) and the PSRAM's chip select (SPICS1/GPIO26) were
already unconnected here, and quad PSRAM leaves GPIO33-37 free for J201 and
USB_SEL_MCU. Firmware needs a 4 MB flash size and partition table.

ERC 0 errors; DRC 0 errors, 0 unconnected, schematic parity 0;
tools/check_board_parity.py passes.

Co-Authored-By: Claude Opus 5.5 <noreply@anthropic.com>
Parts:
- U201: value ESP32-S3FN8 -> ESP32-S3FH4R2
Changed lines of the file:
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@@
 			)
 		)
-		(property "Value" "ESP32-S3FN8"
+		(property "Value" "ESP32-S3FH4R2"
 			(at 2.885 5.635 0)
 			(layer "F.Fab")
@@
 			)
 		)
-		(property "Description" "8 MB flash in the package; the rocket boards' footprint"
+		(property "Description" "4 MB flash and 2 MB quad PSRAM in the package (flash on GPIO27-32, PSRAM on SPICS1/GPIO26); the rocket boards' footprint"
 			(at 0 0 0)
 			(layer "F.Fab")
@@
 			)
 		)
-		(property "LCSC" "C2913196"
+		(property "LCSC" "C3013940"
 			(at 0 0 0)
 			(layer "F.Fab")
@@
 			)
 		)
-		(property "MPN" "ESP32-S3FN8"
+		(property "MPN" "ESP32-S3FH4R2"
 			(at 0 0 0)
 			(layer "F.Fab")
